File: PCB/_autosave-custom_keyboard.sch (KiCad schematic (older format))
At the start: 33 parts

Commit message: Keyboard controller sections
Parts:
- removed MX?: MX-NoLED, symbol MX_Alps_Hybrid:MX-NoLED
- added D? (x2): SOD-123, symbol Device:D_Small
- added SW? (x2): CherryMX, symbol CherryMX:CherryMX
Connections:
- net labels added: ROT2_COL, ROT2_ROW
- wire segments 104 -> 122
Changed lines of the file:
@@
 Wire Wire Line
 	24550 14500 24550 13650
-Text GLabel 21750 12550 1    50   Input ~ 0
-COL0
+Text GLabel 21550 12650 0    50   Input ~ 0
+ROT2_COL
 Text GLabel 24450 12550 1    50   Input ~ 0
 COL17
@@
 $EndComp
 Wire Wire Line
-	21750 12550 21750 13050
-Wire Wire Line
 	24450 12550 24450 13050
 Wire Wire Line
@@
 	24650 12650 24850 12650
 Text GLabel 22150 12650 2    50   Input ~ 0
-ROW0
+ROT2_ROW
 $Comp
 L Device:D_Small D?
@@
 Text Notes 1300 9300 0    118  ~ 24
 RGB LEDs
-Text GLabel 3200 2800 1    50   Input ~ 0
+Text GLabel 2800 2900 1    50   Input ~ 0
 COL3
-Text GLabel 3100 2800 1    50   Input ~ 0
+Text GLabel 2700 2900 1    50   Input ~ 0
 COL2
-Text GLabel 3000 2800 1    50   Input ~ 0
+Text GLabel 2600 2900 1    50   Input ~ 0
 COL1
-Text GLabel 2900 2800 1    50   Input ~ 0
+Text GLabel 1500 2900 1    50   Input ~ 0
 COL0
-Text GLabel 4100 2800 1    50   Input ~ 0
+Text GLabel 3700 2900 1    50   Input ~ 0
 COL12
-Text GLabel 4200 2800 1    50   Input ~ 0
+Text GLabel 3800 2900 1    50   Input ~ 0
 COL13
 Wire Notes Line
@@
 Text GLabel 24350 19950 2    50   Input ~ 0
 COL17
-Text GLabel 4300 2800 1    50   Input ~ 0
+Text GLabel 3900 2900 1    50   Input ~ 0
 COL14
-Text GLabel 4400 2800 1    50   Input ~ 0
+Text GLabel 4000 2900 1    50   Input ~ 0
 COL15
-Text GLabel 4500 2800 1    50   Input ~ 0
+Text GLabel 4100 2900 1    50   Input ~ 0
 COL16
-Text GLabel 4600 2800 1    50   Input ~ 0
+Text GLabel 4200 2900 1    50   Input ~ 0
 COL17
-Text GLabel 4000 2800 1    50   Input ~ 0
+Text GLabel 3600 2900 1    50   Input ~ 0
 COL11
-Text GLabel 3900 2800 1    50   Input ~ 0
+Text GLabel 3500 2900 1    50   Input ~ 0
 COL10
-Text GLabel 3800 2800 1    50   Input ~ 0
+Text GLabel 3400 2900 1    50   Input ~ 0
 COL9
-Text GLabel 3700 2800 1    50   Input ~ 0
+Text GLabel 3300 2900 1    50   Input ~ 0
 COL8
-Text GLabel 3600 2800 1    50   Input ~ 0
+Text GLabel 3200 2900 1    50   Input ~ 0
 COL7
-Text GLabel 3500 2800 1    50   Input ~ 0
+Text GLabel 3100 2900 1    50   Input ~ 0
 COL6
-Text GLabel 3400 2800 1    50   Input ~ 0
+Text GLabel 3000 2900 1    50   Input ~ 0
 COL5
-Text GLabel 3300 2800 1    50   Input ~ 0
+Text GLabel 2900 2900 1    50   Input ~ 0
 COL4
-$Comp
-L MX_Alps_Hybrid:MX-NoLED MX?
-U 1 1 619A7102
-P 2700 3450
-F 0 "MX?" H 2733 3673 60  0000 C CNN
-F 1 "MX-NoLED" H 2733 3599 20  0000 C CNN
-F 2 "" H 2075 3425 60  0001 C CNN
-F 3 "" H 2075 3425 60  0001 C CNN
-	1    2700 3450
-	1    0    0    -1
-$EndComp
-Text GLabel 1300 3300 0    50   Input ~ 0
+Text GLabel 1300 4050 0    50   Input ~ 0
 ROW0
-Text GLabel 1300 3400 0    50   Input ~ 0
+Text GLabel 1300 4850 0    50   Input ~ 0
 ROW1
-Text GLabel 1300 3500 0    50   Input ~ 0
+Text GLabel 1300 5650 0    50   Input ~ 0
 ROW2
-Text GLabel 1300 3600 0    50   Input ~ 0
+Text GLabel 1300 6450 0    50   Input ~ 0
 ROW3
-Text GLabel 1300 3800 0    50   Input ~ 0
+Text GLabel 1300 8050 0    50   Input ~ 0
 ROW5
-Text GLabel 1300 3700 0    50   Input ~ 0
+Text GLabel 1300 7250 0    50   Input ~ 0
 ROW4
+Wire Wire Line
+	2600 5750 2600 2900
+Wire Wire Line
+	3900 4850 1300 4850
+$Comp
+L Device:D_Small D?
+U 1 1 61A82009
+P 2100 4650
+F 0 "D?" V 2146 4580 50  0000 R CNN
+F 1 "SOD-123" V 2055 4580 50  0000 R CNN
+F 2 "" V 2100 4650 50  0001 C CNN
+F 3 "~" V 2100 4650 50  0001 C CNN
+	1    2100 4650
+	0    -1   -1   0
+$EndComp
+$Comp
+L CherryMX:CherryMX SW?
+U 1 1 61A8200F
+P 1800 4450
+F 0 "SW?" H 1800 4735 50  0000 C CNN
+F 1 "CherryMX" H 1800 4644 50  0000 C CNN
+F 2 "" H 1800 4475 50  0001 C CNN
+F 3 "" H 1800 4475 50  0001 C CNN
+	1    1800 4450
+	1    0    0    -1
+$EndComp
+Wire Wire Line
+	1500 4450 1600 4450
+Wire Wire Line
+	2100 4750 2100 4850
+Wire Wire Line
+	2100 4550 2100 4450
+Wire Wire Line
+	2100 4450 2000 4450
+$Comp
+L Device:D_Small D?
+U 1 1 61A87861
+P 3200 3850
+F 0 "D?" V 3246 3780 50  0000 R CNN
+F 1 "SOD-123" V 3155 3780 50  0000 R CNN
+F 2 "" V 3200 3850 50  0001 C CNN
+F 3 "~" V 3200 3850 50  0001 C CNN
+	1    3200 3850
+	0    -1   -1   0
+$EndComp
+$Comp
+L CherryMX:CherryMX SW?
+U 1 1 61A87867
+P 2900 3650
+F 0 "SW?" H 2900 3935 50  0000 C CNN
+F 1 "CherryMX" H 2900 3844 50  0000 C CNN
+F 2 "" H 2900 3675 50  0001 C CNN
+F 3 "" H 2900 3675 50  0001 C CNN
+	1    2900 3650
+	1    0    0    -1
+$EndComp
+Wire Wire Line
+	2600 3650 2700 3650
+Wire Wire Line
+	3200 3950 3200 4050
+Wire Wire Line
+	3200 3750 3200 3650
+Wire Wire Line
+	3200 3650 3100 3650
+Wire Wire Line
+	1500 2900 1500 3600
+Wire Wire Line
+	1300 4050 2100 4050
+Wire Wire Line
+	21750 13050 21750 12650
+Wire Wire Line
+	21750 12650 21550 12650
+Text GLabel 1600 3600 2    50   Input ~ 0
+ROT2_COL
+Text GLabel 2100 3850 1    50   Input ~ 0
+ROT2_ROW
+Wire Wire Line
+	1500 3600 1600 3600
+Wire Wire Line
+	1500 4300 1500 4450
+Wire Wire Line
+	2100 3850 2100 4050
+Connection ~ 2100 4050
+Wire Wire Line
+	2100 4050 3900 4050
+Connection ~ 1500 4450
+Wire Wire Line
+	1500 4450 1500 6450
 $EndSCHEMATC

Commit message: Keyboard matrix
Parts:
- removed D?: SOD-123, symbol Device:D_Small
- removed SW?: CherryMX, symbol CherryMX:CherryMX
- added D? (x91): SOD-123, symbol Device:D_Small
- added SW?: M5, symbol CherryMX:CherryMX
- added SW?: M2, symbol CherryMX:CherryMX
- added SW?: M3, symbol CherryMX:CherryMX
- added SW?: M4, symbol CherryMX:CherryMX
- added SW? (x2): CherryMX, symbol CherryMX:CherryMX
- added SW?: RIGHT, symbol CherryMX:CherryMX
- added SW?: LCTRL, symbol CherryMX:CherryMX
- added SW?: LGUI, symbol CherryMX:CherryMX
- added SW?: LALT, symbol CherryMX:CherryMX
- added SW?: SPACE, symbol CherryMX:CherryMX
- added SW?: RALT, symbol CherryMX:CherryMX
- added SW?: RGUI, symbol CherryMX:CherryMX
- added SW?: MENU, symbol CherryMX:CherryMX
- added SW?: RCTRL, symbol CherryMX:CherryMX
- added SW?: LEFT, symbol CherryMX:CherryMX
- added SW?: DOWN, symbol CherryMX:CherryMX
- added SW?: ESC, symbol CherryMX:CherryMX
- added SW?: `/~, symbol CherryMX:CherryMX
- added SW?: TAB, symbol CherryMX:CherryMX
- added SW?: CAPS, symbol CherryMX:CherryMX
- added SW?: LSHIFT, symbol CherryMX:CherryMX
- added SW?: 1, symbol CherryMX:CherryMX
- added SW?: Q, symbol CherryMX:CherryMX
- added SW?: A, symbol CherryMX:CherryMX
- added SW?: Z, symbol CherryMX:CherryMX
- added SW?: F1, symbol CherryMX:CherryMX
- added SW?: 2, symbol CherryMX:CherryMX
- added SW?: W, symbol CherryMX:CherryMX
- added SW?: S, symbol CherryMX:CherryMX
- added SW?: X, symbol CherryMX:CherryMX
- added SW?: F2, symbol CherryMX:CherryMX
- added SW?: 3, symbol CherryMX:CherryMX
- added SW?: E, symbol CherryMX:CherryMX
- added SW?: D, symbol CherryMX:CherryMX
- added SW?: C, symbol CherryMX:CherryMX
- added SW?: F3, symbol CherryMX:CherryMX
- added SW?: 4, symbol CherryMX:CherryMX
- added SW?: R, symbol CherryMX:CherryMX
- added SW?: F, symbol CherryMX:CherryMX
- added SW?: V, symbol CherryMX:CherryMX
- added SW?: B, symbol CherryMX:CherryMX
- added SW?: G, symbol CherryMX:CherryMX
- added SW?: T, symbol CherryMX:CherryMX
- added SW?: 5, symbol CherryMX:CherryMX
- added SW?: F4, symbol CherryMX:CherryMX
- added SW?: N, symbol CherryMX:CherryMX
- added SW?: M, symbol CherryMX:CherryMX
- added SW?: ,/<, symbol CherryMX:CherryMX
- added SW?: F5, symbol CherryMX:CherryMX
- added SW?: 6, symbol CherryMX:CherryMX
- added SW?: Y, symbol CherryMX:CherryMX
- added SW?: H, symbol CherryMX:CherryMX
- added SW?: J, symbol CherryMX:CherryMX
- added SW?: U, symbol CherryMX:CherryMX
- added SW?: 7, symbol CherryMX:CherryMX
- added SW?: F6, symbol CherryMX:CherryMX
- added SW?: F7, symbol CherryMX:CherryMX
- added SW?: 8, symbol CherryMX:CherryMX
- added SW?: I, symbol CherryMX:CherryMX
- added SW?: K, symbol CherryMX:CherryMX
- added SW?: F8, symbol CherryMX:CherryMX
- added SW?: 9, symbol CherryMX:CherryMX
- added SW?: O, symbol CherryMX:CherryMX
- added SW?: L, symbol CherryMX:CherryMX
- added SW?: ./>, symbol CherryMX:CherryMX
- added SW?: F9, symbol CherryMX:CherryMX
- added SW?: F10, symbol CherryMX:CherryMX
- added SW?: F11, symbol CherryMX:CherryMX
- added SW?: F12, symbol CherryMX:CherryMX
- added SW?: PSCR, symbol CherryMX:CherryMX
- added SW?: 0, symbol CherryMX:CherryMX
- added SW?: -/_, symbol CherryMX:CherryMX
- added SW?: =/+, symbol CherryMX:CherryMX
- added SW?: BACKSPACE, symbol CherryMX:CherryMX
- added SW?: INS, symbol CherryMX:CherryMX
- added SW?: HOME, symbol CherryMX:CherryMX
- added SW?: PGUP, symbol CherryMX:CherryMX
- added SW?: P, symbol CherryMX:CherryMX
- added SW?: [/{, symbol CherryMX:CherryMX
- added SW?: ]/}, symbol CherryMX:CherryMX
- added SW?: \\, symbol CherryMX:CherryMX
- added SW?: DELETE, symbol CherryMX:CherryMX
- added SW?: END, symbol CherryMX:CherryMX
- added SW?: PGDN, symbol CherryMX:CherryMX
- added SW?: ;/:, symbol CherryMX:CherryMX
- added SW?: '/\", symbol CherryMX:CherryMX
- added SW?: ENTER, symbol CherryMX:CherryMX
- added SW?: RSHIFT, symbol CherryMX:CherryMX
- added SW?: /, symbol CherryMX:CherryMX
- added SW?: UP, symbol CherryMX:CherryMX
- SW?: value CherryMX -> M1
Connections:
- net labels added: ROT1_COL, ROT1_ROW
- wire segments 122 -> 485
Other:
- note added: "0"
- note added: "1"
- note added: "10"
- note added: "11"
- note added: "12"
- note added: "13"
- note added: "14"
- note added: "15"
- note added: "16"
- note added: "17"
- note added: "2"
- note added: "3"
- note added: "4"
- note added: "5"
- note added: "6"
- note added: "7"
- note added: "8"
- note added: "9"
