File: PCB/custom_keyboard.sch (KiCad schematic (older format))
At the start: 409 parts, among them J1 Conn_01x08_Male, SW1 M1, SW10 LSHIFT, SW11 LCTRL, SW12 1, SW13 Q, SW14 A, SW15 Z, SW16 LGUI, SW17 F1, SW18 2, SW19 W, SW2 M2, SW20 S, SW21 X, SW22 LALT, SW23 F2, SW24 3, SW25 E, SW26 D, SW27 C, SW28 F3, SW29 4, SW3 M3, SW30 R, SW31 F, SW32 V, SW33 F4, SW34 5, SW35 T, SW36 G, SW37 B, SW38 SPACE, SW39 F5, SW4 M4, SW40 6, SW41 Y, SW42 H, SW43 N, SW44 F6, SW45 7, SW46 U, SW47 J, SW48 M, SW49 F7, SW5 M5, SW50 8, SW51 I, SW52 K, SW53 ,/<, SW54 F8, SW55 9, SW56 O, SW57 L, SW58 ./>, SW59 RALT, SW6 ESC, SW60 F9, SW61 0, SW62 P, SW63 ;/:, SW64 /, SW65 RGUI, SW66 F10, SW67 -/_, SW68 [/{, SW69 '/\", SW7 `/~, SW70 CherryMX, SW71 F11, SW72 =/+, SW73 ]/}, SW74 MENU, SW75 F12, SW76 BACKSPACE, SW77 \\, SW78 ENTER, SW79 RSHIFT, SW8 TAB, SW80 RCTRL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

Commit message: USB hub connections
Parts:
- removed R?: 5.1K, symbol Device:R_Small
- added C101, C102, C103: 0.1uF, symbol Device:C_Small
- added C104, C105, C106: 100uF, symbol Device:C_Small
- added C107, C116: 10uF, symbol Device:C_Small
- added C108: 4.7uF, symbol Device:C_Small
- added C109: 100nF, symbol Device:C_Small
- added D185: Red, symbol Device:LED_Small
- added D186, D187, D188, D189, D190, D191, D192: Green/Amber, symbol Device:LED_Dual_2pin
- added J3, J4: USB_A, symbol Connector:USB_A
- added R11, R12, R13, R14, R15, R16, R17, R18, R19, R20, R21: 330, symbol Device:R_Small
- added R22, R23, R24, R25, R26, R27, R42, R43, R44, R45, R46, R47: 22, symbol Device:R_Small
- added R30, R31: 100k, symbol Device:R_Small
- added R32: 47k, symbol Device:R_Small
- added R34, R36, R37, R38, R39, R40, R41: 5.1K, symbol Device:R_Small
- added R35: 2.7k, symbol Device:R_Small
- added TP2, TP3, TP4: VCC, symbol Connector:TestPoint
- added U3, U4, U5, U7, U8, U9: PRTR5V0U2X, symbol random-keyboard-parts:PRTR5V0U2X
- added USB2, USB3, USB4: HRO-TYPE-C-31-M-12, symbol Type-C:HRO-TYPE-C-31-M-12
- D181: renamed from D186; value LED_Small -> Yellow
- gave numbers to parts that had none: 12
- renumbered C11 to C10, C102 to C100, C12 to C11, C103 to C110, C104 to C111, C105 to C112, C106 to C113, C13 to C12, C14 to C13, C15 to C14, C16 to C15, C17 to C16, C18 to C17, C19 to C18, C21 to C19, C22 to C20, C23 to C21, C24 to C22, C25 to C23, C26 to C24, C27 to C25, C28 to C26, C29 to C27, C30 to C28, C31 to C29, C32 to C30, C33 to C31, C34 to C32, C35 to C33, C36 to C34, C37 to C35, C38 to C36, C39 to C37, C40 to C38, C41 to C39, C42 to C40, C43 to C41, C44 to C42, C45 to C43, C46 to C44, C47 to C45, C48 to C46, C49 to C47, C50 to C48, C51 to C49, C52 to C50, C53 to C51, C54 to C52, C55 to C53, C56 to C54, C57 to C55, C58 to C56, C59 to C57, C60 to C58, C61 to C59, C62 to C60, C63 to C61, C64 to C62, C65 to C63, C66 to C64, C67 to C65, C68 to C66, C69 to C67, C70 to C68, C71 to C69, C72 to C70, C73 to C71, C74 to C72, C75 to C73, C76 to C74, C77 to C75, C78 to C76, C79 to C77, C80 to C78, C81 to C79, C82 to C80, C83 to C81, C84 to C82, C85 to C83, C86 to C84, C87 to C85, C88 to C86, C89 to C87, C90 to C88, C91 to C89, C92 to C90, C93 to C91, C94 to C92, C95 to C93, C96 to C94, C97 to C95, C98 to C96, C99 to C97, C100 to C98, C101 to C99, D11 to D1, D9 to D10, D93 to D100, D94 to D101, D109 to D102, D110 to D103, D111 to D104, D112 to D105, D113 to D106, D114 to D107, D115 to D108, D116 to D109, D10 to D11, D117 to D110, D104 to D111, D105 to D112, D106 to D113, D107 to D114, D108 to D115, D123 to D116, D124 to D117, D125 to D118, D126 to D119, D16 to D12, D127 to D120, D128 to D121, D129 to D122, D130 to D123, D131 to D124, D118 to D125, D119 to D126, D120 to D127, D121 to D128, D122 to D129, D17 to D13, D137 to D130, D138 to D131, D139 to D132, D140 to D133, D141 to D134, D142 to D135, D143 to D136, D144 to D137, D145 to D138, D132 to D139, D2 to D14, D133 to D140, D134 to D141, D135 to D142, D136 to D143, D146 to D144, D147 to D145, D148 to D146, D149 to D147, D150 to D148, D151 to D149, D18 to D15, D152 to D150, D153 to D151, D154 to D152, D155 to D153, D156 to D154, D157 to D155, D167 to D156, D158 to D157, D159 to D158, D160 to D159, D19 to D16, D161 to D160, D162 to D161, D163 to D162, D164 to D163, D165 to D164, D166 to D165, D168 to D166, D169 to D167, D170 to D168, D171 to D169, D20 to D17, D172 to D170, D173 to D171, D178 to D172, D174 to D173, D175 to D174, D176 to D175, D177 to D176, D179 to D177, D180 to D178, D181 to D179, D21 to D18, D182 to D180, D183 to D182, D184 to D183, D185 to D184, D22 to D19, D12 to D2, D23 to D20, D24 to D21, D37 to D22, D3 to D23, D26 to D24, D27 to D25, D28 to D26, D29 to D27, D30 to D28, D31 to D29, D13 to D3, D38 to D30, D39 to D31, D40 to D32, D41 to D33, D42 to D34, D43 to D35, D44 to D36, D45 to D37, D4 to D38, D32 to D39, D14 to D4, D33 to D40, D34 to D41, D35 to D42, D36 to D43, D52 to D44, D53 to D45, D54 to D46, D55 to D47, D56 to D48, D57 to D49, D15 to D5, D58 to D50, D59 to D51, D60 to D52, D46 to D53, D47 to D54, D48 to D55, D49 to D56, D50 to D57, D51 to D58, D66 to D59, D5 to D6, D67 to D60, D68 to D61, D69 to D62, D70 to D63, D71 to D64, D72 to D65, D73 to D66, D74 to D67, D61 to D68, D62 to D69, D6 to D7, D63 to D70, D64 to D71, D65 to D72, D80 to D73, D81 to D74, D82 to D75, D83 to D76, D84 to D77, D85 to D78, D86 to D79, D7 to D8, D87 to D80, D88 to D81, D75 to D82, D76 to D83, D77 to D84, D78 to D85, D79 to D86, D95 to D87, D96 to D88, D97 to D89, D8 to D9, D98 to D90, D99 to D91, D100 to D92, D101 to D93, D102 to D94, D103 to D95, D89 to D96, D90 to D97, D91 to D98, D92 to D99, ROT2 to ROT1, ROT1 to ROT2
Connections:
- net +1V8: now also IC1.21 (VD_PLL), IC1.25 (VD18_0), IC1.28 (VD18), IC1.6 (VD18), C116.1
- net +3V3: now also IC1.15 (VD33), IC1.20 (VD33), IC1.26 (VD33), IC1.31 (VD33), IC1.36 (VD33), IC1.42 (VD33), IC1.43 (OVCJ5), IC1.45 (OVCJ1), IC1.9 (VD33_O), U2.7 (WP), U2.8 (VCC), C107.1, R31.2
- net +5V: now also IC1.8 (VDD5), J2.1 (VBUS), C104.1, C105.1, C106.1, C108.2, C109.2, J3.1 (VBUS), J4.1 (VBUS), R32.1, TP2.1, TP3.1, TP4.1, U3.4 (VCC), U4.4 (VCC), U5.4 (VCC), U7.4 (VCC), U8.4 (VCC), U9.4 (VCC), USB2.11 (VBUS), USB2.2 (VBUS), USB3.11 (VBUS), USB3.2 (VBUS), USB4.11 (VBUS), USB4.2 (VBUS)
- net GND: now also IC1.10 (VSS), IC1.24 (VS_PLL), IC1.39 (VSS), J2.4 (GND), R33.2, C101.2, C102.2, C103.2, C104.2, C105.2, C106.2, C107.2, C116.2, J3.4 (GND), J4.4 (GND), R11.2, R12.2, R13.2, R21.1, R34.2, R35.1, R36.2, R37.2, R38.2, R39.2, R40.2, R41.2, U3.1 (GND), U4.1 (GND), U5.1 (GND), U7.1 (GND), U8.1 (GND), U9.1 (GND), USB2.1 (GND), USB2.12 (GND), USB2.13 (SHIELD), USB3.1 (GND), USB3.12 (GND), USB3.13 (SHIELD), USB4.1 (GND), USB4.12 (GND), USB4.13 (SHIELD); no longer R33.1
- net HUB_LED1: now also R14.2
- net HUB_LED2: now also R15.2
- net HUB_LED3: now also R16.2
- net HUB_LED4: now also R17.2
- net HUB_LED5: now also R18.2
- net HUB_LED6: now also R19.2
- net HUB_LED7: now also R20.2
- net HUB_PORT2_D+: now also R22.2
- net HUB_PORT2_D-: now also R23.2
- net HUB_PORT3_D+: now also R24.2
- net HUB_PORT3_D-: now also R25.2
- net HUB_PORT4_D+: now also R26.2
- net HUB_PORT4_D-: now also R27.2
- net HUB_PORT5_D+: now also R46.2
- net HUB_PORT5_D-: now also R47.2
- net HUB_PORT6_D+: now also R44.2
- net HUB_PORT6_D-: now also R45.2
- net HUB_PORT7_D+: now also R42.2
- net HUB_PORT7_D-: now also R43.2
- net HUB_DRV: now reaches IC1.1 (DRV)
- net HUB_DRV: now also D185.2 (A), D186.1 (KA), D187.1 (KA), D188.1 (KA), D189.1 (KA), D190.1 (KA), D191.1 (KA), D192.1 (KA)
- net at IC1.27 (REXT): now also R35.2
- net at IC1.40 (XRSTJ): now also R31.1
- net at IC1.41 (VBUSM): now also R30.1, R32.2
- net at J2.2 (D-): now also R23.1, U3.3 (IO2)
- net at J2.3 (D+): now also R22.1, U3.2 (IO1)
- net at J2.5 (Shield): now also C101.1, R11.1
- net CC1: no longer names the net of USB1.4 (CC1)
- net CC1: now also R34.1; no longer R33.2
- net CC2: no longer names the net of USB1.10 (CC2)
- net CC2: now also R33.1
- new net: D185.1 (K), R21.2
- new net: D186.2 (AK), R14.1
- new net: D187.2 (AK), R15.1
- new net: D188.2 (AK), R16.1
- new net: D189.2 (AK), R17.1
- new net: D190.2 (AK), R18.1
- new net: D191.2 (AK), R19.1
- new net: D192.2 (AK), R20.1
- new net: C108.1, C109.1, R30.2
- new net: J3.2 (D-), R25.1, U4.3 (IO2)
- new net: J3.3 (D+), R24.1, U4.2 (IO1)
- new net: C102.1, J3.5 (Shield), R12.1
- new net: J4.2 (D-), R27.1, U5.3 (IO2)
- new net: J4.3 (D+), R26.1, U5.2 (IO1)
- new net: C103.1, J4.5 (Shield), R13.1
- new net: R41.1, USB4.10 (CC2)
- new net: R38.1, USB4.4 (CC1)
- new net: R47.1, U9.3 (IO2), USB4.5 (DN2), USB4.7 (DN1)
- new net: R46.1, U9.2 (IO1), USB4.6 (DP1), USB4.8 (DP2)
- new net: R40.1, USB3.10 (CC2)
- new net: R37.1, USB3.4 (CC1)
- new net: R45.1, U8.3 (IO2), USB3.5 (DN2), USB3.7 (DN1)
- new net: R44.1, U8.2 (IO1), USB3.6 (DP1), USB3.8 (DP2)
- new net: R39.1, USB2.10 (CC2)
- new net: R36.1, USB2.4 (CC1)
- new net: R43.1, U7.3 (IO2), USB2.5 (DN2), USB2.7 (DN1)
- new net: R42.1, U7.2 (IO1), USB2.6 (DP1), USB2.8 (DP2)
- no-connect marks 16 -> 23
Other:
- moved on the sheet: C110, C111, C112, C113, C114, C115, IC1, J2, R28, R29, R33, TP1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

Commit message: Reannotated components
Parts:
- removed D161: SOD-123, symbol Device:D_Small
- removed R37, R38: 5.1K, symbol Device:R_Small
- removed R42, R45, R46, R47: 22, symbol Device:R_Small
- removed SW70: CherryMX, symbol CherryMX:CherryMX
- removed U9: PRTR5V0U2X, symbol random-keyboard-parts:PRTR5V0U2X
- added C1, C24, C49, C73: 0.1uF, symbol Device:C_Small
- added R1, R19, R31: 330, symbol Device:R_Small
- added R20, R24, R32: 5.1K, symbol Device:R_Small
- added R22, R23, R33, R35: 22, symbol Device:R_Small
- added U6: PRTR5V0U2X, symbol random-keyboard-parts:PRTR5V0U2X
- R39: value 5.1K -> 330
- R41: value 5.1K -> 22
- R44: value 22 -> 5.1K
- renumbered C102 to C10, C35 to C100, C44 to C101, C53 to C102, C62 to C103, C71 to C104, C80 to C105, C89 to C106, C9 to C107, C18 to C108, C27 to C109, C106 to C11, C36 to C110, C45 to C111, C54 to C112, C63 to C113, C72 to C114, C81 to C115, C90 to C116, C110 to C117, C111 to C118, C112 to C119, C1 to C12, C113 to C120, C10 to C13, C19 to C14, C28 to C15, C37 to C16, C46 to C17, C55 to C18, C64 to C19, C104 to C2, C73 to C20, C82 to C21, C103 to C22, C116 to C23, C2 to C25, C11 to C26, C20 to C27, C29 to C28, C38 to C29, C101 to C3, C47 to C30, C56 to C31, C65 to C32, C74 to C33, C83 to C34, C3 to C35, C12 to C36, C21 to C37, C30 to C38, C114 to C4, C48 to C40, C57 to C41, C66 to C42, C75 to C43, C84 to C44, C93 to C45, C94 to C46, C97 to C47, C98 to C48, C108 to C5, C99 to C50, C4 to C51, C13 to C52, C22 to C53, C31 to C54, C40 to C55, C49 to C56, C58 to C57, C67 to C58, C76 to C59, C109 to C6, C85 to C60, C100 to C61, C5 to C62, C14 to C63, C23 to C64, C32 to C65, C41 to C66, C50 to C67, C59 to C68, C68 to C69, C115 to C7, C77 to C70, C86 to C71, C95 to C72, C96 to C74, C6 to C75, C15 to C76, C24 to C77, C33 to C78, C42 to C79, C105 to C8, C51 to C80, C60 to C81, C69 to C82, C78 to C83, C87 to C84, C91 to C85, C7 to C86, C16 to C87, C25 to C88, C34 to C89, C107 to C9, C43 to C90, C52 to C91, C61 to C92, C70 to C93, C79 to C94, C88 to C95, C92 to C96, C8 to C97, C17 to C98, C26 to C99, D24 to D1, D150 to D10, D130 to D100, D7 to D101, D16 to D102, D31 to D103, D45 to D104, D60 to D105, D74 to D106, D88 to D107, D103 to D108, D117 to D109, D157 to D11, D131 to D110, D156 to D111, D172 to D112, D186 to D113, D8 to D114, D17 to D115, D32 to D116, D46 to D117, D61 to D118, D75 to D119, D162 to D12, D89 to D120, D104 to D121, D118 to D122, D132 to D123, D187 to D124, D188 to D125, D9 to D126, D18 to D127, D33 to D128, D47 to D129, D166 to D13, D62 to D130, D76 to D131, D90 to D132, D105 to D133, D119 to D134, D133 to D135, D189 to D136, D190 to D137, D10 to D138, D19 to D139, D173 to D14, D34 to D140, D48 to D141, D63 to D142, D77 to D143, D91 to D144, D106 to D145, D120 to D146, D134 to D147, D191 to D148, D11 to D149, D1 to D15, D20 to D150, D35 to D151, D49 to D152, D64 to D153, D78 to D154, D92 to D155, D107 to D156, D121 to D157, D135 to D158, D192 to D159, D25 to D16, D185 to D160, D181 to D161, D12 to D162, D21 to D163, D36 to D164, D50 to D165, D65 to D166, D79 to D167, D93 to D168, D108 to D169, D39 to D17, D122 to D170, D136 to D171, D13 to D172, D22 to D173, D37 to D174, D51 to D175, D66 to D176, D80 to D177, D94 to D178, D109 to D179, D54 to D18, D123 to D180, D137 to D181, D14 to D182, D23 to D183, D38 to D184, D52 to D185, D67 to D186, D81 to D187, D95 to D188, D110 to D189, D69 to D19, D124 to D190, D138 to D191, D53 to D2, D83 to D20, D97 to D21, D112 to D22, D126 to D23, D140 to D24, D145 to D25, D151 to D26, D158 to D27, D163 to D28, D167 to D29, D68 to D3, D174 to D30, D177 to D31, D182 to D32, D2 to D33, D26 to D34, D40 to D35, D55 to D36, D70 to D37, D84 to D38, D98 to D39, D82 to D4, D113 to D40, D127 to D41, D141 to D42, D146 to D43, D152 to D44, D159 to D45, D164 to D46, D168 to D47, D175 to D48, D178 to D49, D96 to D5, D183 to D50, D3 to D51, D27 to D52, D41 to D53, D56 to D54, D71 to D55, D85 to D56, D99 to D57, D114 to D58, D128 to D59, D111 to D6, D142 to D60, D147 to D61, D153 to D62, D160 to D63, D169 to D64, D4 to D65, D28 to D66, D42 to D67, D57 to D68, D72 to D69, D125 to D7, D86 to D70, D100 to D71, D115 to D72, D129 to D73, D143 to D74, D148 to D75, D154 to D76, D170 to D77, D179 to D78, D5 to D79, D139 to D8, D29 to D80, D43 to D81, D58 to D82, D101 to D83, D149 to D84, D155 to D85, D165 to D86, D171 to D87, D176 to D88, D180 to D89, D144 to D9, D184 to D90, D6 to D91, D15 to D92, D30 to D93, D44 to D94, D59 to D95, D73 to D96, D87 to D97, D102 to D98, D116 to D99, J2 to J1, J3 to J2, J4 to J3, J1 to J4, R30 to R10, R31 to R11, R24 to R12, R25 to R13, R12 to R14, R35 to R15, R26 to R16, R27 to R17, R13 to R18, R33 to R2, R9 to R21, R14 to R25, R2 to R26, R4 to R27, R7 to R28, R8 to R29, R28 to R3, R15 to R30, R16 to R34, R17 to R37, R18 to R38, R29 to R4, R19 to R42, R20 to R45, R5 to R46, R3 to R47, R10 to R48, R21 to R49, R34 to R5, R6 to R50, R1 to R51, R22 to R6, R23 to R7, R11 to R8, R32 to R9, SW6 to SW1, SW60 to SW10, SW66 to SW11, SW71 to SW12, SW75 to SW13, SW81 to SW14, SW1 to SW15, SW7 to SW16, SW12 to SW17, SW24 to SW19, SW17 to SW2, SW29 to SW20, SW34 to SW21, SW40 to SW22, SW45 to SW23, SW50 to SW24, SW55 to SW25, SW61 to SW26, SW67 to SW27, SW72 to SW28, SW76 to SW29, SW23 to SW3, SW82 to SW30, SW85 to SW31, SW89 to SW32, SW2 to SW33, SW8 to SW34, SW13 to SW35, SW19 to SW36, SW25 to SW37, SW30 to SW38, SW35 to SW39, SW28 to SW4, SW41 to SW40, SW46 to SW41, SW51 to SW42, SW56 to SW43, SW62 to SW44, SW68 to SW45, SW73 to SW46, SW77 to SW47, SW83 to SW48, SW86 to SW49, SW33 to SW5, SW90 to SW50, SW3 to SW51, SW9 to SW52, SW14 to SW53, SW20 to SW54, SW26 to SW55, SW31 to SW56, SW36 to SW57, SW42 to SW58, SW47 to SW59, SW39 to SW6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
Connections:
- net +5V: now also U6.4 (VCC)
- net GND: now also R44.2, C1.2, C24.2, C49.2, C73.2, R1.2, R19.2, R20.2, R24.2, R31.2, R32.2, U6.1 (GND); no longer R41.2, USB1.13 (SHIELD), USB2.13 (SHIELD), USB3.13 (SHIELD), USB4.13 (SHIELD)
- net HUB_PORT5_D+: now also R22.2
- net HUB_PORT5_D-: now also R23.2
- net HUB_PORT6_D+: now also R33.2; no longer R44.2
- net HUB_PORT6_D-: now also R35.2
- net HUB_PORT7_D+: now also R41.2
- net at USB4.10 (CC2): now also R40.1; no longer R41.1
- net at USB4.4 (CC1): now also R44.1
- net at USB4.5 (DN2), USB4.7 (DN1): now also R43.1, U8.3 (IO2)
- net at USB4.6 (DP1), USB4.8 (DP2): now also R41.1, U8.2 (IO1)
- net at USB3.10 (CC2): now also R32.1; no longer R40.1
- net at USB3.4 (CC1): now also R36.1
- net at USB3.5 (DN2), USB3.7 (DN1): now also U7.3 (IO2), R35.1; no longer U8.3 (IO2)
- net at USB3.6 (DP1), USB3.8 (DP2): now also U7.2 (IO1), R33.1; no longer R44.1, U8.2 (IO1)
- net at USB2.10 (CC2): now also R20.1; no longer R39.1
- net at USB2.4 (CC1): now also R24.1; no longer R36.1
- net at USB2.5 (DN2), USB2.7 (DN1): now also R23.1, U6.3 (IO2); no longer R43.1, U7.3 (IO2)
- net at USB2.6 (DP1), USB2.8 (DP2): now also R22.1, U6.2 (IO1); no longer U7.2 (IO1)
- new net: C1.1, R1.1, USB1.13 (SHIELD)
- new net: C24.1, R19.1, USB2.13 (SHIELD)
- new net: C49.1, R31.1, USB3.13 (SHIELD)
- new net: C73.1, R39.1, USB4.13 (SHIELD)
Other:
- moved on the sheet: C10, C11, C2, C22, C3, C8, J1, J2, J3, R12, R13, R14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

Commit message: USB Hub sections
Other:
- note added: "USB A Outputs (2-4)"
- note added: "USB C Outputs (5-7)"
- note added: "USB Hub Controller\n"
- note added: "USB Hub EEPROM"
- note added: "USB Hub Indicators\n"
- note added: "USB In"
- moved on the sheet: C1, C10, C11, C117, C118, C119, C120, C2, C22, C23, C24, C3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

Commit message: Adjusted section outlines
Other:
- note added: "USB Input"
- note removed: "USB In"
- moved on the sheet: C1, C10, C11, C2, C22, C23, C24, C3, C4, C49, C5, C6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
