File: PCB/custom_keyboard - Copy.sch (KiCad schematic (older format))
At the start: 390 parts, among them IC1 FE2.1, J1 USB_A, J2 USB_A, J3 USB_A, J4 Conn_01x08_Male, SW1 SW_Push, U1 PRTR5V0U2X, U2 24LC02, U3 PRTR5V0U2X, U4 PRTR5V0U2X, U5 PRTR5V0U2X, U6 PRTR5V0U2X, U7 PRTR5V0U2X, U8 PRTR5V0U2X, U9 AT90USB646-MU, Y1 12MHz, Y2 16MHz

Commit message: Assigned footprints to alternate schematic
Parts:
- removed D40, D41, D42, D43, D44, D45, D46: Green/Amber, symbol Device:LED_Dual_2pin
- added D102, D104, D106, D108, D41, D43, D45: Amber, LED_SMD:LED_0402_1005Metric, symbol Device:LED_Small
- added D103, D105, D107, D40, D42, D44, D46: Green, LED_SMD:LED_0402_1005Metric, symbol Device:LED_Small
- D39: renamed from D?; footprint (none) -> LED_SMD:LED_0402_1005Metric
- D84: footprint (none) -> LED_SMD:LED_0402_1005Metric
- MX1, MX12, MX13, MX14, MX15, MX17, MX18, MX19, MX2, MX20, MX21, MX23, MX24, MX25, MX26, MX27, MX28, MX29, MX3, MX30, MX31, MX32, MX33, MX34, MX35, MX36, MX37, MX39, MX4, MX40, MX41, MX42, MX43, MX44, MX45, MX46, MX47, MX48, MX49, MX5, MX50, MX51, MX52, MX53, MX54, MX55, MX56, MX57, MX58, MX6, MX60, MX61, MX62, MX63, MX64, MX66, MX67, MX68, MX69, MX7, MX70, MX71, MX72, MX74, MX80, MX81, MX82, MX83, MX84, MX85, MX86, MX87, MX88, MX89, MX90: footprint (none) -> CherryMX_PCB_KailhSocket_LTST-A683CEGBW:CherryMX_1.00u_PCB_KailhSocket_LTST-A683CEGBW
- MX10, MX77: footprint (none) -> CherryMX_PCB_KailhSocket_LTST-A683CEGBW:CherryMX_2.25u_PCB_KailhSocket_LTST-A683CEGBW
- MX11, MX16, MX22, MX59, MX65, MX73, MX79: footprint (none) -> CherryMX_PCB_KailhSocket_LTST-A683CEGBW:CherryMX_1.25u_PCB_KailhSocket_LTST-A683CEGBW
- MX38: footprint (none) -> CherryMX_PCB_KailhSocket_LTST-A683CEGBW:CherryMX_6.25u_PCB_KailhSocket_LTST-A683CEGBW
- MX75: footprint (none) -> CherryMX_PCB_KailhSocket_LTST-A683CEGBW:CherryMX_2.00u_PCB_KailhSocket_LTST-A683CEGBW
- MX76, MX8: footprint (none) -> CherryMX_PCB_KailhSocket_LTST-A683CEGBW:CherryMX_1.50u_PCB_KailhSocket_LTST-A683CEGBW
- MX78: footprint (none) -> CherryMX_PCB_KailhSocket_LTST-A683CEGBW:CherryMX_2.75u_PCB_KailhSocket_LTST-A683CEGBW
- MX9: footprint (none) -> CherryMX_PCB_KailhSocket_LTST-A683CEGBW:CherryMX_1.75u_PCB_KailhSocket_LTST-A683CEGBW
- R10, R13, R4, R5, R6, R7, R8, R9: renamed from R?; footprint (none) -> Resistor_SMD:R_0805_2012Metric
- R51: footprint (none) -> Resistor_SMD:R_0805_2012Metric
- SW1: footprint (none) -> Button_Switch_SMD:SW_SPST_SKQG_WithStem
- TP1, TP2, TP3, TP4: footprint (none) -> TestPoint:TestPoint_Pad_D1.0mm
- U1, U3, U4, U5, U6, U7, U8: footprint (none) -> random-keyboard-parts:SOT143B
- U2: footprint (none) -> Package_TO_SOT_SMD:SOT-23-8
- USB1, USB2, USB3, USB4: footprint (none) -> Type-C:HRO-TYPE-C-31-M-12
- Y1, Y2: footprint (none) -> Crystal:Crystal_SMD_3225-4Pin_3.2x2.5mm
Connections:
- wire segments 2305 -> 2361
Other:
- moved on the sheet: C1, C10, C100, C101, C102, C103, C104, C105, C106, C107, C108, C109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
