File: PCB/custom_keyboard.kicad_pcb (KiCad board)
At the start: 2 copper layers, 3.4 x 3 mm, 96 parts, among them SW1 SW_Push, U1 PRTR5V0U2X, U2 24LC02, U3 PRTR5V0U2X, U4 PRTR5V0U2X, U5 PRTR5V0U2X, U6 PRTR5V0U2X, U7 PRTR5V0U2X, U8 PRTR5V0U2X, U9 AT90USB646-MU, Y1 12MHz, Y2 16MHz

Commit message: Positioned key diodes
Parts:
- R1, R10, R11, R12, R13, R14, R15, R16, R17, R18, R19, R2, R20, R21, R22, R23, R24, R25, R26, R27, R28, R29, R3, R30, R31, R32, R33, R34, R35, R36, R37, R38, R39, R4, R40, R41, R42, R43, R44, R45, R46, R47, R48, R49, R5, R50, R51, R6, R7, R8, R9, SW1, TP1, TP2, TP3, TP4, U1, U2, U3, U4, U5, U6, U7, U8, U9, USB1, USB2, USB3, USB4, Y1, Y2: moved to B.Cu
- moved R33 546.0 mm to (413.6, -275.7)
- moved U8 541.1 mm to (419.1, -273.2)
- moved R18 540.2 mm to (414.9, -272.7)
- moved R31 534.2 mm to (419.3, -269.7)
- moved ROT2 530.5 mm to (527.0, -76.2), turned to 270 degrees
- moved R4 527.6 mm to (420.6, -266.4)
- moved R35 516.6 mm to (428.6, -260.8)
- moved R7 516.6 mm to (424.2, -260.8)
- moved R44 510.6 mm to (432.1, -257.8)
- moved R16 503.3 mm to (433.4, -254.1)
- moved U6 500.1 mm to (437.7, -252.4)
- moved R28 493.1 mm to (439.9, -248.9)
- moved R23 487.3 mm to (439.9, -246.0)
- moved R40 486.5 mm to (444.4, -245.6)
- moved R15 480.7 mm to (444.4, -242.6)
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Connections:
- U9 pad 33: COL12 -> COL13
- U9 pad 34: COL13 -> COL12

Commit message: Placed resistors and capacitators
Parts:
- moved R28 616.6 mm to (486.6, 365.9), turned to 180 degrees
- moved TP1 598.7 mm to (670.3, 313.3), turned to 180 degrees
- moved R33 594.9 mm to (496.1, 313.5), turned to 180 degrees
- moved R29 583.1 mm to (93.7, 225.4)
- moved R51 580.9 mm to (114.3, 242.1), turned to 180 degrees
- moved R21 573.6 mm to (100.8, 225.4)
- moved R40 568.4 mm to (492.9, 320.7), turned to 180 degrees
- moved U4 566.8 mm to (119.1, 221.5), turned to 180 degrees
- moved R32 566.6 mm to (99.2, 211.1), turned to 180 degrees
- moved R38 563.4 mm to (102.4, 204.8), turned to 180 degrees
- moved R26 560.7 mm to (117.5, 215.9), turned to 180 degrees
- moved R23 560.4 mm to (113.5, 209.6), turned to 180 degrees
- moved R37 559.8 mm to (102.4, 200.0), turned to 180 degrees
- moved R16 551.9 mm to (154.8, 222.2), turned to 180 degrees
- moved R3 551.2 mm to (131.8, 219.9), turned to 180 degrees
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- renumbered ROT2 to ROT1, ROT1 to ROT2
Connections:
- U7 pad 2: Net-(J2-Pad3) -> Net-(J2-Pad2)
- U7 pad 3: Net-(J2-Pad2) -> Net-(J2-Pad3)

Commit message: Halfway done USB ports
Parts:
- removed TP1, TP2, TP3, TP4: VCC, TestPoint:TestPoint_Pad_D1.0mm
- added IC1: FE2.1, custom-footprints:FE2.1, B.Cu at (125.7, 194.0)
- U2: footprint Package_TO_SOT_SMD:SOT-23-8 -> custom-footprints:24LC04
- moved U1 467.9 mm to (138.0, 226.2), turned to 270 degrees
- moved U4 47.2 mm to (72.0, 217.4)
- moved R26 44.2 mm to (76.9, 198.4)
- moved R23 38.2 mm to (75.3, 209.6)
- moved R4 31.6 mm to (165.9, 172.2)
- moved R5 31.6 mm to (172.1, 172.2)
- moved R7 31.5 mm to (185.6, 173.0)
- moved R6 30.2 mm to (177.8, 173.0)
- moved R9 26.8 mm to (200.7, 173.8)
- moved R37 26.1 mm to (80.0, 213.5)
- moved R8 25.7 mm to (191.2, 173.0)
- moved USB3 25.5 mm to (87.3, 201.1)
- moved R38 23.7 mm to (82.4, 217.5)
- moved U6 23.5 mm to (231.2, 223.9), turned to 0 degrees
- moved U8 23.4 mm to (436.8, 223.9), turned to 0 degrees
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Connections:
- U6 pad 2: Net-(J1-Pad3) -> HUB_PORT2_D-
- U6 pad 3: Net-(J1-Pad2) -> HUB_PORT2_D+
- U7 pad 2: Net-(J2-Pad2) -> HUB_PORT3_D-
- U7 pad 3: Net-(J2-Pad3) -> HUB_PORT3_D+
- U8 pad 2: Net-(J3-Pad3) -> HUB_PORT4_D-
- U8 pad 3: Net-(J3-Pad2) -> HUB_PORT4_D+
Routing:
- net +5V: track 0.00 -> 47.7 mm
- net Net-(C41-Pad1): track 0.00 -> 17.4 mm
- net Net-(R2-Pad1): track 0.00 -> 15.4 mm
- net Net-(C62-Pad1): track 0.00 -> 14.4 mm
- net Net-(C64-Pad1): track 0.00 -> 14.4 mm
- net Net-(C63-Pad1): track 0.00 -> 14.3 mm
- net Net-(R1-Pad1): track 0.00 -> 11.5 mm
- net Net-(R16-Pad1): track 0.00 -> 3.72 mm
- net Net-(R14-Pad1): track 0.00 -> 3.21 mm
- net HUB_PORT4_D-: track 0.00 -> 3.15 mm, vias 0 -> 1
- net HUB_PORT2_D-: track 0.00 -> 3.15 mm, vias 0 -> 1
- net HUB_PORT3_D-: track 0.00 -> 3.11 mm, vias 0 -> 1
- net HUB_PORT4_D+: track 0.00 -> 3.10 mm, vias 0 -> 1
- net HUB_PORT3_D+: track 0.00 -> 3.06 mm, vias 0 -> 1
- net HUB_PORT2_D+: track 0.00 -> 2.98 mm, vias 0 -> 1
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
Commit message: Routed lights
Parts:
- added C117: 0.1uF, Capacitor_SMD:C_0805_2012Metric, B.Cu at (535.8, 300.0)
- added C118: 0.1uF, Capacitor_SMD:C_0805_2012Metric, B.Cu at (535.8, 297.0)
- added C119: 0.1uF, Capacitor_SMD:C_0805_2012Metric, B.Cu at (540.2, 300.0)
- added C120: 10uF, Capacitor_SMD:C_0805_2012Metric, B.Cu at (540.2, 297.0)
- added D84: Yellow, LED_SMD:LED_0402_1005Metric, B.Cu at (418.0, 294.5)
- moved R50 134.5 mm to (416.8, 296.1)
- moved R49 109.7 mm to (453.2, 292.8), turned to 270 degrees
- moved U9 106.6 mm to (413.0, 302.6)
- moved Y2 105.5 mm to (424.7, 301.6), turned to 180 degrees
- moved R34 105.4 mm to (412.0, 310.5)
- moved SW1 99.9 mm to (454.8, 299.2), turned to 270 degrees
- moved U5 48.8 mm to (459.4, 311.8)
- moved R26 42.1 mm to (112.6, 220.7), turned to 0 degrees
- moved R39 40.2 mm to (460.4, 315.8), turned to 270 degrees
- moved R40 35.3 mm to (458.0, 315.8), turned to 270 degrees
- moved U4 34.1 mm to (105.4, 224.4), turned to 270 degrees
- moved R23 31.5 mm to (104.8, 220.7)
- moved R37 31.1 mm to (109.7, 223.0), turned to 0 degrees
- moved R33 29.9 mm to (466.6, 308.8), turned to 0 degrees
- moved R24 28.5 mm to (462.8, 311.3), turned to 90 degrees
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Connections:
- MX70 pad 5: +5V -> Net-(MX70-Pad5)
- MX74 pad 4: +5V -> Net-(MX70-Pad5)
Routing:
- net DOUT3: track 0.00 -> 406.1 mm
- net DOUT2: track 0.00 -> 405.6 mm
- net DOUT5: track 0.00 -> 388.6 mm
- net ROT1_ROW: track 0.00 -> 381.9 mm
- net ROW1: track 0.00 -> 378.0 mm
- net DOUT1: track 0.00 -> 372.8 mm
- net DOUT4: track 0.00 -> 329.0 mm
- net Net-(MX38-Pad5): track 0.00 -> 66.9 mm
- net Net-(MX22-Pad5): track 0.00 -> 66.9 mm
- net Net-(MX78-Pad5): track 0.00 -> 59.7 mm
- net Net-(MX17-Pad4): track 0.00 -> 33.5 mm
- net Net-(MX75-Pad5): track 0.00 -> 33.5 mm
- net Net-(MX64-Pad5): track 0.00 -> 31.1 mm
- net Net-(MX10-Pad4): track 0.00 -> 31.1 mm
- net Net-(MX76-Pad5): track 0.00 -> 28.8 mm
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
Commit message: Rows routed
Parts:
- added MX46: U, CherryMX_PCB_KailhSocket_LTST-A683CEGBW:CherryMX_1.00u_PCB_KailhSocket_LTST-A683CEGBW, F.Cu at (264.3, 278.6)
- added MX9: CAPS, CherryMX_PCB_KailhSocket_LTST-A683CEGBW:CherryMX_1.75u_PCB_KailhSocket_LTST-A683CEGBW, F.Cu at (128.6, 297.7)
- moved R34 98.0 mm to (508.0, 291.2), turned to 90 degrees
- moved U9 93.9 mm to (506.9, 299.1), turned to 90 degrees
- moved R50 86.8 mm to (503.1, 305.6), turned to 0 degrees
- moved D84 84.9 mm to (502.0, 307.2), turned to 0 degrees
- moved Y2 70.7 mm to (495.3, 300.0), turned to 0 degrees
- moved R49 34.3 mm to (485.0, 305.7), turned to 90 degrees
- moved SW1 28.6 mm to (483.4, 299.2), turned to 90 degrees
Routing:
- net ROW2: track 0.00 -> 378.7 mm
- net ROW5: track 0.00 -> 371.1 mm
- net ROW4: track 0.00 -> 354.7 mm
- net ROW3: track 0.00 -> 295.1 mm
- net Net-(D1-Pad2): track 0.00 -> 4.62 mm
- net Net-(D7-Pad2): track 0.00 -> 4.56 mm
- net Net-(D6-Pad2): track 0.00 -> 4.56 mm
- net Net-(D23-Pad2): track 0.00 -> 4.56 mm
- net Net-(D12-Pad2): track 0.00 -> 4.49 mm
- net Net-(D89-Pad2): track 0.00 -> 4.29 mm
- net Net-(D88-Pad2): track 0.00 -> 4.23 mm
- net Net-(D79-Pad2): track 0.00 -> 4.23 mm
- net Net-(D72-Pad2): track 0.00 -> 4.23 mm
- net Net-(D60-Pad2): track 0.00 -> 4.23 mm
- net Net-(D55-Pad2): track 0.00 -> 4.23 mm
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