File: PCB/custom_keyboard.kicad_pcb (KiCad board)
At the start: 2 copper layers, 3.4 x 3 mm, 116 parts, among them IC1 FE2.1, SW1 SW_Push, U1 PRTR5V0U2X, U2 24LC02, U3 PRTR5V0U2X, U4 PRTR5V0U2X, U5 PRTR5V0U2X, U6 PRTR5V0U2X, U7 PRTR5V0U2X, U8 PRTR5V0U2X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

Commit message: Connected controller to columns
Parts:
- added C53: 20pF, Capacitor_SMD:C_0805_2012Metric, B.Cu at (218.3, 304.0)
- added D102: Amber, LED_SMD:LED_0402_1005Metric, B.Cu at (181.8, 195.3)
- added D103: Green, LED_SMD:LED_0402_1005Metric, B.Cu at (188.9, 196.8)
- added D104: Amber, LED_SMD:LED_0402_1005Metric, B.Cu at (188.9, 195.3)
- added D105: Green, LED_SMD:LED_0402_1005Metric, B.Cu at (196.1, 196.8)
- added D106: Amber, LED_SMD:LED_0402_1005Metric, B.Cu at (196.1, 195.3)
- added D39: Red, LED_SMD:LED_0402_1005Metric, B.Cu at (195.0, 315.1)
- added D40: Green, LED_SMD:LED_0402_1005Metric, B.Cu at (159.2, 196.8)
- added D41: Amber, LED_SMD:LED_0402_1005Metric, B.Cu at (159.2, 195.3)
- added D42: Green, LED_SMD:LED_0402_1005Metric, B.Cu at (167.2, 195.3)
- added D43: Amber, LED_SMD:LED_0402_1005Metric, B.Cu at (167.2, 196.8)
- added D44: Green, LED_SMD:LED_0402_1005Metric, B.Cu at (174.6, 196.8)
- added D45: Amber, LED_SMD:LED_0402_1005Metric, B.Cu at (174.6, 195.3)
- added D46: Green, LED_SMD:LED_0402_1005Metric, B.Cu at (181.8, 196.8)
- added MX3: M3, CherryMX_PCB_KailhSocket_LTST-A683CEGBW:CherryMX_1.00u_PCB_KailhSocket_LTST-A683CEGBW, F.Cu at (88.9, 269.9)
- added MX43: N, CherryMX_PCB_KailhSocket_LTST-A683CEGBW:CherryMX_1.00u_PCB_KailhSocket_LTST-A683CEGBW, F.Cu at (250.8, 288.9)
- moved C40 287.1 mm to (181.8, 312.1), turned to 270 degrees
- moved R15 284.6 mm to (185.1, 304.8), turned to 180 degrees
- moved R13 283.2 mm to (185.1, 307.2), turned to 180 degrees
- moved R11 282.1 mm to (185.1, 309.6), turned to 180 degrees
- moved C42 269.5 mm to (208.1, 315.1)
- moved R24 259.3 mm to (215.1, 307.2), turned to 270 degrees
- moved FB2 207.0 mm to (220.7, 190.8), turned to 270 degrees
- moved R12 164.8 mm to (203.9, 315.1)
- moved Y1 156.6 mm to (218.3, 307.2), turned to 0 degrees
- moved R4 146.6 mm to (198.6, 315.1), turned to 0 degrees
- moved U2 138.5 mm to (179.4, 307.2), turned to 90 degrees
- moved IC1 135.9 mm to (200.5, 307.4), turned to 90 degrees
- moved R17 133.6 mm to (211.1, 305.6)
- moved FB5 120.3 mm to (312.7, 191.6), turned to 90 degrees
- moved R34 120.2 mm to (388.1, 282.6), turned to 270 degrees
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Connections:
- FB1 pad 1: VCC -> Net-(FB1-Pad1)
- FB2 pad 1: +5V -> Net-(FB2-Pad1)
- FB3 pad 2: GND -> Net-(FB3-Pad2)
- FB4 pad 1: +5V -> Net-(FB4-Pad1)
- FB5 pad 2: GND -> Net-(FB5-Pad2)
- FB6 pad 1: +5V -> Net-(FB6-Pad1)
- FB7 pad 2: GND -> Net-(FB7-Pad2)
- U6 pad 2: HUB_PORT2_D- -> Net-(J1-Pad3)
- U6 pad 3: HUB_PORT2_D+ -> Net-(J1-Pad2)
- U6 pad 4: +5V -> Net-(FB2-Pad1)
- U7 pad 2: HUB_PORT3_D- -> Net-(J2-Pad3)
- U7 pad 3: HUB_PORT3_D+ -> Net-(J2-Pad2)
- U7 pad 4: +5V -> Net-(FB4-Pad1)
- U8 pad 2: HUB_PORT4_D- -> Net-(J3-Pad3)
- U8 pad 3: HUB_PORT4_D+ -> Net-(J3-Pad2)
- U8 pad 4: +5V -> Net-(FB6-Pad1)
- U9 pad 32: COL14 -> COL0
- U9 pad 33: COL13 -> COL1
- U9 pad 34: COL12 -> COL2
- U9 pad 35: COL11 -> COL3
- U9 pad 36: COL10 -> COL4
- U9 pad 37: COL9 -> COL5
- U9 pad 38: COL8 -> COL6
- U9 pad 40: COL6 -> COL8
- U9 pad 41: COL5 -> COL9
- U9 pad 42: COL4 -> COL10
- U9 pad 44: COL3 -> COL11
- U9 pad 45: COL2 -> COL12
- U9 pad 46: COL1 -> COL13
- U9 pad 47: COL0 -> COL14
- U9 pad 56: ROT1_ROW -> ROW5
- U9 pad 57: ROW1 -> ROW4
- U9 pad 58: ROW2 -> ROW3
- U9 pad 59: ROW3 -> ROW2
- U9 pad 60: ROW4 -> ROW1
- U9 pad 61: ROW5 -> ROT1_ROW
- USB1 pad 11: VCC -> Net-(FB1-Pad1)
- USB1 pad 2: VCC -> Net-(FB1-Pad1)
Routing:
- net COL0: track 103.1 -> 468.8 mm, vias 5 -> 6
- net COL1: track 118.7 -> 455.1 mm, vias 6 -> 7
- net COL2: track 100.3 -> 411.7 mm, vias 5 -> 6
- net COL3: track 124.6 -> 411.0 mm, vias 6 -> 7
- net COL4: track 101.8 -> 376.1 mm, vias 5 -> 6
- net COL5: track 98.6 -> 353.3 mm, vias 5 -> 6
- net COL7: track 102.5 -> 322.1 mm, vias 5 -> 6
- net COL6: track 121.1 -> 334.1 mm, vias 6 -> 7
- net COL8: track 102.5 -> 299.0 mm, vias 5 -> 6
- net COL9: track 102.5 -> 277.0 mm, vias 5 -> 6
- net COL10: track 124.6 -> 259.7 mm, vias 6 -> 7
- net COL12: track 81.0 -> 212.0 mm, vias 4 -> 5
- net COL11: track 129.0 -> 241.1 mm, vias 6 -> 7
- net COL13: track 118.2 -> 198.4 mm, vias 4 -> 5
- net COL14: track 127.5 -> 168.4 mm, vias 6 -> 7
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Other:
- board size 3.4 x 3 mm -> 385.8 x 128.6 mm

Commit message: LED routing
Parts:
- added C109: 0.1uF, Capacitor_SMD:C_0805_2012Metric, B.Cu at (414.5, 314.3)
- moved R28 104.3 mm to (397.7, 283.4), turned to 270 degrees
- moved R30 102.6 mm to (400.1, 283.4), turned to 270 degrees
- moved R10 0.92 mm to (193.7, 196.2), turned to 270 degrees
- moved R5 0.92 mm to (156.4, 196.2), turned to 270 degrees
- moved R6 0.92 mm to (164.3, 196.2), turned to 270 degrees
- moved R8 0.92 mm to (179.4, 196.2), turned to 270 degrees
- moved R9 0.92 mm to (186.5, 196.2), turned to 270 degrees
- moved R52 0.80 mm to (200.8, 196.2), turned to 270 degrees
- moved D44 0.79 mm to (173.8, 196.8)
- moved D45 0.79 mm to (173.8, 195.3)
- moved R7 0.17 mm to (171.4, 196.2), turned to 270 degrees
Connections:
- U9 pad 29: COL17 -> COL16
- U9 pad 30: COL16 -> COL17
- U9 pad 49: ENCODER_B1 -> ENCODER_A
- U9 pad 50: ENCODER_A -> ENCODER_B1
- U9 pad 59: ROW2 -> ROT1_ROW
- U9 pad 61: ROT1_ROW -> ROW2
Routing:
- net KEYBOARD_D+: track 0.00 -> 217.3 mm, vias 0 -> 2
- net KEYBOARD_D-: track 0.00 -> 216.8 mm, vias 0 -> 2
- net HUB_DRV: track 15.4 -> 205.7 mm, vias 1 -> 2
- net HUB_LED1: track 35.9 -> 157.8 mm, vias 1 -> 2
- net COL17: track 104.0 -> 170.2 mm
- net COL16: track 93.7 -> 138.3 mm
- net ENCODER_B2: track 0.00 -> 34.7 mm, vias 0 -> 2
- net ENCODER_A: track 0.00 -> 30.5 mm, vias 0 -> 2
- net ENCODER_B1: track 0.00 -> 27.4 mm, vias 0 -> 2
- net Net-(R30-Pad1): track 0.00 -> 26.9 mm, vias 0 -> 2
- net Net-(R28-Pad1): track 0.00 -> 26.8 mm, vias 0 -> 2
- net BKL_DATA_IN: track 0.00 -> 25.9 mm, vias 0 -> 2
- net ROW4: track 354.7 -> 379.0 mm
- net ROT1_ROW: track 382.0 -> 400.9 mm
- net ROW1: track 378.0 -> 393.5 mm
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
Commit message: Routed some of the USB lanes
Parts:
- added MX26: D, CherryMX_PCB_KailhSocket_LTST-A683CEGBW:CherryMX_1.00u_PCB_KailhSocket_LTST-A683CEGBW, F.Cu at (184.2, 269.9)
- added MX28: F3, CherryMX_PCB_KailhSocket_LTST-A683CEGBW:CherryMX_1.00u_PCB_KailhSocket_LTST-A683CEGBW, F.Cu at (188.9, 208.0)
- added MX29: 4, CherryMX_PCB_KailhSocket_LTST-A683CEGBW:CherryMX_1.00u_PCB_KailhSocket_LTST-A683CEGBW, F.Cu at (188.9, 231.8)
- added MX38: SPACE, CherryMX_PCB_KailhSocket_LTST-A683CEGBW:CherryMX_6.25u_PCB_KailhSocket_LTST-A683CEGBW, F.Cu at (240.8, 375.0)
- added R54: 20k, Resistor_SMD:R_0805_2012Metric, B.Cu at (442.2, 273.8)
- added R55: 20k, Resistor_SMD:R_0805_2012Metric, B.Cu at (442.2, 271.5)
- moved R20 207.2 mm to (228.6, 180.3)
- moved U8 207.2 mm to (221.7, 186.6)
- moved R45 207.2 mm to (223.0, 181.8)
- moved R46 207.2 mm to (219.9, 181.9)
- moved R42 204.0 mm to (427.0, 189.8)
- moved U6 204.0 mm to (428.0, 186.5)
- moved FB2 204.0 mm to (424.7, 186.8)
- moved R18 204.0 mm to (438.8, 181.0)
- moved R41 204.0 mm to (429.4, 189.8)
- moved R50 98.5 mm to (396.8, 265.1), turned to 180 degrees
- moved D84 94.6 mm to (399.7, 265.1), turned to 180 degrees
- moved R49 74.4 mm to (402.4, 268.4)
- moved SW1 66.9 mm to (408.0, 265.9), turned to 0 degrees
- moved Y2 58.0 mm to (428.6, 269.9), turned to 180 degrees
- moved U7 4.76 mm to (309.0, 191.3)
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Connections:
- U9 pad 49: ENCODER_A -> Net-(U9-Pad49)
Routing:
- net HUB_PORT2_D+: track 4.92 -> 359.3 mm, vias 2 -> 3
- net HUB_PORT2_D-: track 5.59 -> 359.7 mm, vias 2 -> 3
- net HUB_PORT5_D+: track 0.00 -> 347.2 mm, vias 0 -> 2
- net HUB_PORT5_D-: track 0.00 -> 346.1 mm, vias 0 -> 2
- net HUB_PORT3_D+: track 5.50 -> 247.4 mm, vias 2 -> 3
- net HUB_PORT3_D-: track 6.31 -> 248.0 mm, vias 2 -> 3
- net HUB_PORT6_D-: track 1.35 -> 226.1 mm, vias 1 -> 2
- net HUB_PORT6_D+: track 1.35 -> 224.3 mm, vias 1 -> 2
- net HUB_D-: track 1.47 -> 202.6 mm, vias 1 -> 2
- net HUB_D+: track 1.47 -> 200.9 mm, vias 1 -> 2
- net KEYBOARD_SDA: track 0.00 -> 64.6 mm
- net +5V: track 41.4 -> 104.1 mm, vias 2 -> 3
- net KEYBOARD_SCL: track 0.00 -> 61.1 mm
- net HUB_LED2: track 13.3 -> 57.5 mm
- net HUB_PORT4_D-: track 5.14 -> 43.0 mm
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
Commit message: LEDs routed, removed 1 USB port
Parts:
- removed D107: Green, LED_SMD:LED_0402_1005Metric
- removed D108: Amber, LED_SMD:LED_0402_1005Metric
- removed FB6, FB7: 3A, Inductor_SMD:L_0805_2012Metric
- removed R20, R52: 330, Resistor_SMD:R_0805_2012Metric
- removed R45, R46: 22, Resistor_SMD:R_0805_2012Metric
- removed U8: PRTR5V0U2X, random-keyboard-parts:SOT143B
- added MX17: F1, CherryMX_PCB_KailhSocket_LTST-A683CEGBW:CherryMX_1.00u_PCB_KailhSocket_LTST-A683CEGBW, F.Cu at (150.8, 208.0)
- added MX23: F2, CherryMX_PCB_KailhSocket_LTST-A683CEGBW:CherryMX_1.00u_PCB_KailhSocket_LTST-A683CEGBW, F.Cu at (169.9, 208.0)
- added MX27: C, CherryMX_PCB_KailhSocket_LTST-A683CEGBW:CherryMX_1.00u_PCB_KailhSocket_LTST-A683CEGBW, F.Cu at (193.7, 288.9)
- moved R5 120.2 mm to (185.9, 312.7), turned to 0 degrees
- moved D41 117.5 mm to (184.9, 309.9), turned to 270 degrees
- moved R6 117.0 mm to (189.8, 310.4), turned to 0 degrees
- moved D40 116.3 mm to (186.5, 309.9), turned to 90 degrees
- moved D42 114.3 mm to (188.9, 307.5), turned to 90 degrees
- moved D43 113.1 mm to (190.5, 307.5), turned to 270 degrees
- moved R7 111.2 mm to (185.9, 306.4), turned to 0 degrees
- moved D45 109.3 mm to (184.9, 304.0), turned to 270 degrees
- moved R8 108.3 mm to (189.8, 304.0), turned to 0 degrees
- moved D44 107.9 mm to (186.5, 304.0), turned to 90 degrees
- moved D102 106.6 mm to (188.9, 301.6), turned to 270 degrees
- moved D46 105.1 mm to (190.5, 301.6), turned to 90 degrees
- moved D103 103.2 mm to (187.3, 300.0)
- moved D104 103.2 mm to (187.3, 298.4)
- moved R9 103.2 mm to (184.9, 299.4)
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Connections:
- IC1 pad 46: HUB_LED7 -> GND
- R39 pad 2: HUB_PORT7_D+ -> HUB_PORT4_D+
- R40 pad 2: HUB_PORT7_D- -> HUB_PORT4_D-
Routing:
- net HUB_DRV: track 172.0 -> 43.7 mm
- net HUB_LED1: track 122.3 -> 40.2 mm, vias 2 -> 0
- net HUB_LED2: track 57.5 -> 6.24 mm, vias 1 -> 0
- net HUB_LED7: track 32.6 -> 0.00 mm, vias 1 -> 0
- net HUB_LED4: track 27.9 -> 7.00 mm, vias 1 -> 0
- net HUB_LED3: track 30.2 -> 10.3 mm, vias 1 -> 0
- net HUB_LED5: track 7.00 -> 24.4 mm, vias 1 -> 2
- net +5V: track 104.1 -> 88.1 mm
- net HUB_LED6: track 38.3 -> 22.4 mm, vias 1 -> 2
- net +1V8: track 0.00 -> 7.45 mm, vias 0 -> 1
- net Net-(C64-Pad1): track 7.18 -> 0.00 mm
- net HUB_SDA: track 30.4 -> 37.4 mm
- net Net-(D107-Pad1): track 3.48 -> 0.00 mm
- net Net-(J3-Pad2): track 2.71 -> 0.00 mm
- net HUB_PORT4_D-: track 43.0 -> 40.4 mm, vias 2 -> 1
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
Commit message: Moved USB hub to top, made top gap 0.5u
Parts:
- added MX19: W, CherryMX_PCB_KailhSocket_LTST-A683CEGBW:CherryMX_1.00u_PCB_KailhSocket_LTST-A683CEGBW, F.Cu at (160.3, 250.8)
- added MX31: F, CherryMX_PCB_KailhSocket_LTST-A683CEGBW:CherryMX_1.00u_PCB_KailhSocket_LTST-A683CEGBW, F.Cu at (203.2, 269.9)
- moved Y1 142.1 mm to (108.7, 216.7), turned to 180 degrees
- moved C53 138.1 mm to (108.7, 219.9), turned to 180 degrees
- moved R24 137.2 mm to (111.9, 216.7), turned to 90 degrees
- moved C42 132.7 mm to (132.7, 206.4)
- moved R12 132.7 mm to (128.5, 206.4)
- moved R17 130.3 mm to (115.9, 216.7), turned to 0 degrees
- moved IC1 117.6 mm to (128.1, 214.8), turned to 270 degrees
- moved R4 109.0 mm to (153.2, 216.0), turned to 270 degrees
- moved D39 106.5 mm to (155.6, 216.2), turned to 270 degrees
- moved C40 101.6 mm to (139.5, 215.1), turned to 180 degrees
- moved R5 100.4 mm to (158.8, 216.0), turned to 270 degrees
- moved D41 97.6 mm to (161.6, 215.1), turned to 180 degrees
- moved R6 97.3 mm to (165.9, 216.0), turned to 270 degrees
- moved U2 96.6 mm to (144.5, 212.7), turned to 0 degrees
- moved R11 96.6 mm to (142.1, 218.4), turned to 90 degrees
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Routing:
- net KEYBOARD_D+: track 217.3 -> 15.8 mm, vias 2 -> 1
- net KEYBOARD_D-: track 216.8 -> 15.8 mm, vias 2 -> 1
- net HUB_D-: track 202.6 -> 4.74 mm, vias 2 -> 1
- net HUB_D+: track 200.9 -> 4.55 mm, vias 2 -> 1
- net HUB_PORT6_D-: track 226.1 -> 36.2 mm, vias 2 -> 1
- net HUB_PORT6_D+: track 224.3 -> 36.0 mm, vias 2 -> 1
- net HUB_PORT5_D+: track 347.2 -> 207.5 mm, vias 2 -> 0
- net HUB_PORT5_D-: track 346.1 -> 207.5 mm, vias 2 -> 0
- net HUB_PORT3_D-: track 247.4 -> 126.1 mm, vias 3 -> 2
- net HUB_PORT3_D+: track 246.7 -> 126.3 mm, vias 3 -> 2
- net HUB_PORT2_D-: track 359.7 -> 242.0 mm, vias 3 -> 2
- net HUB_PORT2_D+: track 359.3 -> 242.2 mm, vias 3 -> 2
- net HUB_LED4: track 7.00 -> 52.0 mm
- net HUB_LED6: track 22.4 -> 67.1 mm, vias 2 -> 0
- net HUB_DRV: track 43.7 -> 87.1 mm, vias 2 -> 0
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Other:
- board size 385.8 x 128.6 mm -> 385.8 x 133.3 mm

Commit message: Connected all USB ports to hub
Parts:
- moved FB4 127.7 mm to (305.1, 196.8), turned to 180 degrees
- moved FB3 67.3 mm to (432.3, 196.8), turned to 180 degrees
- moved R30 26.7 mm to (384.1, 261.9), turned to 180 degrees
- moved R43 25.4 mm to (311.1, 201.6)
- moved R44 25.4 mm to (308.8, 201.7)
- moved R28 23.3 mm to (384.2, 264.3), turned to 180 degrees
- moved R18 20.7 mm to (438.8, 192.1)
- moved FB2 20.7 mm to (424.7, 197.9)
- moved R41 20.7 mm to (429.4, 200.9)
- moved R42 20.7 mm to (427.0, 200.9)
- moved U6 20.7 mm to (428.0, 197.6)
- moved FB5 20.4 mm to (314.9, 196.8), turned to 180 degrees
- moved R19 17.2 mm to (321.6, 192.1), turned to 0 degrees
- moved U7 16.8 mm to (309.8, 197.8), turned to 180 degrees
- moved U3 13.5 mm to (390.4, 197.1)
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Connections:
- net Net-(IC1-Pad44) renamed HUB_OUTPUT_POWER
- R39 pad 2: HUB_PORT4_D+ -> HUB_PORT2_D+
- R40 pad 2: HUB_PORT4_D- -> HUB_PORT2_D-
- R41 pad 2: HUB_PORT2_D+ -> HUB_PORT3_D+
- R42 pad 2: HUB_PORT2_D- -> HUB_PORT3_D-
- R43 pad 2: HUB_PORT3_D+ -> HUB_PORT4_D+
- R44 pad 2: HUB_PORT3_D- -> HUB_PORT4_D-
- U9 pad 49: Net-(U9-Pad49) -> ENCODER_A
Routing:
- net KEYBOARD_D-: track 15.8 -> 354.6 mm, vias 1 -> 2
- net KEYBOARD_D+: track 15.8 -> 354.1 mm, vias 1 -> 2
- net HUB_PORT3_D-: track 126.1 -> 353.2 mm
- net HUB_PORT3_D+: track 126.3 -> 351.5 mm
- net HUB_PORT4_D+: track 0.00 -> 221.7 mm, vias 0 -> 2
- net HUB_PORT4_D-: track 0.00 -> 219.8 mm, vias 0 -> 2
- net HUB_PORT2_D-: track 242.0 -> 452.8 mm
- net HUB_PORT2_D+: track 242.2 -> 451.3 mm
- net HUB_PORT5_D-: track 207.5 -> 306.6 mm, vias 0 -> 2
- net HUB_PORT5_D+: track 207.5 -> 305.6 mm, vias 0 -> 2
- net HUB_D-: track 4.74 -> 40.8 mm, vias 1 -> 2
- net HUB_D+: track 4.55 -> 40.5 mm, vias 1 -> 2
- net Net-(R28-Pad1): track 26.6 -> 5.29 mm, vias 2 -> 0
- net Net-(R30-Pad1): track 25.8 -> 7.62 mm, vias 2 -> 0
- net +5V: track 88.1 -> 74.6 mm
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
Commit message: State before deleting all traces
Parts:
- moved R23 0.79 mm to (96.0, 194.5)
- moved R26 0.79 mm to (103.9, 194.5)
- moved R37 0.79 mm to (100.9, 196.8)
- moved R38 0.79 mm to (100.9, 199.2)
- moved U4 0.79 mm to (96.7, 198.2)
Routing:
- net +5V: track 74.6 -> 198.2 mm
- net Net-(R37-Pad1): track 10.5 -> 11.7 mm
- net Net-(R23-Pad1): track 3.77 -> 4.56 mm
- net Net-(R38-Pad1): track 14.0 -> 14.7 mm
- net Net-(R26-Pad1): track 3.12 -> 3.91 mm
