File: PCB/_autosave-custom_keyboard.kicad_pcb (KiCad board)
At the start: 2 copper layers, 3.4 x 3 mm, 116 parts, among them IC1 FE2.1, SW1 SW_Push, U1 PRTR5V0U2X, U2 24LC02, U3 PRTR5V0U2X, U4 PRTR5V0U2X, U5 PRTR5V0U2X, U6 PRTR5V0U2X, U7 PRTR5V0U2X, U8 PRTR5V0U2X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

Commit message: Organized USB Hub location
Parts:
- added C53: 20pF, Capacitor_SMD:C_0805_2012Metric, B.Cu at (218.3, 304.0)
- added D102: Amber, LED_SMD:LED_0402_1005Metric, B.Cu at (181.8, 195.3)
- added D103: Green, LED_SMD:LED_0402_1005Metric, B.Cu at (188.9, 196.8)
- added D104: Amber, LED_SMD:LED_0402_1005Metric, B.Cu at (188.9, 195.3)
- added D105: Green, LED_SMD:LED_0402_1005Metric, B.Cu at (196.1, 196.8)
- added D106: Amber, LED_SMD:LED_0402_1005Metric, B.Cu at (196.1, 195.3)
- added D39: Red, LED_SMD:LED_0402_1005Metric, B.Cu at (195.0, 315.1)
- added D40: Green, LED_SMD:LED_0402_1005Metric, B.Cu at (159.2, 196.8)
- added D41: Amber, LED_SMD:LED_0402_1005Metric, B.Cu at (159.2, 195.3)
- added D42: Green, LED_SMD:LED_0402_1005Metric, B.Cu at (167.2, 195.3)
- added D43: Amber, LED_SMD:LED_0402_1005Metric, B.Cu at (167.2, 196.8)
- added D44: Green, LED_SMD:LED_0402_1005Metric, B.Cu at (174.6, 196.8)
- added D45: Amber, LED_SMD:LED_0402_1005Metric, B.Cu at (174.6, 195.3)
- added D46: Green, LED_SMD:LED_0402_1005Metric, B.Cu at (181.8, 196.8)
- added MX3: M3, CherryMX_PCB_KailhSocket_LTST-A683CEGBW:CherryMX_1.00u_PCB_KailhSocket_LTST-A683CEGBW, F.Cu at (88.9, 269.9)
- moved C40 287.1 mm to (181.8, 312.1), turned to 270 degrees
- moved R15 284.6 mm to (185.1, 304.8), turned to 180 degrees
- moved R13 283.2 mm to (185.1, 307.2), turned to 180 degrees
- moved R11 282.1 mm to (185.1, 309.6), turned to 180 degrees
- moved C42 269.5 mm to (208.1, 315.1)
- moved R24 259.3 mm to (215.1, 307.2), turned to 270 degrees
- moved FB2 207.0 mm to (220.7, 190.8), turned to 270 degrees
- moved R12 164.8 mm to (203.9, 315.1)
- moved Y1 156.6 mm to (218.3, 307.2), turned to 0 degrees
- moved R4 146.6 mm to (198.6, 315.1), turned to 0 degrees
- moved U2 138.5 mm to (179.4, 307.2), turned to 90 degrees
- moved IC1 135.9 mm to (200.5, 307.4), turned to 90 degrees
- moved R17 133.6 mm to (211.1, 305.6)
- moved FB5 120.3 mm to (312.7, 191.6), turned to 90 degrees
- moved U9 103.7 mm to (407.1, 270.7), turned to 270 degrees
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Connections:
- FB1 pad 1: VCC -> Net-(FB1-Pad1)
- FB2 pad 1: +5V -> Net-(FB2-Pad1)
- FB3 pad 2: GND -> Net-(FB3-Pad2)
- FB4 pad 1: +5V -> Net-(FB4-Pad1)
- FB5 pad 2: GND -> Net-(FB5-Pad2)
- FB6 pad 1: +5V -> Net-(FB6-Pad1)
- FB7 pad 2: GND -> Net-(FB7-Pad2)
- U6 pad 2: HUB_PORT2_D- -> Net-(J1-Pad3)
- U6 pad 3: HUB_PORT2_D+ -> Net-(J1-Pad2)
- U6 pad 4: +5V -> Net-(FB2-Pad1)
- U7 pad 2: HUB_PORT3_D- -> Net-(J2-Pad3)
- U7 pad 3: HUB_PORT3_D+ -> Net-(J2-Pad2)
- U7 pad 4: +5V -> Net-(FB4-Pad1)
- U8 pad 2: HUB_PORT4_D- -> Net-(J3-Pad3)
- U8 pad 3: HUB_PORT4_D+ -> Net-(J3-Pad2)
- U8 pad 4: +5V -> Net-(FB6-Pad1)
- USB1 pad 11: VCC -> Net-(FB1-Pad1)
- USB1 pad 2: VCC -> Net-(FB1-Pad1)
Routing:
- net HUB_LED1: track 0.00 -> 35.9 mm, vias 0 -> 1
- net HUB_SDA: track 0.00 -> 30.4 mm
- net HUB_DRV: track 0.00 -> 15.4 mm, vias 0 -> 1
- net +3V3: track 0.00 -> 14.2 mm
- net Net-(FB1-Pad1): track 0.00 -> 13.6 mm
- net +5V: track 51.8 -> 38.5 mm
- net HUB_LED5: track 0.00 -> 12.6 mm, vias 0 -> 1
- net HUB_LED6: track 0.00 -> 12.5 mm, vias 0 -> 1
- net HUB_LED7: track 0.00 -> 12.5 mm, vias 0 -> 1
- net ROW5: track 371.1 -> 381.5 mm
- net HUB_LED2: track 0.00 -> 9.87 mm, vias 0 -> 1
- net COL4: track 101.8 -> 111.2 mm, vias 5 -> 6
- net HUB_XOUT: track 15.3 -> 24.0 mm
- net COL5: track 98.6 -> 107.3 mm, vias 5 -> 6
- net COL6: track 121.1 -> 129.1 mm, vias 6 -> 7
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Other:
- board size 3.4 x 3 mm -> 385.8 x 128.6 mm
