File: PCB/_autosave-custom_keyboard.kicad_pcb (KiCad board)
At the start: 2 copper layers, 385.8 x 128.6 mm, 133 parts, among them IC1 FE2.1, SW1 SW_Push, U1 PRTR5V0U2X, U2 24LC02, U3 PRTR5V0U2X, U4 PRTR5V0U2X, U5 PRTR5V0U2X, U6 PRTR5V0U2X, U7 PRTR5V0U2X, U8 PRTR5V0U2X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

Commit message: LED routing
Parts:
- moved R28 104.3 mm to (397.7, 283.4), turned to 270 degrees
- moved R30 102.6 mm to (400.1, 283.4), turned to 270 degrees
- moved R50 98.5 mm to (396.8, 265.1), turned to 180 degrees
- moved D84 94.6 mm to (399.7, 265.1), turned to 180 degrees
- moved R49 74.4 mm to (402.4, 268.4)
- moved SW1 66.9 mm to (408.0, 265.9), turned to 0 degrees
- moved Y2 58.0 mm to (428.6, 269.9), turned to 180 degrees
- moved R10 0.92 mm to (193.7, 196.2), turned to 270 degrees
- moved R5 0.92 mm to (156.4, 196.2), turned to 270 degrees
- moved R6 0.92 mm to (164.3, 196.2), turned to 270 degrees
- moved R8 0.92 mm to (179.4, 196.2), turned to 270 degrees
- moved R9 0.92 mm to (186.5, 196.2), turned to 270 degrees
- moved R52 0.80 mm to (200.8, 196.2), turned to 270 degrees
- moved D44 0.79 mm to (173.8, 196.8)
- moved D45 0.79 mm to (173.8, 195.3)
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Routing:
- net KEYBOARD_D+: track 0.00 -> 217.3 mm, vias 0 -> 2
- net KEYBOARD_D-: track 0.00 -> 216.8 mm, vias 0 -> 2
- net HUB_DRV: track 15.4 -> 205.7 mm, vias 1 -> 2
- net HUB_LED1: track 35.9 -> 157.8 mm, vias 1 -> 2
- net KEYBOARD_SDA: track 0.00 -> 56.2 mm
- net +5V: track 41.4 -> 97.5 mm, vias 2 -> 3
- net KEYBOARD_SCL: track 0.00 -> 51.5 mm
- net KEYBOARD_XTAL1: track 10.9 -> 37.7 mm
- net KEYBOARD_XTAL2: track 9.09 -> 35.8 mm
- net Net-(R28-Pad1): track 0.00 -> 26.6 mm, vias 0 -> 2
- net Net-(R30-Pad1): track 0.00 -> 25.8 mm, vias 0 -> 2
- net ENCODER_A: track 30.5 -> 11.7 mm
- net ENCODER_B2: track 34.7 -> 16.2 mm
- net ROT1_ROW: track 400.9 -> 383.4 mm
- net KEYBOARD_RESET: track 0.00 -> 17.0 mm
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