File: PCB/_autosave-custom_keyboard (2).sch (KiCad schematic (older format))
At the start: 487 parts, among them IC1 FE2.1, J1 Conn_01x08_Male, J2 USB_A, J3 USB_A, J4 USB_A, SW1 SW_Push, U1 AT90USB646-MU, U2 PRTR5V0U2X, U3 24LC02, U4 PRTR5V0U2X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

Commit message: replaced controller with ATMEGA32U4
Parts:
- added C?: 1uF, Capacitor_SMD:C_0805_2012Metric, symbol Device:C_Small
- added R?: 10k, Resistor_SMD:R_0805_2012Metric, symbol Device:R_Small
- added R? (x2): 22, Resistor_SMD:R_0805_2012Metric, symbol Device:R_Small
- added U?: ATmega32U4-MU, Package_DFN_QFN:QFN-44-1EP_7x7mm_P0.5mm_EP5.2x5.2mm, symbol MCU_Microchip_ATmega:ATmega32U4-MU
Connections:
- wire segments 2008 -> 2048
Other:
- moved on the sheet: C1, C10, C11, C12, C2, C3, C4, C5, C6, C7, C8, C9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
