File: PCB/custom_keyboard (2).kicad_pcb (KiCad board)
At the start: 2 copper layers, 88 parts, among them SW1 SW_Push, U1 ATmega32U4-MU, U2 PRTR5V0U2X, U3 24LC02, U4 PRTR5V0U2X, U5 PRTR5V0U2X, U6 PRTR5V0U2X, U7 PRTR5V0U2X, U8 PRTR5V0U2X, U9 PRTR5V0U2X, Y1 16MHz, Y2 12MHz

Commit message: Keyboard diodes in place
Parts:
- added LED1: WS2812B, LED_SMD:LED_SK6812MINI_PLCC4_3.5x3.5mm_P1.75mm, B.Cu at (177.0, 0.79)
- added LED10: WS2812B, LED_SMD:LED_SK6812MINI_PLCC4_3.5x3.5mm_P1.75mm, B.Cu at (380.9, -97.8)
- added LED11: WS2812B, LED_SMD:LED_SK6812MINI_PLCC4_3.5x3.5mm_P1.75mm, B.Cu at (276.9, -203.7)
- added LED12: WS2812B, LED_SMD:LED_SK6812MINI_PLCC4_3.5x3.5mm_P1.75mm, B.Cu at (319.5, -151.9)
- added LED13: WS2812B, LED_SMD:LED_SK6812MINI_PLCC4_3.5x3.5mm_P1.75mm, B.Cu at (339.7, -126.1)
- added LED14: WS2812B, LED_SMD:LED_SK6812MINI_PLCC4_3.5x3.5mm_P1.75mm, B.Cu at (239.8, -227.8)
- added LED15: WS2812B, LED_SMD:LED_SK6812MINI_PLCC4_3.5x3.5mm_P1.75mm, B.Cu at (390.6, -77.7)
- added LED16: WS2812B, LED_SMD:LED_SK6812MINI_PLCC4_3.5x3.5mm_P1.75mm, B.Cu at (250.5, -218.0)
- added LED17: WS2812B, LED_SMD:LED_SK6812MINI_PLCC4_3.5x3.5mm_P1.75mm, B.Cu at (280.2, -181.8)
- added LED18: WS2812B, LED_SMD:LED_SK6812MINI_PLCC4_3.5x3.5mm_P1.75mm, B.Cu at (196.1, -238.8)
- added LED19: WS2812B, LED_SMD:LED_SK6812MINI_PLCC4_3.5x3.5mm_P1.75mm, B.Cu at (268.4, -197.1)
- added LED2: WS2812B, LED_SMD:LED_SK6812MINI_PLCC4_3.5x3.5mm_P1.75mm, B.Cu at (196.0, 0.00)
- added LED20: WS2812B, LED_SMD:LED_SK6812MINI_PLCC4_3.5x3.5mm_P1.75mm, B.Cu at (390.6, -71.1)
- added LED21: WS2812B, LED_SMD:LED_SK6812MINI_PLCC4_3.5x3.5mm_P1.75mm, B.Cu at (303.5, -163.3)
- added LED22: WS2812B, LED_SMD:LED_SK6812MINI_PLCC4_3.5x3.5mm_P1.75mm, B.Cu at (229.8, -238.2)
- added LED23: WS2812B, LED_SMD:LED_SK6812MINI_PLCC4_3.5x3.5mm_P1.75mm, B.Cu at (179.3, -238.8)
- added LED24: WS2812B, LED_SMD:LED_SK6812MINI_PLCC4_3.5x3.5mm_P1.75mm, B.Cu at (260.0, -203.7)
- added LED25: WS2812B, LED_SMD:LED_SK6812MINI_PLCC4_3.5x3.5mm_P1.75mm, B.Cu at (382.2, -82.5)
- added LED26: WS2812B, LED_SMD:LED_SK6812MINI_PLCC4_3.5x3.5mm_P1.75mm, B.Cu at (353.9, -111.5)
- added LED27: WS2812B, LED_SMD:LED_SK6812MINI_PLCC4_3.5x3.5mm_P1.75mm, B.Cu at (407.1, -55.7)
- added LED28: WS2812B, LED_SMD:LED_SK6812MINI_PLCC4_3.5x3.5mm_P1.75mm, B.Cu at (221.4, -238.2)
- added LED29: WS2812B, LED_SMD:LED_SK6812MINI_PLCC4_3.5x3.5mm_P1.75mm, B.Cu at (303.5, -156.7)
- added LED3: WS2812B, LED_SMD:LED_SK6812MINI_PLCC4_3.5x3.5mm_P1.75mm, B.Cu at (219.9, 0.79)
- added LED30: WS2812B, LED_SMD:LED_SK6812MINI_PLCC4_3.5x3.5mm_P1.75mm, B.Cu at (382.2, -75.9)
- added LED31: WS2812B, LED_SMD:LED_SK6812MINI_PLCC4_3.5x3.5mm_P1.75mm, B.Cu at (260.0, -197.1)
- added LED32: WS2812B, LED_SMD:LED_SK6812MINI_PLCC4_3.5x3.5mm_P1.75mm, B.Cu at (212.9, -238.8)
- added LED33: WS2812B, LED_SMD:LED_SK6812MINI_PLCC4_3.5x3.5mm_P1.75mm, B.Cu at (204.5, -238.8)
- added LED34: WS2812B, LED_SMD:LED_SK6812MINI_PLCC4_3.5x3.5mm_P1.75mm, B.Cu at (295.6, -172.0)
- added LED35: WS2812B, LED_SMD:LED_SK6812MINI_PLCC4_3.5x3.5mm_P1.75mm, B.Cu at (137.2, -239.4)
- added LED36: WS2812B, LED_SMD:LED_SK6812MINI_PLCC4_3.5x3.5mm_P1.75mm, B.Cu at (128.7, -239.4)
- added LED37: WS2812B, LED_SMD:LED_SK6812MINI_PLCC4_3.5x3.5mm_P1.75mm, B.Cu at (120.3, -239.4)
- added LED38: WS2812B, LED_SMD:LED_SK6812MINI_PLCC4_3.5x3.5mm_P1.75mm, B.Cu at (111.9, -239.4)
- added LED39: WS2812B, LED_SMD:LED_SK6812MINI_PLCC4_3.5x3.5mm_P1.75mm, B.Cu at (103.5, -239.4)
- added LED4: WS2812B, LED_SMD:LED_SK6812MINI_PLCC4_3.5x3.5mm_P1.75mm, B.Cu at (242.1, 0.79)
- added LED40: WS2812B, LED_SMD:LED_SK6812MINI_PLCC4_3.5x3.5mm_P1.75mm, B.Cu at (95.1, -239.4)
- added LED41: WS2812B, LED_SMD:LED_SK6812MINI_PLCC4_3.5x3.5mm_P1.75mm, B.Cu at (86.6, -239.4)
- added LED42: WS2812B, LED_SMD:LED_SK6812MINI_PLCC4_3.5x3.5mm_P1.75mm, B.Cu at (389.3, -91.0)
- added LED43: WS2812B, LED_SMD:LED_SK6812MINI_PLCC4_3.5x3.5mm_P1.75mm, B.Cu at (350.3, -118.1)
- added LED44: WS2812B, LED_SMD:LED_SK6812MINI_PLCC4_3.5x3.5mm_P1.75mm, B.Cu at (338.0, -143.1)
- added LED45: WS2812B, LED_SMD:LED_SK6812MINI_PLCC4_3.5x3.5mm_P1.75mm, B.Cu at (297.1, -178.6)
- added LED46: WS2812B, LED_SMD:LED_SK6812MINI_PLCC4_3.5x3.5mm_P1.75mm, B.Cu at (407.4, -69.0)
- added LED47: WS2812B, LED_SMD:LED_SK6812MINI_PLCC4_3.5x3.5mm_P1.75mm, B.Cu at (268.4, -210.4)
- added LED48: WS2812B, LED_SMD:LED_SK6812MINI_PLCC4_3.5x3.5mm_P1.75mm, B.Cu at (145.6, -239.4)
- added LED49: WS2812B, LED_SMD:LED_SK6812MINI_PLCC4_3.5x3.5mm_P1.75mm, B.Cu at (380.9, -104.4)
- added LED5: WS2812B, LED_SMD:LED_SK6812MINI_PLCC4_3.5x3.5mm_P1.75mm, B.Cu at (265.9, 0.79)
- added LED50: WS2812B, LED_SMD:LED_SK6812MINI_PLCC4_3.5x3.5mm_P1.75mm, B.Cu at (238.2, -241.0)
- added LED51: WS2812B, LED_SMD:LED_SK6812MINI_PLCC4_3.5x3.5mm_P1.75mm, B.Cu at (346.4, -132.8)
- added LED52: WS2812B, LED_SMD:LED_SK6812MINI_PLCC4_3.5x3.5mm_P1.75mm, B.Cu at (297.1, -185.2)
- added LED53: WS2812B, LED_SMD:LED_SK6812MINI_PLCC4_3.5x3.5mm_P1.75mm, B.Cu at (312.5, -165.1)
- added LED54: WS2812B, LED_SMD:LED_SK6812MINI_PLCC4_3.5x3.5mm_P1.75mm, B.Cu at (248.2, -234.4)
- added LED55: WS2812B, LED_SMD:LED_SK6812MINI_PLCC4_3.5x3.5mm_P1.75mm, B.Cu at (370.8, -111.5)
- added LED56: WS2812B, LED_SMD:LED_SK6812MINI_PLCC4_3.5x3.5mm_P1.75mm, B.Cu at (285.3, -195.0)
- added LED57: WS2812B, LED_SMD:LED_SK6812MINI_PLCC4_3.5x3.5mm_P1.75mm, B.Cu at (356.5, -124.7)
- added LED58: WS2812B, LED_SMD:LED_SK6812MINI_PLCC4_3.5x3.5mm_P1.75mm, B.Cu at (356.5, -131.4)
- added LED59: WS2812B, LED_SMD:LED_SK6812MINI_PLCC4_3.5x3.5mm_P1.75mm, B.Cu at (256.7, -224.6)
- added LED6: WS2812B, LED_SMD:LED_SK6812MINI_PLCC4_3.5x3.5mm_P1.75mm, B.Cu at (291.3, 0.00)
- added LED60: WS2812B, LED_SMD:LED_SK6812MINI_PLCC4_3.5x3.5mm_P1.75mm, B.Cu at (256.7, -231.2)
- added LED61: WS2812B, LED_SMD:LED_SK6812MINI_PLCC4_3.5x3.5mm_P1.75mm, B.Cu at (336.3, -151.9)
- added LED62: WS2812B, LED_SMD:LED_SK6812MINI_PLCC4_3.5x3.5mm_P1.75mm, B.Cu at (346.4, -139.4)
- added LED63: WS2812B, LED_SMD:LED_SK6812MINI_PLCC4_3.5x3.5mm_P1.75mm, B.Cu at (320.9, -165.1)
- added LED64: WS2812B, LED_SMD:LED_SK6812MINI_PLCC4_3.5x3.5mm_P1.75mm, B.Cu at (187.7, -238.8)
- added LED65: WS2812B, LED_SMD:LED_SK6812MINI_PLCC4_3.5x3.5mm_P1.75mm, B.Cu at (372.4, -91.2)
- added LED66: WS2812B, LED_SMD:LED_SK6812MINI_PLCC4_3.5x3.5mm_P1.75mm, B.Cu at (320.4, -158.5)
- added LED67: WS2812B, LED_SMD:LED_SK6812MINI_PLCC4_3.5x3.5mm_P1.75mm, B.Cu at (327.9, -151.9)
- added LED68: WS2812B, LED_SMD:LED_SK6812MINI_PLCC4_3.5x3.5mm_P1.75mm, B.Cu at (288.6, -188.4)
- added LED69: WS2812B, LED_SMD:LED_SK6812MINI_PLCC4_3.5x3.5mm_P1.75mm, B.Cu at (372.4, -104.4)
- added LED7: WS2812B, LED_SMD:LED_SK6812MINI_PLCC4_3.5x3.5mm_P1.75mm, B.Cu at (407.4, -75.6)
- added LED70: WS2812B, LED_SMD:LED_SK6812MINI_PLCC4_3.5x3.5mm_P1.75mm, B.Cu at (399.0, -77.7)
- added LED71: WS2812B, LED_SMD:LED_SK6812MINI_PLCC4_3.5x3.5mm_P1.75mm, B.Cu at (358.7, -118.1)
- added LED72: WS2812B, LED_SMD:LED_SK6812MINI_PLCC4_3.5x3.5mm_P1.75mm, B.Cu at (258.9, -218.0)
- added LED73: WS2812B, LED_SMD:LED_SK6812MINI_PLCC4_3.5x3.5mm_P1.75mm, B.Cu at (311.9, -158.5)
- added LED74: WS2812B, LED_SMD:LED_SK6812MINI_PLCC4_3.5x3.5mm_P1.75mm, B.Cu at (304.0, -170.0)
- added LED75: WS2812B, LED_SMD:LED_SK6812MINI_PLCC4_3.5x3.5mm_P1.75mm, B.Cu at (390.6, -84.3)
- added LED76: WS2812B, LED_SMD:LED_SK6812MINI_PLCC4_3.5x3.5mm_P1.75mm, B.Cu at (248.2, -227.8)
- added LED77: WS2812B, LED_SMD:LED_SK6812MINI_PLCC4_3.5x3.5mm_P1.75mm, B.Cu at (288.6, -181.8)
- added LED78: WS2812B, LED_SMD:LED_SK6812MINI_PLCC4_3.5x3.5mm_P1.75mm, B.Cu at (362.4, -111.5)
- added LED79: WS2812B, LED_SMD:LED_SK6812MINI_PLCC4_3.5x3.5mm_P1.75mm, B.Cu at (78.2, -239.4)
- added LED8: WS2812B, LED_SMD:LED_SK6812MINI_PLCC4_3.5x3.5mm_P1.75mm, B.Cu at (305.5, -178.4)
- added LED80: WS2812B, LED_SMD:LED_SK6812MINI_PLCC4_3.5x3.5mm_P1.75mm, B.Cu at (380.9, -91.2)
- added LED81: WS2812B, LED_SMD:LED_SK6812MINI_PLCC4_3.5x3.5mm_P1.75mm, B.Cu at (268.4, -203.7)
- added LED82: WS2812B, LED_SMD:LED_SK6812MINI_PLCC4_3.5x3.5mm_P1.75mm, B.Cu at (276.9, -197.1)
- added LED83: WS2812B, LED_SMD:LED_SK6812MINI_PLCC4_3.5x3.5mm_P1.75mm, B.Cu at (239.8, -234.4)
- added LED84: WS2812B, LED_SMD:LED_SK6812MINI_PLCC4_3.5x3.5mm_P1.75mm, B.Cu at (348.1, -126.1)
- added LED85: WS2812B, LED_SMD:LED_SK6812MINI_PLCC4_3.5x3.5mm_P1.75mm, B.Cu at (338.0, -136.5)
- added LED86: WS2812B, LED_SMD:LED_SK6812MINI_PLCC4_3.5x3.5mm_P1.75mm, B.Cu at (407.1, -62.3)
- added LED87: WS2812B, LED_SMD:LED_SK6812MINI_PLCC4_3.5x3.5mm_P1.75mm, B.Cu at (260.0, -210.4)
- added LED88: WS2812B, LED_SMD:LED_SK6812MINI_PLCC4_3.5x3.5mm_P1.75mm, B.Cu at (372.4, -97.8)
- added LED89: WS2812B, LED_SMD:LED_SK6812MINI_PLCC4_3.5x3.5mm_P1.75mm, B.Cu at (399.0, -71.1)
- added LED9: WS2812B, LED_SMD:LED_SK6812MINI_PLCC4_3.5x3.5mm_P1.75mm, B.Cu at (312.5, -171.8)
- added LED90: WS2812B, LED_SMD:LED_SK6812MINI_PLCC4_3.5x3.5mm_P1.75mm, B.Cu at (280.2, -188.4)
- added MX8: TAB, MX_Only:MXOnly-1.5U-Hotswap, F.Cu at (177.0, 236.5)
- moved RD2 424.1 mm to (499.2, 196.0), turned to 90 degrees
- moved RD1 376.8 mm to (157.2, 181.8), turned to 270 degrees
- moved USB1 300.5 mm to (-14.3, -167.5)
- moved MX68 280.6 mm to (396.1, 255.6)
- moved MX74 280.6 mm to (436.5, 293.7)
- moved MX76 280.6 mm to (429.4, 217.5)
- moved MX77 280.6 mm to (434.2, 236.5)
- moved MX80 280.6 mm to (467.5, 293.7)
- moved MX81 280.6 mm to (467.5, 188.9)
- moved MX82 280.6 mm to (467.5, 217.5)
- moved MX83 280.6 mm to (467.5, 236.5)
- moved MX89 280.6 mm to (505.6, 217.5)
- moved MX90 280.6 mm to (505.6, 236.5)
- moved MX91 280.6 mm to (505.6, 293.7)
- moved ROT2 280.6 mm to (142.5, 185.6)
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Other:
- board outline added: 385.7 x 133.3 mm

Commit message: Routed rows and some columns
Parts:
- added F1: 500mA, Fuse:Fuse_1206_3216Metric, B.Cu at (469.1, 105.6)
- added F2: 500mA, Fuse:Fuse_1206_3216Metric, B.Cu at (469.1, 102.3)
- added F3: 500mA, Fuse:Fuse_1206_3216Metric, B.Cu at (474.7, 105.6)
- added F4: 500mA, Fuse:Fuse_1206_3216Metric, B.Cu at (469.1, 99.0)
- added F5: 500mA, Fuse:Fuse_1206_3216Metric, B.Cu at (474.7, 102.3)
- added F6: 500mA, Fuse:Fuse_1206_3216Metric, B.Cu at (480.3, 105.6)
- added F7: 500mA, Fuse:Fuse_1206_3216Metric, B.Cu at (474.7, 99.0)
- added FB1: 60 @ 100MHz, Inductor_SMD:L_0805_2012Metric, B.Cu at (490.7, 115.0)
- added FB3: 60 @ 100MHz, Inductor_SMD:L_0805_2012Metric, B.Cu at (490.7, 112.3)
- added FB4: 60 @ 100MHz, Inductor_SMD:L_0805_2012Metric, B.Cu at (495.2, 115.0)
- added FB5: 60 @ 100MHz, Inductor_SMD:L_0805_2012Metric, B.Cu at (495.2, 112.3)
- added IC1: FE2.1, custom-footprints:FE2.1, B.Cu at (342.1, 106.4)
- added MX17: 1, MX_Only:MXOnly-1U-Hotswap, F.Cu at (191.3, 217.5)
- added MX3: M3, MX_Only:MXOnly-1U-Hotswap, F.Cu at (148.4, 255.6)
- OL1: footprint Resistor_SMD:R_0805_2012Metric -> kbd:OLED_v2
- moved OL1 447.3 mm to (468.3, 255.6), turned to 90 degrees
- moved Y1 323.5 mm to (381.0, 107.9)
- moved U1 318.3 mm to (393.7, 104.8), turned to 90 degrees
- moved R7 281.9 mm to (397.6, 99.2), turned to 180 degrees
- moved SW1 251.1 mm to (370.7, 122.2), turned to 180 degrees
- moved R9 227.5 mm to (368.2, 118.3), turned to 180 degrees
- moved LED1 193.7 mm to (172.2, 194.5)
Routing:
- net ROW9: track 0.00 -> 386.4 mm, vias 0 -> 2
- net ROW8: track 0.00 -> 376.8 mm
- net ROT1_ROW: track 0.00 -> 364.7 mm, vias 0 -> 2
- net ROT2_ROW: track 0.00 -> 363.4 mm
- net ROW2: track 0.00 -> 357.2 mm
- net ROW3: track 0.00 -> 357.1 mm
- net ROW5: track 0.00 -> 352.2 mm
- net ROW4: track 0.00 -> 350.8 mm
- net ROW10: track 0.00 -> 349.5 mm, vias 0 -> 2
- net ROW6: track 0.00 -> 290.4 mm
- net COL0: track 0.00 -> 255.2 mm, vias 0 -> 10
- net COL1: track 0.00 -> 249.9 mm, vias 0 -> 11
- net ROW7: track 0.00 -> 218.7 mm
- net COL2: track 0.00 -> 218.4 mm, vias 0 -> 11
- net Net-(KD90-Pad2): track 0.00 -> 4.30 mm
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