File: PCB/custom_keyboard (2).sch (KiCad schematic (older format))
At the start: 487 parts, among them IC1 FE2.1, J1 USB_A, J2 USB_A, J3 USB_A, J4 Conn_01x08_Male, SW1 ESC, SW10 F9, SW11 F10, SW12 F11, SW13 F12, SW14 PSCR, SW15 M1, SW16 `/~, SW17 1, SW18 2, SW19 3, SW2 F1, SW20 4, SW21 5, SW22 6, SW23 7, SW24 8, SW25 9, SW26 0, SW27 -/_, SW28 =/+, SW29 BACKSPACE, SW3 F2, SW30 INS, SW31 HOME, SW32 PGUP, SW33 M2, SW34 TAB, SW35 Q, SW36 W, SW37 E, SW38 R, SW39 T, SW4 F3, SW40 Y, SW41 U, SW42 I, SW43 O, SW44 P, SW45 [/{, SW46 ]/}, SW47 \\, SW48 DELETE, SW49 END, SW5 F4, SW50 PGDN, SW51 M3, SW52 CAPS, SW53 A, SW54 S, SW55 D, SW56 F, SW57 G, SW58 H, SW59 J, SW6 F5, SW60 K, SW61 L, SW62 ;/:, SW63 '/\", SW64 ENTER, SW65 M4, SW66 LSHIFT, SW67 Z, SW68 X, SW69 C, SW7 F6, SW70 V, SW71 B, SW72 N, SW73 M, SW74 ,/<, SW75 ./>, SW76 /, SW77 RSHIFT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

Commit message: Relabeled keyboard and LED matrix
Parts:
- removed C107, C25, C35, C51, C62, C75, C86, C97: 0.1uF, Capacitor_SMD:C_0805_2012Metric, symbol Device:C_Small
- added LC2, LC3, LC4, LC5, LC6, LC7, LC8, LC9: 0.1uF, Capacitor_SMD:C_0805_2012Metric, symbol Device:C_Small
- gave numbers to parts that had none: 11
- renumbered C85 to C1, C48 to C10, C50 to C11, C61 to C12, C9 to C13, C5 to C14, C1 to C15, C6 to C16, C4 to C17, C7 to C18, C23 to C19, C117 to C2, C3 to C23, C10 to C24, C22 to C25, C2 to C28, C8 to C29, C118 to C3, C11 to C30, C24 to C32, C49 to C33, C73 to C34, C96 to C4, C45 to C5, C119 to C6, C46 to C7, C120 to C8, C47 to C9, D161 to D1, D160 to D2, D113 to D3, D124 to D4, D125 to D5, D136 to D6, D137 to D7, D148 to D8, D159 to D9, J4 to J1, J1 to J2, J2 to J3, J3 to J4, D15 to KD1, D66 to KD10, D80 to KD11, D17 to KD12, D35 to KD13, D53 to KD14, D67 to KD15, D81 to KD16, D2 to KD17, D18 to KD18, D36 to KD19, D33 to KD2, D54 to KD20, D68 to KD21, D82 to KD22, D3 to KD23, D19 to KD24, D37 to KD25, D55 to KD26, D69 to KD27, D4 to KD28, D20 to KD29, D51 to KD3, D38 to KD30, D56 to KD31, D70 to KD32, D5 to KD33, D21 to KD34, D39 to KD35, D57 to KD36, D71 to KD37, D83 to KD38, D6 to KD39, D65 to KD4, D22 to KD40, D40 to KD41, D58 to KD42, D72 to KD43, D7 to KD44, D23 to KD45, D41 to KD46, D59 to KD47, D73 to KD48, D8 to KD49, D79 to KD5, D24 to KD50, D42 to KD51, D60 to KD52, D74 to KD53, D9 to KD54, D25 to KD55, D43 to KD56, D61 to KD57, D75 to KD58, D84 to KD59, D1 to KD6, D10 to KD60, D26 to KD61, D44 to KD62, D62 to KD63, D76 to KD64, D85 to KD65, D11 to KD66, D27 to KD67, D45 to KD68, D63 to KD69, D16 to KD7, D12 to KD70, D28 to KD71, D46 to KD72, D86 to KD73, D13 to KD74, D29 to KD75, D47 to KD76, D64 to KD77, D77 to KD78, D87 to KD79, D34 to KD8, D14 to KD80, D30 to KD81, D48 to KD82, D88 to KD83, D31 to KD84, D49 to KD85, D78 to KD86, D89 to KD87, D32 to KD88, D50 to KD89, D52 to KD9, D90 to KD90, C12 to LC1, C13 to LC10, C26 to LC11, C36 to LC12, C52 to LC13, C63 to LC14, C76 to LC15, C87 to LC16, C98 to LC17, C108 to LC18, C14 to LC19, C27 to LC20, C37 to LC21, C53 to LC22, C64 to LC23, C77 to LC24, C88 to LC25, C99 to LC26, C109 to LC27, C15 to LC28, C28 to LC29, C38 to LC30, C54 to LC31, C65 to LC32, C78 to LC33, C89 to LC34, C100 to LC35, C110 to LC36, C16 to LC37, C29 to LC38, C39 to LC39, C55 to LC40, C66 to LC41, C79 to LC42, C90 to LC43, C101 to LC44, C111 to LC45, C17 to LC46, C30 to LC47, C40 to LC48, C56 to LC49, C67 to LC50, C80 to LC51, C91 to LC52, C102 to LC53, C112 to LC54, C18 to LC55, C31 to LC56, C41 to LC57, C57 to LC58, C68 to LC59, C81 to LC60, C92 to LC61, C103 to LC62, C113 to LC63, C19 to LC64, C32 to LC65, C42 to LC66, C58 to LC67, C69 to LC68, C82 to LC69, C93 to LC70, C104 to LC71, C114 to LC72, C20 to LC73, C33 to LC74, C43 to LC75, C59 to LC76, C70 to LC77, C83 to LC78, C94 to LC79, C105 to LC80, C115 to LC81, C21 to LC82, C34 to LC83, C44 to LC84, C60 to LC85, C71 to LC86, C84 to LC87, C95 to LC88, C106 to LC89, C116 to LC90, D91 to LED1, D92 to LED10, D102 to LED11, D115 to LED12, D127 to LED13, D139 to LED14, D150 to LED15, D163 to LED16, D173 to LED17, D183 to LED18, D93 to LED19, D101 to LED2, D103 to LED20, D116 to LED21, D128 to LED22, D140 to LED23, D151 to LED24, D164 to LED25, D174 to LED26, D184 to LED27, D94 to LED28, D104 to LED29, D114 to LED3, D117 to LED30, D129 to LED31, D141 to LED32, D152 to LED33, D165 to LED34, D175 to LED35, D185 to LED36, D95 to LED37, D105 to LED38, D118 to LED39, D126 to LED4, D130 to LED40, D142 to LED41, D153 to LED42, D166 to LED43, D176 to LED44, D186 to LED45, D96 to LED46, D106 to LED47, D119 to LED48, D131 to LED49, D138 to LED5, D143 to LED50, D154 to LED51, D167 to LED52, D177 to LED53, D187 to LED54, D97 to LED55, D107 to LED56, D120 to LED57, D132 to LED58, D144 to LED59, D149 to LED6, D155 to LED60, D168 to LED61, D178 to LED62, D188 to LED63, D98 to LED64, D108 to LED65, D121 to LED66, D133 to LED67, D145 to LED68, D156 to LED69, D162 to LED7, D169 to LED70, D179 to LED71, D189 to LED72, D99 to LED73, D109 to LED74, D122 to LED75, D134 to LED76, D146 to LED77, D157 to LED78, D170 to LED79, D172 to LED8, D180 to LED80, D190 to LED81, D100 to LED82, D110 to LED83, D123 to LED84, D135 to LED85, D147 to LED86, D158 to LED87, D171 to LED88, D181 to LED89, D182 to LED9, D191 to LED90, SW15 to MX1, SW66 to MX10, SW80 to MX11, SW17 to MX12, SW35 to MX13, SW53 to MX14, SW67 to MX15, SW81 to MX16, SW2 to MX17, SW18 to MX18, SW36 to MX19, SW33 to MX2, SW54 to MX20, SW68 to MX21, SW82 to MX22, SW3 to MX23, SW19 to MX24, SW37 to MX25, SW55 to MX26, SW69 to MX27, SW4 to MX28, SW20 to MX29, SW51 to MX3, SW38 to MX30, SW56 to MX31, SW70 to MX32, SW5 to MX33, SW21 to MX34, SW39 to MX35, SW57 to MX36, SW71 to MX37, SW83 to MX38, SW6 to MX39, SW65 to MX4, SW22 to MX40, SW40 to MX41, SW58 to MX42, SW72 to MX43, SW7 to MX44, SW23 to MX45, SW41 to MX46, SW59 to MX47, SW73 to MX48, SW8 to MX49, SW79 to MX5, SW24 to MX50, SW42 to MX51, SW60 to MX52, SW74 to MX53, SW9 to MX54, SW25 to MX55, SW43 to MX56, SW61 to MX57, SW75 to MX58, SW84 to MX59, SW1 to MX6, SW10 to MX60, SW26 to MX61, SW44 to MX62, SW62 to MX63, SW76 to MX64, SW85 to MX65, SW11 to MX66, SW27 to MX67, SW45 to MX68, SW63 to MX69, SW16 to MX7, SW12 to MX70, SW28 to MX71, SW46 to MX72, SW86 to MX73, SW13 to MX74, SW29 to MX75, SW47 to MX76, SW64 to MX77, SW77 to MX78, SW87 to MX79, SW34 to MX8, SW14 to MX80, SW30 to MX81, SW48 to MX82, SW88 to MX83, SW31 to MX84, SW49 to MX85, SW78 to MX86, SW89 to MX87, SW32 to MX88, SW50 to MX89, SW52 to MX9, SW90 to MX90, R51 to R1, R4 to R10, R1 to R11, R25 to R12, R30 to R13, R34 to R14, R37 to R15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
Connections:
- net labels removed: COL10, COL11, COL12, COL13, COL14, COL15, COL16, COL17, COL9
Other:
- moved on the sheet: LC1

Commit message: Updated USB hub schematic
Parts:
- removed C22: 10uF, symbol Device:C_Small
- removed C26, C27, C31, C35, C36, C37, C38: 100nF, symbol Device:C_Small
- removed D3, D4, D5, D6, D7, D8, D9: Green/Amber, symbol Device:LED_Dual_2pin
- removed FB1: 100 @ 100 MHz, symbol Device:Ferrite_Bead_Small
- added D10, D12, D14, D16, D4, D6, D8: Green, symbol Device:LED_Small
- added D11, D13, D15, D3, D5, D7, D9: Amber, symbol Device:LED_Small
- added R50: 100k, symbol Device:R_Small
- added R51: 100k, Resistor_SMD:R_0805_2012Metric, symbol Device:R_Small
- C13: value 10uF -> 100nF
- C14: value 4.7uF -> 100nF
- C20: value 100nF -> 10uF; footprint (none) -> Capacitor_SMD:C_0805_2012Metric
- C21: value 10uF -> 100nF; footprint (none) -> Capacitor_SMD:C_0805_2012Metric
- R19, R20: value 100k -> 22
- R23: value 47k -> 10k
Connections:
- net labels added: VBUSM, XRSTJ
- net labels removed: +3.3VA
- wire segments 1988 -> 2020
Other:
- moved on the sheet: C16, C19, R23

Commit message: replaced controller with ATMEGA32U4
Connections:
- net COL0: no longer MX10.1
- net COL1: now also MX10.1; no longer MX21.1
- net COL2: now also MX21.1
- net COL5: no longer MX65.1
- net COL6: now also MX65.1, MX79.1
- net COL7: no longer MX79.1
- net ROT1_ROW: now also KD12.1 (K); no longer KD17.1 (K)
- net ROT2_ROW: now also KD17.1 (K)
- net ROW10: now also KD11.1 (K), KD22.1 (K), KD32.1 (K), KD73.1 (K), KD83.1 (K); no longer KD16.1 (K), KD5.1 (K), KD79.1 (K)
- net ROW2: now also KD18.1 (K); no longer KD12.1 (K)
- net ROW3: now also KD13.1 (K); no longer KD18.1 (K)
- net ROW4: now also KD19.1 (K); no longer KD13.1 (K)
- net ROW5: now also KD14.1 (K); no longer KD19.1 (K)
- net ROW6: now also KD20.1 (K); no longer KD14.1 (K)
- net ROW7: now also KD10.1 (K); no longer KD20.1 (K)
- net ROW8: now also KD21.1 (K), KD65.1 (K); no longer KD27.1 (K)
- net ROW9: now also KD16.1 (K), KD27.1 (K), KD5.1 (K), KD79.1 (K), KD90.1 (K); no longer KD10.1 (K), KD21.1 (K), KD32.1 (K)
- removed net ROW11: KD11.1 (K), KD22.1 (K), KD65.1 (K), KD73.1 (K), KD83.1 (K), KD90.1 (K)
Other:
- moved on the sheet: KD10, KD11, KD12, KD13, KD14, KD16, KD17, KD18, KD19, KD20, KD21, KD22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

Commit message: better USB circuitry
Parts:
- removed C1, C15, C23, C24, C25, C32, C33, C34: 0.1uF, Capacitor_SMD:C_0805_2012Metric, symbol Device:C_Small
- removed C28, C29, C30: 100uF, Capacitor_SMD:C_0805_2012Metric, symbol Device:C_Small
- removed C4: 1uF, Capacitor_SMD:C_0805_2012Metric, symbol Device:C_Small
- removed D1: Yellow, symbol Device:LED_Small
- removed J1: Conn_01x08_Male, symbol Connector:Conn_01x08_Male
- removed J2, J3: USB_A, symbol Connector:USB_A
- removed R11, R26, R27, R28, R35, R36, R37: 330, Resistor_SMD:R_0805_2012Metric, symbol Device:R_Small
- removed R19, R20, R38, R39, R40, R41, R42, R43, R44, R45, R46, R47: 22, Resistor_SMD:R_0805_2012Metric, symbol Device:R_Small
- removed R29, R30, R31, R32, R33, R34: 5.1K, Resistor_SMD:R_0805_2012Metric, symbol Device:R_Small
- removed R8: 150, Resistor_SMD:R_0805_2012Metric, symbol Device:R_Small
- removed TP1, TP2, TP3, TP4: VCC, symbol Connector:TestPoint
- removed U1: AT90USB646-MU, Package_DFN_QFN:QFN-64-1EP_9x9mm_P0.5mm_EP7.5x7.5mm, symbol MCU_Microchip_AVR:AT90USB646-MU
- removed U4, U5, U6, U7, U8, U9: PRTR5V0U2X, symbol random-keyboard-parts:PRTR5V0U2X
- removed USB2, USB3, USB4: HRO-TYPE-C-31-M-12, symbol Type-C:HRO-TYPE-C-31-M-12
- added C2, C?: 0.1uF, Capacitor_SMD:C_0805_2012Metric, symbol Device:C_Small
- added C7: 1uF, Capacitor_SMD:C_0805_2012Metric, symbol Device:C_Small
- added C? (x6): 100uF, Capacitor_SMD:C_0805_2012Metric, symbol Device:C_Small
- added FB? (x7): 500mA, symbol Device:Ferrite_Bead_Small
- added FB? (x7): 60 @ 100MHz, symbol Device:Ferrite_Bead_Small
- added J?: AVR-ISP-6, symbol Connector:AVR-ISP-6
- added J? (x2): USB_A, symbol Connector:USB_A
- added KD84: SOD-123, Diode_SMD:D_SOD-123, symbol Device:D_Small
- added MX84: SCLCK, CherryMX_PCB_KailhSocket_LTST-A683CEGBW:CherryMX_1.00u_PCB_KailhSocket_LTST-A683CEGBW, symbol CherryMX:CherryMX
- added R5, R? (x10): 22, Resistor_SMD:R_0805_2012Metric, symbol Device:R_Small
- added R7: 10k, Resistor_SMD:R_0805_2012Metric, symbol Device:R_Small
- added R? (x6): 5.1K, Resistor_SMD:R_0805_2012Metric, symbol Device:R_Small
- added U1: ATmega32U4-MU, Package_DFN_QFN:QFN-44-1EP_7x7mm_P0.5mm_EP5.2x5.2mm, symbol MCU_Microchip_ATmega:ATmega32U4-MU
- added U? (x6): PRTR5V0U2X, symbol random-keyboard-parts:PRTR5V0U2X
- added USB? (x3): HRO-TYPE-C-31-M-12, symbol Type-C:HRO-TYPE-C-31-M-12
- C11, C12: value 18pF -> 22pF
- R4: value 10k -> 22
- renumbered C2 to C1, C20 to C15, C21 to C16, C19 to C17, C16 to C18, C17 to C20, C18 to C21, C5 to C4, C6 to C5, C7 to C6, KD5 to KD10, KD17 to KD11, KD18 to KD12, KD19 to KD13, KD20 to KD14, KD22 to KD16, KD12 to KD17, KD13 to KD18, KD14 to KD19, KD10 to KD20, KD16 to KD21, KD23 to KD22, KD24 to KD23, KD25 to KD24, KD26 to KD25, KD21 to KD26, KD32 to KD27, KD27 to KD32, KD11 to KD5, KD66 to KD65, KD67 to KD66, KD68 to KD67, KD69 to KD68, KD65 to KD69, KD73 to KD70, KD70 to KD71, KD71 to KD72, KD72 to KD73, KD79 to KD74, KD74 to KD75, KD75 to KD76, KD76 to KD77, KD77 to KD78, KD78 to KD79, KD83 to KD80, KD80 to KD81, KD81 to KD82, KD82 to KD83, KD84 to KD85, KD85 to KD86, KD86 to KD87, KD87 to KD88, KD88 to KD89, KD89 to KD90, KD90 to KD91, MX5 to MX10, MX17 to MX11, MX18 to MX12, MX19 to MX13, MX20 to MX14, MX22 to MX16, MX12 to MX17, MX13 to MX18, MX14 to MX19, MX10 to MX20, MX16 to MX21, MX23 to MX22, MX24 to MX23, MX25 to MX24, MX26 to MX25, MX21 to MX26, MX32 to MX27, MX27 to MX32, MX11 to MX5, MX66 to MX65, MX67 to MX66, MX68 to MX67, MX69 to MX68, MX65 to MX69, MX73 to MX70, MX70 to MX71, MX71 to MX72, MX72 to MX73, MX79 to MX74, MX74 to MX75, MX75 to MX76, MX76 to MX77, MX77 to MX78, MX78 to MX79, MX83 to MX80, MX80 to MX81, MX81 to MX82, MX82 to MX83, MX84 to MX85, MX85 to MX86, MX86 to MX87, MX87 to MX88, MX88 to MX89, MX89 to MX90, MX90 to MX91, R50 to R11, R9 to R12, R10 to R13, R23 to R14, R51 to R15, R12 to R17, R13 to R18, R14 to R19, R15 to R20, R16 to R21, R17 to R22, R18 to R23, R21 to R24, R22 to R25, R24 to R26, R25 to R27, R48 to R50, R49 to R51, R5 to R6, R6 to R8, R7 to R9
Connections:
- net ENCODER_B2 is gone; now on net ENCODER_B1: R3.1
- net +5V: now also C?.1, C?.1, C?.1, C?.1, C?.1, C?.1, C?.1, FB?.1, FB?.1, FB?.1, FB?.1, FB?.1, FB?.1, FB?.1, J?.2 (VCC), U1.14 (VCC), U1.2 (UVCC), U1.24 (AVCC), U1.34 (VCC), U1.44 (AVCC), U1.7 (VBUS); no longer J4.1 (VBUS), U2.4 (VCC), USB1.11 (VBUS), USB1.2 (VBUS)
- net BKL_DATA_IN: now also R1.2, U1.1 (PE6); no longer R1.1
- net COL0: now also U1.8 (PB0)
- net COL1: now also J?.3 (SCK), U1.9 (PB1)
- net COL2: now also J?.4 (MOSI), U1.10 (PB2)
- net COL3: now also J?.1 (MISO), U1.11 (PB3)
- net COL4: now also U1.12 (PB7)
- net COL5: now also U1.20 (PD2)
- net COL6: now also U1.21 (PD3)
- net COL7: now also U1.22 (PD5)
- net COL8: now also MX84.1, U1.25 (PD4)
- net ENCODER_B1: now also U1.40 (PF1)
- net GND: now also R25.1, R26.1, C2.2, C7.2, C?.2, C?.2, C?.2, C?.2, C?.2, C?.2, C?.2, FB?.1, FB?.1, FB?.1, FB?.1, FB?.1, FB?.1, FB?.1, J?.4 (GND), J?.4 (GND), J?.6 (GND), R7.1, R?.1, R?.1, R?.1, R?.1, R?.1, R?.1, U1.15 (GND), U1.23 (GND), U1.35 (GND), U1.43 (GND), U1.45 (GND), U1.5 (UGND), U?.1 (GND), U?.1 (GND), U?.1 (GND), U?.1 (GND), U?.1 (GND), U?.1 (GND), USB?.1 (GND), USB?.1 (GND), USB?.1 (GND), USB?.12 (GND), USB?.12 (GND), USB?.12 (GND); no longer R25.2, R26.2, R4.2
- net HUB_PORT2_D+: now also R?.2
- net HUB_PORT2_D-: now also R?.2
- net HUB_PORT3_D+: now also R?.2
- net HUB_PORT3_D-: now also R?.2
- net HUB_PORT5_D+: now also R?.2
- net HUB_PORT5_D-: now also R?.2
- net HUB_PORT6_D+: now also R?.2
- net HUB_PORT6_D-: now also R?.2
- net HUB_PORT7_D+: now also R?.2
- net HUB_PORT7_D-: now also R?.2
- net KEYBOARD_D+: now also R4.1
- net KEYBOARD_D-: now also R5.1
- net KEYBOARD_RESET: now also J?.5 (~RST), U1.13 (~RESET)
- net KEYBOARD_SCL: now also U1.18 (PD0)
- net KEYBOARD_SDA: now also U1.19 (PD1)
- net KEYBOARD_XTAL1: now also U1.17 (XTAL1)
- net KEYBOARD_XTAL2: now also U1.16 (XTAL2)
- net ROT1_ROW: now also U1.38 (PF5), U1.41 (PF0)
- net ROT2_ROW: now also KD84.1 (K), U1.39 (PF4)
- net ROW10: now also U1.26 (PD6)
- net ROW2: now also U1.37 (PF6)
- net ROW3: now also U1.36 (PF7)
- net ROW4: now also U1.32 (PC7)
- net ROW5: now also U1.31 (PC6)
- net ROW6: now also U1.30 (PB6)
- net ROW7: now also U1.29 (PB5)
- net ROW8: now also U1.28 (PB4)
- net ROW9: now also U1.27 (PD7)
- net at LED90.4 (DIN): no longer R1.2
- net at LED1.2 (DOUT): now also R1.1
- net at USB1.10 (CC2): now also R25.2; no longer R25.1
- net Earth: now reaches USB1.13 (SHIELD)
- net Earth: now also J4.5 (Shield), FB?.2, FB?.2, FB?.2, FB?.2, FB?.2, FB?.2, FB?.2, J?.5 (Shield), J?.5 (Shield), USB?.13 (SHIELD), USB?.13 (SHIELD), USB?.13 (SHIELD)
- net at USB1.4 (CC1): now also R26.2; no longer R26.1
- net at R13.1, U2.3 (IO2), USB1.5 (DN2)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: now also USB1.8 (DP2)
- net at R12.1, U2.2 (IO1), USB1.6 (DP1): no longer USB1.8 (DP2)
- net at J4.2 (D-), R51.1: now also U?.3 (IO2)
- net at J4.3 (D+), R50.1: now also U?.2 (IO1)
- new net: R5.2, U1.3 (D-)
- new net: R7.2, U1.33 (~HWB~/PE2)
- new net: R4.2, U1.4 (D+)
- new net: C2.1, U1.42 (AREF)
- new net: C7.1, U1.6 (UCAP)
- new net: KD84.2 (A), MX84.2
- new net: R?.2, USB?.10 (CC2) (x3)
- new net: R?.2, USB?.4 (CC1) (x3)
- new net: R?.1, U?.3 (IO2), USB?.5 (DN2), USB?.7 (DN1), USB?.8 (DP2) (x3)
- new net: R?.1, U?.2 (IO1), USB?.6 (DP1) (x3)
- new net: J?.3 (D+), R?.1, U?.2 (IO1) (x2)
- new net: J?.2 (D-), R?.1, U?.3 (IO2) (x2)
- new net VCC: FB?.2, FB?.2, FB?.2, FB?.2, FB?.2, FB?.2, FB?.2, J4.1 (VBUS), J?.1 (VBUS), J?.1 (VBUS), U2.4 (VCC), U?.4 (VCC), U?.4 (VCC), U?.4 (VCC), U?.4 (VCC), U?.4 (VCC), U?.4 (VCC), USB1.11 (VBUS), USB1.2 (VBUS), USB?.11 (VBUS), USB?.11 (VBUS), USB?.11 (VBUS), USB?.2 (VBUS), USB?.2 (VBUS), USB?.2 (VBUS)
- no-connect marks 23 -> 9
Other:
- note removed: "Keyboard Signalling LED"
- moved on the sheet: C1, C3, C5, C8, J4, OL1, R1, R12, R13, R25, R26, R50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

Commit message: Assigned footprints to symbols
Parts:
- removed FB? (x7): 500mA, symbol Device:Ferrite_Bead_Small
- removed J?: USB_A, symbol Connector:USB_A
- added F1, F2, F3, F4, F5, F6, F7: 500mA, Fuse:Fuse_1206_3216Metric, symbol Device:Fuse_Small
- added J2: USB_A, random-keyboard-parts:USB-A-Generic, symbol Connector:USB_A
- D10, D11, D12, D13, D14, D15, D16, D2, D3, D4, D5, D6, D7, D8, D9: footprint (none) -> LED_SMD:LED_0402_1005Metric
- FB10, FB11, FB12, FB13, FB14, FB2, FB9: renamed from FB?; footprint (none) -> Inductor_SMD:L_0805_2012Metric
- J1: renamed from J?; footprint (none) -> random-keyboard-parts:Reset_Pretty-Mask
- J3: renamed from J?; footprint (none) -> random-keyboard-parts:USB-A-Generic
- J4: footprint (none) -> random-keyboard-parts:USB-A-Generic
- R11: footprint (none) -> Resistor_SMD:R_0805_2012Metric
- SW1: footprint (none) -> Button_Switch_SMD:SW_SPST_SKQG_WithStem
- U2: footprint (none) -> random-keyboard-parts:SOT143B
- U3: footprint (none) -> custom-footprints:24LC04
- U4, U5, U6, U7, U8, U9: renamed from U?; footprint (none) -> random-keyboard-parts:SOT143B
- USB1: footprint (none) -> Type-C:HRO-TYPE-C-31-M-12-Assembly
- USB2, USB3, USB4: renamed from USB?; footprint (none) -> Type-C:HRO-TYPE-C-31-M-12-Assembly
- Y1, Y2: footprint (none) -> Crystal:Crystal_SMD_3225-4Pin_3.2x2.5mm
- gave numbers to parts that had none: 23
Connections:
- net +5V: now also F1.2, F2.2, F3.2, F4.2, F5.2, F6.2, F7.2
- net Earth: now also J2.5 (Shield)
- net GND: now also C7.1, J2.4 (GND); no longer C7.2
- net KEYBOARD_D-: now also R5.2; no longer R5.1
- net VCC: now also F1.1, F2.1, F3.1, F4.1, F5.1, F6.1, F7.1, J2.1 (VBUS)
- net at U1.3 (D-): now also R5.1; no longer R5.2
- net at U1.6 (UCAP): now also C7.2; no longer C7.1
- net at R38.1, U4.2 (IO1): now also J2.3 (D+)
- net at R39.1, U4.3 (IO2): now also J2.2 (D-)
Other:
- moved on the sheet: C1, C13, C14, C15, C16, C17, C18, C19, C2, C20, C21, C25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

Commit message: MX keys positioned
Parts:
- renumbered ROT2 to ROT1, ROT1 to ROT2
Changed lines of the file:
@@
 Connection ~ 20650 10500
 $Comp
-L Device:Rotary_Encoder_Switch ROT1
+L Device:Rotary_Encoder_Switch ROT2
 U 1 1 616029B6
 P 15350 10850
-F 0 "ROT1" V 15396 10620 50  0000 R CNN
+F 0 "ROT2" V 15396 10620 50  0000 R CNN
 F 1 "Rotary_Encoder_Switch" V 15305 10620 50  0000 R CNN
 F 2 "Rotary_Encoder:RotaryEncoder_Alps_EC11E-Switch_Vertical_H20mm" H 15200 11010 50  0001 C CNN
@@
 $EndComp
 $Comp
-L Device:Rotary_Encoder_Switch ROT2
+L Device:Rotary_Encoder_Switch ROT1
 U 1 1 61614FF0
 P 18050 10850
-F 0 "ROT2" V 18096 10620 50  0000 R CNN
+F 0 "ROT1" V 18096 10620 50  0000 R CNN
 F 1 "Rotary_Encoder_Switch" V 18005 10620 50  0000 R CNN
 F 2 "Rotary_Encoder:RotaryEncoder_Alps_EC11E-Switch_Vertical_H20mm" H 17900 11010 50  0001 C CNN

Commit message: Updated footprints
Parts:
- LED1, LED10, LED11, LED12, LED13, LED14, LED15, LED16, LED17, LED18, LED19, LED2, LED20, LED21, LED22, LED23, LED24, LED25, LED26, LED27, LED28, LED29, LED3, LED30, LED31, LED32, LED33, LED34, LED35, LED36, LED37, LED38, LED39, LED4, LED40, LED41, LED42, LED43, LED44, LED45, LED46, LED47, LED48, LED49, LED5, LED50, LED51, LED52, LED53, LED54, LED55, LED56, LED57, LED58, LED59, LED6, LED60, LED61, LED62, LED63, LED64, LED65, LED66, LED67, LED68, LED69, LED7, LED70, LED71, LED72, LED73, LED74, LED75, LED76, LED77, LED78, LED79, LED8, LED80, LED81, LED82, LED83, LED84, LED85, LED86, LED87, LED88, LED89, LED9, LED90: footprint LED_SMD:LED_WS2812B_PLCC4_5.0x5.0mm_P3.2mm -> LED_SMD:LED_SK6812MINI_PLCC4_3.5x3.5mm_P1.75mm
- MX1, MX10, MX11, MX12, MX13, MX14, MX15, MX17, MX18, MX19, MX2, MX22, MX23, MX24, MX25, MX26, MX27, MX28, MX29, MX3, MX30, MX31, MX32, MX33, MX34, MX35, MX36, MX37, MX39, MX4, MX40, MX41, MX42, MX43, MX44, MX45, MX46, MX47, MX48, MX49, MX50, MX51, MX52, MX53, MX54, MX55, MX56, MX57, MX58, MX6, MX60, MX61, MX62, MX63, MX64, MX65, MX66, MX67, MX68, MX7, MX71, MX72, MX73, MX75, MX80, MX81, MX82, MX83, MX84, MX85, MX86, MX87, MX88, MX89, MX90, MX91: footprint CherryMX_PCB_KailhSocket_LTST-A683CEGBW:CherryMX_1.00u_PCB_KailhSocket_LTST-A683CEGBW -> MX_Only:MXOnly-1U-Hotswap
- MX16, MX21, MX5, MX59, MX69, MX70, MX74, MX8: footprint CherryMX_PCB_KailhSocket_LTST-A683CEGBW:CherryMX_1.00u_PCB_KailhSocket_LTST-A683CEGBW -> MX_Only:MXOnly-1.25U-Hotswap
- MX20, MX78: footprint CherryMX_PCB_KailhSocket_LTST-A683CEGBW:CherryMX_1.00u_PCB_KailhSocket_LTST-A683CEGBW -> MX_Only:MXOnly-2.25U-Hotswap
- MX38: footprint CherryMX_PCB_KailhSocket_LTST-A683CEGBW:CherryMX_1.00u_PCB_KailhSocket_LTST-A683CEGBW -> MX_Only:MXOnly-6.25U-Hotswap
- MX76: footprint CherryMX_PCB_KailhSocket_LTST-A683CEGBW:CherryMX_1.00u_PCB_KailhSocket_LTST-A683CEGBW -> MX_Only:MXOnly-2U-Hotswap
- MX77: footprint CherryMX_PCB_KailhSocket_LTST-A683CEGBW:CherryMX_1.00u_PCB_KailhSocket_LTST-A683CEGBW -> MX_Only:MXOnly-1.5U-Hotswap
- MX79: footprint CherryMX_PCB_KailhSocket_LTST-A683CEGBW:CherryMX_1.00u_PCB_KailhSocket_LTST-A683CEGBW -> MX_Only:MXOnly-2.75U-Hotswap
- MX9: footprint CherryMX_PCB_KailhSocket_LTST-A683CEGBW:CherryMX_1.00u_PCB_KailhSocket_LTST-A683CEGBW -> MX_Only:MXOnly-1.75U-Hotswap

Commit message: Routed rows and some columns
Parts:
- removed F1, F2, F3, F4, F5, F6, F7: 500mA, Fuse:Fuse_1206_3216Metric, symbol Device:Fuse_Small
- removed FB10, FB11, FB12, FB13: 60 @ 100MHz, Inductor_SMD:L_0805_2012Metric, symbol Device:Ferrite_Bead_Small
- added F1, F2, F3, F4, F5, F6, F7: 500mA, Fuse:Fuse_1206_3216Metric, symbol Device:Polyfuse_Small
- added FB1, FB3, FB4, FB5: 60 @ 100MHz, Inductor_SMD:L_0805_2012Metric, symbol Device:Ferrite_Bead_Small
- IC1: footprint FE2.1:LQFP-48_L7.0-W7.0-P0.50-LS9.0-BL -> custom-footprints:FE2.1
- MX8: footprint MX_Only:MXOnly-1.25U-Hotswap -> MX_Only:MXOnly-1.5U-Hotswap
- OL1: footprint Resistor_SMD:R_0805_2012Metric -> kbd:OLED_v2
Connections:
- net +5V: now also F1.1, F2.1, F3.1, F4.1, F5.1, F6.1, F7.1
- net Earth: now also FB14.1, FB1.1, FB3.1, FB4.2, FB5.2; no longer FB14.2
- net GND: now also FB14.2, FB1.2, FB3.2, FB4.1, FB5.1; no longer FB14.1
- net VCC: now also F1.2, F2.2, F3.2, F4.2, F5.2, F6.2, F7.2
- no-connect marks 9 -> 10
Other:
- moved on the sheet: C27, FB14, FB9, J4, R50, R51, U6
