File: PCB/_autosave-custom_keyboard (3).sch (KiCad schematic (older format))
At the start: 503 parts, among them IC1 FE2.1, J1 USB_A, J2 USB_A, J3 USB_A, J4 Conn_01x03_Male, J5 AVR-ISP-6, Q1 DTC123J, SW1 SW_Push, U1 24LC02, U10 PRTR5V0U2X, U11 XC6206P332MR, U12 74LVC1G34, U2 PRTR5V0U2X, U3 PRTR5V0U2X, U4 PRTR5V0U2X, U5 PRTR5V0U2X, U6 PRTR5V0U2X, U7 PRTR5V0U2X, U8 PRTR5V0U2X, U9 STM32F303CBTx, Y1 12MHz, Y2 8MHz, Y3 32.768kHZ

Commit message: Placed some of the LEDs
Parts:
- IC1: footprint FE2.1:LQFP-48_L7.0-W7.0-P0.50-LS9.0-BL -> custom-footprints:FE2.1
- LED1, LED10, LED11, LED12, LED13, LED14, LED15, LED16, LED17, LED18, LED19, LED2, LED20, LED21, LED22, LED23, LED24, LED25, LED26, LED27, LED28, LED29, LED3, LED30, LED31, LED32, LED33, LED34, LED35, LED36, LED37, LED38, LED39, LED4, LED40, LED41, LED42, LED43, LED44, LED45, LED46, LED47, LED48, LED49, LED5, LED50, LED51, LED52, LED53, LED54, LED55, LED56, LED57, LED58, LED59, LED6, LED60, LED61, LED62, LED63, LED64, LED65, LED66, LED67, LED68, LED69, LED7, LED70, LED71, LED72, LED73, LED74, LED75, LED76, LED77, LED78, LED79, LED8, LED80, LED81, LED82, LED83, LED84, LED85, LED86, LED87, LED88, LED89, LED9, LED90: footprint LED_SMD:LED_SK6812MINI_PLCC4_3.5x3.5mm_P1.75mm -> custom-footprints:SK6812MINI
