File: PCB/custom_keyboard (3).sch (KiCad schematic (older format))
At the start: 498 parts, among them IC1 FE2.1, J1 USB_A, SW1 ESC, SW10 F9, SW11 F10, SW12 F11, SW13 F12, SW14 PSCR, SW15 M1, SW16 `/~, SW17 1, SW18 2, SW19 3, SW2 F1, SW20 4, SW21 5, SW22 6, SW23 7, SW24 8, SW25 9, SW26 0, SW27 -/_, SW28 =/+, SW29 BACKSPACE, SW3 F2, SW30 INS, SW31 HOME, SW32 PGUP, SW33 M2, SW34 TAB, SW35 Q, SW36 W, SW37 E, SW38 R, SW39 T, SW4 F3, SW40 Y, SW41 U, SW42 I, SW43 O, SW44 P, SW45 [/{, SW46 ]/}, SW47 \\, SW48 DELETE, SW49 END, SW5 F4, SW50 PGDN, SW51 M3, SW52 CAPS, SW53 A, SW54 S, SW55 D, SW56 F, SW57 G, SW58 H, SW59 J, SW6 F5, SW60 K, SW61 L, SW62 ;/:, SW63 '/\", SW64 ENTER, SW65 M4, SW66 LSHIFT, SW67 Z, SW68 X, SW69 C, SW7 F6, SW70 V, SW71 B, SW72 N, SW73 M, SW74 ,/<, SW75 ./>, SW76 /, SW77 RSHIFT, SW78 UP, SW79 M5, SW8 F7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

Commit message: Updated USB Hub schematic
Parts:
- removed C9: 10uF, Capacitor_SMD:C_0805_2012Metric, symbol Device:C_Small
- removed D? (x7): Amber, symbol Device:LED_Small
- added C117, C118, C119, C121, C122, C123, C124, C125, C74, C85, C96: 100nF, Capacitor_SMD:C_0805_2012Metric, symbol Device:C_Small
- added C120: 10uF, Capacitor_SMD:C_0805_2012Metric, symbol Device:C_Small
- added J?: Conn_01x03_Male, symbol Connector:Conn_01x03_Male
- gave numbers to parts that had none: 82
Connections:
- net +1V8: now also C119.1, C123.2, C85.2; no longer IC1.21 (VD_PLL)
- net +3V3: now also IC1.21 (VD_PLL), R11.1, C117.1, C118.2, C120.1, C121.2, C124.1, C125.1, C74.1, C96.1, J?.1 (Pin_1); no longer R11.2, U4.1 (VBAT)
- net GND: now also C5.1, C6.1, R10.2, C117.2, C118.1, C119.2, C120.2, C121.1, C122.2, C123.1, C124.2, C125.2, C74.2, C85.1, C96.2, J?.3 (Pin_3); no longer C11.1, C22.2
- net KEYBOARD_RESET: now also U4.7 (NRST)
- net EXTRA_1: now reaches U4.2 (PC13)
- net EXTRA_1: now also J?.2 (Pin_2)
- net XRSTJ: now reaches IC1.40 (XRSTJ)
- net XRSTJ: now also R11.2, C122.1; no longer R11.1
- net VBUSM: now reaches IC1.41 (VBUSM), R10.1, R9.2
- new net: C11.1, C22.2
Other:
- moved on the sheet: C1, C23, C4, C5, C6, C7, C8, D124, D136, D148, D161, D193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

Commit message: Reannotated the keyboard and LED matrices
Parts:
- gave numbers to parts that had none: 1
- renumbered D15 to KD1, D66 to KD10, D80 to KD11, D17 to KD12, D35 to KD13, D53 to KD14, D67 to KD15, D81 to KD16, D2 to KD17, D18 to KD18, D36 to KD19, D33 to KD2, D54 to KD20, D68 to KD21, D82 to KD22, D3 to KD23, D19 to KD24, D37 to KD25, D55 to KD26, D69 to KD27, D4 to KD28, D20 to KD29, D51 to KD3, D38 to KD30, D56 to KD31, D70 to KD32, D5 to KD33, D21 to KD34, D39 to KD35, D57 to KD36, D71 to KD37, D83 to KD38, D6 to KD39, D65 to KD4, D22 to KD40, D40 to KD41, D58 to KD42, D72 to KD43, D7 to KD44, D23 to KD45, D41 to KD46, D59 to KD47, D73 to KD48, D8 to KD49, D79 to KD5, D24 to KD50, D42 to KD51, D60 to KD52, D74 to KD53, D9 to KD54, D25 to KD55, D43 to KD56, D61 to KD57, D75 to KD58, D84 to KD59, D1 to KD6, D10 to KD60, D26 to KD61, D44 to KD62, D62 to KD63, D76 to KD64, D85 to KD65, D11 to KD66, D27 to KD67, D45 to KD68, D63 to KD69, D16 to KD7, D12 to KD70, D28 to KD71, D46 to KD72, D86 to KD73, D13 to KD74, D29 to KD75, D47 to KD76, D64 to KD77, D77 to KD78, D87 to KD79, D34 to KD8, D14 to KD80, D30 to KD81, D48 to KD82, D88 to KD83, D31 to KD84, D49 to KD85, D78 to KD86, D89 to KD87, D32 to KD88, D50 to KD89, D52 to KD9, D90 to KD90, C12 to LC1, C13 to LC10, C26 to LC11, C36 to LC12, C52 to LC13, C63 to LC14, C76 to LC15, C87 to LC16, C98 to LC17, C108 to LC18, C14 to LC19, C25 to LC2, C27 to LC20, C37 to LC21, C53 to LC22, C64 to LC23, C77 to LC24, C88 to LC25, C99 to LC26, C109 to LC27, C15 to LC28, C28 to LC29, C35 to LC3, C38 to LC30, C54 to LC31, C65 to LC32, C78 to LC33, C89 to LC34, C100 to LC35, C110 to LC36, C16 to LC37, C29 to LC38, C39 to LC39, C51 to LC4, C55 to LC40, C66 to LC41, C79 to LC42, C90 to LC43, C101 to LC44, C111 to LC45, C17 to LC46, C30 to LC47, C40 to LC48, C56 to LC49, C62 to LC5, C67 to LC50, C80 to LC51, C91 to LC52, C102 to LC53, C112 to LC54, C18 to LC55, C31 to LC56, C41 to LC57, C57 to LC58, C68 to LC59, C75 to LC6, C81 to LC60, C92 to LC61, C103 to LC62, C113 to LC63, C19 to LC64, C32 to LC65, C42 to LC66, C58 to LC67, C69 to LC68, C82 to LC69, C86 to LC7, C93 to LC70, C104 to LC71, C114 to LC72, C20 to LC73, C33 to LC74, C43 to LC75, C59 to LC76, C70 to LC77, C83 to LC78, C94 to LC79, C97 to LC8, C105 to LC80, C115 to LC81, C21 to LC82, C34 to LC83, C44 to LC84, C60 to LC85, C71 to LC86, C84 to LC87, C95 to LC88, C106 to LC89, C107 to LC9, C116 to LC90, D91 to LED1, D92 to LED10, D102 to LED11, D115 to LED12, D127 to LED13, D139 to LED14, D150 to LED15, D163 to LED16, D173 to LED17, D183 to LED18, D93 to LED19, D101 to LED2, D103 to LED20, D116 to LED21, D128 to LED22, D140 to LED23, D151 to LED24, D164 to LED25, D174 to LED26, D184 to LED27, D94 to LED28, D104 to LED29, D114 to LED3, D117 to LED30, D129 to LED31, D141 to LED32, D152 to LED33, D165 to LED34, D175 to LED35, D185 to LED36, D95 to LED37, D105 to LED38, D118 to LED39, D126 to LED4, D130 to LED40, D142 to LED41, D153 to LED42, D166 to LED43, D176 to LED44, D186 to LED45, D96 to LED46, D106 to LED47, D119 to LED48, D131 to LED49, D138 to LED5, D143 to LED50, D154 to LED51, D167 to LED52, D177 to LED53, D187 to LED54, D97 to LED55, D107 to LED56, D120 to LED57, D132 to LED58, D144 to LED59, D149 to LED6, D155 to LED60, D168 to LED61, D178 to LED62, D188 to LED63, D98 to LED64, D108 to LED65, D121 to LED66, D133 to LED67, D145 to LED68, D156 to LED69, D162 to LED7, D169 to LED70, D179 to LED71, D189 to LED72, D99 to LED73, D109 to LED74, D122 to LED75, D134 to LED76, D146 to LED77, D157 to LED78, D170 to LED79, D172 to LED8, D180 to LED80, D190 to LED81, D100 to LED82, D110 to LED83, D123 to LED84, D135 to LED85, D147 to LED86, D158 to LED87, D171 to LED88, D181 to LED89, D182 to LED9, D191 to LED90, SW15 to MX1, SW66 to MX10, SW80 to MX11, SW17 to MX12, SW35 to MX13, SW53 to MX14, SW67 to MX15, SW81 to MX16, SW2 to MX17, SW18 to MX18, SW36 to MX19, SW33 to MX2, SW54 to MX20, SW68 to MX21, SW82 to MX22, SW3 to MX23, SW19 to MX24, SW37 to MX25, SW55 to MX26, SW69 to MX27, SW4 to MX28, SW20 to MX29, SW51 to MX3, SW38 to MX30, SW56 to MX31, SW70 to MX32, SW5 to MX33, SW21 to MX34, SW39 to MX35, SW57 to MX36, SW71 to MX37, SW83 to MX38, SW6 to MX39, SW65 to MX4, SW22 to MX40, SW40 to MX41, SW58 to MX42, SW72 to MX43, SW7 to MX44, SW23 to MX45, SW41 to MX46, SW59 to MX47, SW73 to MX48, SW8 to MX49, SW79 to MX5, SW24 to MX50, SW42 to MX51, SW60 to MX52, SW74 to MX53, SW9 to MX54, SW25 to MX55, SW43 to MX56, SW61 to MX57, SW75 to MX58, SW84 to MX59, SW1 to MX6, SW10 to MX60, SW26 to MX61, SW44 to MX62, SW62 to MX63, SW76 to MX64, SW85 to MX65, SW11 to MX66, SW27 to MX67, SW45 to MX68, SW63 to MX69, SW16 to MX7, SW12 to MX70, SW28 to MX71, SW46 to MX72, SW86 to MX73, SW13 to MX74, SW29 to MX75, SW47 to MX76, SW64 to MX77, SW77 to MX78, SW87 to MX79, SW34 to MX8, SW14 to MX80, SW30 to MX81, SW48 to MX82, SW88 to MX83, SW31 to MX84, SW49 to MX85, SW78 to MX86, SW89 to MX87, SW32 to MX88, SW50 to MX89, SW52 to MX9, SW90 to MX90
Connections:
- net +3V3: now also U4.1 (VBAT)

Commit message: Assigned footprints to symbols
Parts:
- D124, D136, D148, D160, D161, D193, D195, D197: footprint (none) -> LED_SMD:LED_0402_1005Metric
- DRST1: footprint (none) -> Diode_SMD:D_SOD-123
- F1, F2, F3, F4, F5, F6, F7: footprint (none) -> Fuse:Fuse_1206_3216Metric
- FB1, FB2, FB3, FB4, FB5, FB6, FB7: footprint (none) -> Inductor_SMD:L_0805_2012Metric
- J1, J3, J4: footprint (none) -> random-keyboard-parts:USB-A-Generic
- J2: footprint (none) -> random-keyboard-parts:Reset_Pretty-Mask
- J5: footprint (none) -> Connector_JST:JST_GH_SM03B-GHS-TB_1x03-1MP_P1.25mm_Horizontal
- Q1: footprint (none) -> Package_TO_SOT_SMD:SOT-23
- SW91: footprint (none) -> random-keyboard-parts:SKQG-1155865
- U1: footprint (none) -> custom-footprints:24LC04
- U10, U11, U12, U2, U6, U7, U8, U9: footprint (none) -> random-keyboard-parts:SOT143B
- U5: footprint (none) -> Package_TO_SOT_SMD:SOT-353_SC-70-5
- USB1, USB2, USB3, USB4: footprint (none) -> Type-C:HRO-TYPE-C-31-M-12-Assembly
- Y1, Y2, Y3: footprint (none) -> Crystal:Crystal_SMD_3225-4Pin_3.2x2.5mm

Commit message: Created pcb and mapped keyboard matrix
Parts:
- MX1: renamed from MX6; footprint CherryMX_PCB_KailhSocket_LTST-A683CEGBW:CherryMX_1.00u_PCB_KailhSocket_LTST-A683CEGBW -> MX_Only:MXOnly-1U-Hotswap
- MX10: renamed from MX60; footprint CherryMX_PCB_KailhSocket_LTST-A683CEGBW:CherryMX_1.00u_PCB_KailhSocket_LTST-A683CEGBW -> MX_Only:MXOnly-1U-Hotswap
- MX11: renamed from MX66; footprint CherryMX_PCB_KailhSocket_LTST-A683CEGBW:CherryMX_1.00u_PCB_KailhSocket_LTST-A683CEGBW -> MX_Only:MXOnly-1U-Hotswap
- MX12: renamed from MX70; footprint CherryMX_PCB_KailhSocket_LTST-A683CEGBW:CherryMX_1.00u_PCB_KailhSocket_LTST-A683CEGBW -> MX_Only:MXOnly-1U-Hotswap
- MX13: renamed from MX74; footprint CherryMX_PCB_KailhSocket_LTST-A683CEGBW:CherryMX_1.00u_PCB_KailhSocket_LTST-A683CEGBW -> MX_Only:MXOnly-1U-Hotswap
- MX14: renamed from MX80; footprint CherryMX_PCB_KailhSocket_LTST-A683CEGBW:CherryMX_1.00u_PCB_KailhSocket_LTST-A683CEGBW -> MX_Only:MXOnly-1U-Hotswap
- MX15: renamed from MX1; footprint CherryMX_PCB_KailhSocket_LTST-A683CEGBW:CherryMX_1.00u_PCB_KailhSocket_LTST-A683CEGBW -> MX_Only:MXOnly-1U-Hotswap
- MX16: renamed from MX7; footprint CherryMX_PCB_KailhSocket_LTST-A683CEGBW:CherryMX_1.00u_PCB_KailhSocket_LTST-A683CEGBW -> MX_Only:MXOnly-1U-Hotswap
- MX17: renamed from MX12; footprint CherryMX_PCB_KailhSocket_LTST-A683CEGBW:CherryMX_1.00u_PCB_KailhSocket_LTST-A683CEGBW -> MX_Only:MXOnly-1U-Hotswap
- MX18, MX90: footprint CherryMX_PCB_KailhSocket_LTST-A683CEGBW:CherryMX_1.00u_PCB_KailhSocket_LTST-A683CEGBW -> MX_Only:MXOnly-1U-Hotswap
- MX19: renamed from MX24; footprint CherryMX_PCB_KailhSocket_LTST-A683CEGBW:CherryMX_1.00u_PCB_KailhSocket_LTST-A683CEGBW -> MX_Only:MXOnly-1U-Hotswap
- MX2: renamed from MX17; footprint CherryMX_PCB_KailhSocket_LTST-A683CEGBW:CherryMX_1.00u_PCB_KailhSocket_LTST-A683CEGBW -> MX_Only:MXOnly-1U-Hotswap
- MX20: renamed from MX29; footprint CherryMX_PCB_KailhSocket_LTST-A683CEGBW:CherryMX_1.00u_PCB_KailhSocket_LTST-A683CEGBW -> MX_Only:MXOnly-1U-Hotswap
- MX21: renamed from MX34; footprint CherryMX_PCB_KailhSocket_LTST-A683CEGBW:CherryMX_1.00u_PCB_KailhSocket_LTST-A683CEGBW -> MX_Only:MXOnly-1U-Hotswap
- MX22: renamed from MX40; footprint CherryMX_PCB_KailhSocket_LTST-A683CEGBW:CherryMX_1.00u_PCB_KailhSocket_LTST-A683CEGBW -> MX_Only:MXOnly-1U-Hotswap
- MX23: renamed from MX45; footprint CherryMX_PCB_KailhSocket_LTST-A683CEGBW:CherryMX_1.00u_PCB_KailhSocket_LTST-A683CEGBW -> MX_Only:MXOnly-1U-Hotswap
- MX24: renamed from MX50; footprint CherryMX_PCB_KailhSocket_LTST-A683CEGBW:CherryMX_1.00u_PCB_KailhSocket_LTST-A683CEGBW -> MX_Only:MXOnly-1U-Hotswap
- MX25: renamed from MX55; footprint CherryMX_PCB_KailhSocket_LTST-A683CEGBW:CherryMX_1.00u_PCB_KailhSocket_LTST-A683CEGBW -> MX_Only:MXOnly-1U-Hotswap
- MX26: renamed from MX61; footprint CherryMX_PCB_KailhSocket_LTST-A683CEGBW:CherryMX_1.00u_PCB_KailhSocket_LTST-A683CEGBW -> MX_Only:MXOnly-1U-Hotswap
- MX27: renamed from MX67; footprint CherryMX_PCB_KailhSocket_LTST-A683CEGBW:CherryMX_1.00u_PCB_KailhSocket_LTST-A683CEGBW -> MX_Only:MXOnly-1U-Hotswap
- MX28: renamed from MX71; footprint CherryMX_PCB_KailhSocket_LTST-A683CEGBW:CherryMX_1.00u_PCB_KailhSocket_LTST-A683CEGBW -> MX_Only:MXOnly-1U-Hotswap
- MX29: renamed from MX75; footprint CherryMX_PCB_KailhSocket_LTST-A683CEGBW:CherryMX_1.00u_PCB_KailhSocket_LTST-A683CEGBW -> MX_Only:MXOnly-2U-Hotswap
- MX3: renamed from MX23; footprint CherryMX_PCB_KailhSocket_LTST-A683CEGBW:CherryMX_1.00u_PCB_KailhSocket_LTST-A683CEGBW -> MX_Only:MXOnly-1U-Hotswap
- MX30: renamed from MX81; footprint CherryMX_PCB_KailhSocket_LTST-A683CEGBW:CherryMX_1.00u_PCB_KailhSocket_LTST-A683CEGBW -> MX_Only:MXOnly-1U-Hotswap
- MX31: renamed from MX84; footprint CherryMX_PCB_KailhSocket_LTST-A683CEGBW:CherryMX_1.00u_PCB_KailhSocket_LTST-A683CEGBW -> MX_Only:MXOnly-1U-Hotswap
- MX32: renamed from MX88; footprint CherryMX_PCB_KailhSocket_LTST-A683CEGBW:CherryMX_1.00u_PCB_KailhSocket_LTST-A683CEGBW -> MX_Only:MXOnly-1U-Hotswap
- MX33: renamed from MX2; footprint CherryMX_PCB_KailhSocket_LTST-A683CEGBW:CherryMX_1.00u_PCB_KailhSocket_LTST-A683CEGBW -> MX_Only:MXOnly-1U-Hotswap
- MX34: renamed from MX8; footprint CherryMX_PCB_KailhSocket_LTST-A683CEGBW:CherryMX_1.00u_PCB_KailhSocket_LTST-A683CEGBW -> MX_Only:MXOnly-1.5U-Hotswap
- MX35: renamed from MX13; footprint CherryMX_PCB_KailhSocket_LTST-A683CEGBW:CherryMX_1.00u_PCB_KailhSocket_LTST-A683CEGBW -> MX_Only:MXOnly-1U-Hotswap
- MX36: renamed from MX19; footprint CherryMX_PCB_KailhSocket_LTST-A683CEGBW:CherryMX_1.00u_PCB_KailhSocket_LTST-A683CEGBW -> MX_Only:MXOnly-1U-Hotswap
- MX37: renamed from MX25; footprint CherryMX_PCB_KailhSocket_LTST-A683CEGBW:CherryMX_1.00u_PCB_KailhSocket_LTST-A683CEGBW -> MX_Only:MXOnly-1U-Hotswap
- MX38: renamed from MX30; footprint CherryMX_PCB_KailhSocket_LTST-A683CEGBW:CherryMX_1.00u_PCB_KailhSocket_LTST-A683CEGBW -> MX_Only:MXOnly-1U-Hotswap
- MX39: renamed from MX35; footprint CherryMX_PCB_KailhSocket_LTST-A683CEGBW:CherryMX_1.00u_PCB_KailhSocket_LTST-A683CEGBW -> MX_Only:MXOnly-1U-Hotswap
- MX4: renamed from MX28; footprint CherryMX_PCB_KailhSocket_LTST-A683CEGBW:CherryMX_1.00u_PCB_KailhSocket_LTST-A683CEGBW -> MX_Only:MXOnly-1U-Hotswap
- MX40: renamed from MX41; footprint CherryMX_PCB_KailhSocket_LTST-A683CEGBW:CherryMX_1.00u_PCB_KailhSocket_LTST-A683CEGBW -> MX_Only:MXOnly-1U-Hotswap
- MX41: renamed from MX46; footprint CherryMX_PCB_KailhSocket_LTST-A683CEGBW:CherryMX_1.00u_PCB_KailhSocket_LTST-A683CEGBW -> MX_Only:MXOnly-1U-Hotswap
- MX42: renamed from MX51; footprint CherryMX_PCB_KailhSocket_LTST-A683CEGBW:CherryMX_1.00u_PCB_KailhSocket_LTST-A683CEGBW -> MX_Only:MXOnly-1U-Hotswap
- MX43: renamed from MX56; footprint CherryMX_PCB_KailhSocket_LTST-A683CEGBW:CherryMX_1.00u_PCB_KailhSocket_LTST-A683CEGBW -> MX_Only:MXOnly-1U-Hotswap
- MX44: renamed from MX62; footprint CherryMX_PCB_KailhSocket_LTST-A683CEGBW:CherryMX_1.00u_PCB_KailhSocket_LTST-A683CEGBW -> MX_Only:MXOnly-1U-Hotswap
- MX45: renamed from MX68; footprint CherryMX_PCB_KailhSocket_LTST-A683CEGBW:CherryMX_1.00u_PCB_KailhSocket_LTST-A683CEGBW -> MX_Only:MXOnly-1U-Hotswap
- MX46: renamed from MX72; footprint CherryMX_PCB_KailhSocket_LTST-A683CEGBW:CherryMX_1.00u_PCB_KailhSocket_LTST-A683CEGBW -> MX_Only:MXOnly-1U-Hotswap
- MX47: renamed from MX76; footprint CherryMX_PCB_KailhSocket_LTST-A683CEGBW:CherryMX_1.00u_PCB_KailhSocket_LTST-A683CEGBW -> MX_Only:MXOnly-1.5U-Hotswap
- MX48: renamed from MX82; footprint CherryMX_PCB_KailhSocket_LTST-A683CEGBW:CherryMX_1.00u_PCB_KailhSocket_LTST-A683CEGBW -> MX_Only:MXOnly-1U-Hotswap
- MX49: renamed from MX85; footprint CherryMX_PCB_KailhSocket_LTST-A683CEGBW:CherryMX_1.00u_PCB_KailhSocket_LTST-A683CEGBW -> MX_Only:MXOnly-1U-Hotswap
- MX5: renamed from MX33; footprint CherryMX_PCB_KailhSocket_LTST-A683CEGBW:CherryMX_1.00u_PCB_KailhSocket_LTST-A683CEGBW -> MX_Only:MXOnly-1U-Hotswap
- MX50: renamed from MX89; footprint CherryMX_PCB_KailhSocket_LTST-A683CEGBW:CherryMX_1.00u_PCB_KailhSocket_LTST-A683CEGBW -> MX_Only:MXOnly-1U-Hotswap
- MX51: renamed from MX3; footprint CherryMX_PCB_KailhSocket_LTST-A683CEGBW:CherryMX_1.00u_PCB_KailhSocket_LTST-A683CEGBW -> MX_Only:MXOnly-1U-Hotswap
- MX52: renamed from MX9; footprint CherryMX_PCB_KailhSocket_LTST-A683CEGBW:CherryMX_1.00u_PCB_KailhSocket_LTST-A683CEGBW -> MX_Only:MXOnly-1.75U-Hotswap
- MX53: renamed from MX14; footprint CherryMX_PCB_KailhSocket_LTST-A683CEGBW:CherryMX_1.00u_PCB_KailhSocket_LTST-A683CEGBW -> MX_Only:MXOnly-1U-Hotswap
- MX54: renamed from MX20; footprint CherryMX_PCB_KailhSocket_LTST-A683CEGBW:CherryMX_1.00u_PCB_KailhSocket_LTST-A683CEGBW -> MX_Only:MXOnly-1U-Hotswap
- MX55: renamed from MX26; footprint CherryMX_PCB_KailhSocket_LTST-A683CEGBW:CherryMX_1.00u_PCB_KailhSocket_LTST-A683CEGBW -> MX_Only:MXOnly-1U-Hotswap
- MX56: renamed from MX31; footprint CherryMX_PCB_KailhSocket_LTST-A683CEGBW:CherryMX_1.00u_PCB_KailhSocket_LTST-A683CEGBW -> MX_Only:MXOnly-1U-Hotswap
- MX57: renamed from MX36; footprint CherryMX_PCB_KailhSocket_LTST-A683CEGBW:CherryMX_1.00u_PCB_KailhSocket_LTST-A683CEGBW -> MX_Only:MXOnly-1U-Hotswap
- MX58: renamed from MX42; footprint CherryMX_PCB_KailhSocket_LTST-A683CEGBW:CherryMX_1.00u_PCB_KailhSocket_LTST-A683CEGBW -> MX_Only:MXOnly-1U-Hotswap
- MX59: renamed from MX47; footprint CherryMX_PCB_KailhSocket_LTST-A683CEGBW:CherryMX_1.00u_PCB_KailhSocket_LTST-A683CEGBW -> MX_Only:MXOnly-1U-Hotswap
- MX6: renamed from MX39; footprint CherryMX_PCB_KailhSocket_LTST-A683CEGBW:CherryMX_1.00u_PCB_KailhSocket_LTST-A683CEGBW -> MX_Only:MXOnly-1U-Hotswap
- MX60: renamed from MX52; footprint CherryMX_PCB_KailhSocket_LTST-A683CEGBW:CherryMX_1.00u_PCB_KailhSocket_LTST-A683CEGBW -> MX_Only:MXOnly-1U-Hotswap
- MX61: renamed from MX57; footprint CherryMX_PCB_KailhSocket_LTST-A683CEGBW:CherryMX_1.00u_PCB_KailhSocket_LTST-A683CEGBW -> MX_Only:MXOnly-1U-Hotswap
- MX62: renamed from MX63; footprint CherryMX_PCB_KailhSocket_LTST-A683CEGBW:CherryMX_1.00u_PCB_KailhSocket_LTST-A683CEGBW -> MX_Only:MXOnly-1U-Hotswap
- MX63: renamed from MX69; footprint CherryMX_PCB_KailhSocket_LTST-A683CEGBW:CherryMX_1.00u_PCB_KailhSocket_LTST-A683CEGBW -> MX_Only:MXOnly-1U-Hotswap
- MX64: renamed from MX77; footprint CherryMX_PCB_KailhSocket_LTST-A683CEGBW:CherryMX_1.00u_PCB_KailhSocket_LTST-A683CEGBW -> MX_Only:MXOnly-2.25U-Hotswap
- MX65: renamed from MX4; footprint CherryMX_PCB_KailhSocket_LTST-A683CEGBW:CherryMX_1.00u_PCB_KailhSocket_LTST-A683CEGBW -> MX_Only:MXOnly-1U-Hotswap
- MX66: renamed from MX10; footprint CherryMX_PCB_KailhSocket_LTST-A683CEGBW:CherryMX_1.00u_PCB_KailhSocket_LTST-A683CEGBW -> MX_Only:MXOnly-2.25U-Hotswap
- MX67: renamed from MX15; footprint CherryMX_PCB_KailhSocket_LTST-A683CEGBW:CherryMX_1.00u_PCB_KailhSocket_LTST-A683CEGBW -> MX_Only:MXOnly-1U-Hotswap
- MX68: renamed from MX21; footprint CherryMX_PCB_KailhSocket_LTST-A683CEGBW:CherryMX_1.00u_PCB_KailhSocket_LTST-A683CEGBW -> MX_Only:MXOnly-1U-Hotswap
- MX69: renamed from MX27; footprint CherryMX_PCB_KailhSocket_LTST-A683CEGBW:CherryMX_1.00u_PCB_KailhSocket_LTST-A683CEGBW -> MX_Only:MXOnly-1U-Hotswap
- MX7: renamed from MX44; footprint CherryMX_PCB_KailhSocket_LTST-A683CEGBW:CherryMX_1.00u_PCB_KailhSocket_LTST-A683CEGBW -> MX_Only:MXOnly-1U-Hotswap
- MX70: renamed from MX32; footprint CherryMX_PCB_KailhSocket_LTST-A683CEGBW:CherryMX_1.00u_PCB_KailhSocket_LTST-A683CEGBW -> MX_Only:MXOnly-1U-Hotswap
- MX71: renamed from MX37; footprint CherryMX_PCB_KailhSocket_LTST-A683CEGBW:CherryMX_1.00u_PCB_KailhSocket_LTST-A683CEGBW -> MX_Only:MXOnly-1U-Hotswap
- MX72: renamed from MX43; footprint CherryMX_PCB_KailhSocket_LTST-A683CEGBW:CherryMX_1.00u_PCB_KailhSocket_LTST-A683CEGBW -> MX_Only:MXOnly-1U-Hotswap
- MX73: renamed from MX48; footprint CherryMX_PCB_KailhSocket_LTST-A683CEGBW:CherryMX_1.00u_PCB_KailhSocket_LTST-A683CEGBW -> MX_Only:MXOnly-1U-Hotswap
- MX74: renamed from MX53; footprint CherryMX_PCB_KailhSocket_LTST-A683CEGBW:CherryMX_1.00u_PCB_KailhSocket_LTST-A683CEGBW -> MX_Only:MXOnly-1U-Hotswap
- MX75: renamed from MX58; footprint CherryMX_PCB_KailhSocket_LTST-A683CEGBW:CherryMX_1.00u_PCB_KailhSocket_LTST-A683CEGBW -> MX_Only:MXOnly-1U-Hotswap
- MX76: renamed from MX64; footprint CherryMX_PCB_KailhSocket_LTST-A683CEGBW:CherryMX_1.00u_PCB_KailhSocket_LTST-A683CEGBW -> MX_Only:MXOnly-1U-Hotswap
- MX77: renamed from MX78; footprint CherryMX_PCB_KailhSocket_LTST-A683CEGBW:CherryMX_1.00u_PCB_KailhSocket_LTST-A683CEGBW -> MX_Only:MXOnly-2.75U-Hotswap
- MX78: renamed from MX86; footprint CherryMX_PCB_KailhSocket_LTST-A683CEGBW:CherryMX_1.00u_PCB_KailhSocket_LTST-A683CEGBW -> MX_Only:MXOnly-1U-Hotswap
- MX79: renamed from MX5; footprint CherryMX_PCB_KailhSocket_LTST-A683CEGBW:CherryMX_1.00u_PCB_KailhSocket_LTST-A683CEGBW -> MX_Only:MXOnly-1U-Hotswap
- MX8: renamed from MX49; footprint CherryMX_PCB_KailhSocket_LTST-A683CEGBW:CherryMX_1.00u_PCB_KailhSocket_LTST-A683CEGBW -> MX_Only:MXOnly-1U-Hotswap
- MX80: renamed from MX11; footprint CherryMX_PCB_KailhSocket_LTST-A683CEGBW:CherryMX_1.00u_PCB_KailhSocket_LTST-A683CEGBW -> MX_Only:MXOnly-1.25U-Hotswap
- MX81: renamed from MX16; footprint CherryMX_PCB_KailhSocket_LTST-A683CEGBW:CherryMX_1.00u_PCB_KailhSocket_LTST-A683CEGBW -> MX_Only:MXOnly-1.25U-Hotswap
- MX82: renamed from MX22; footprint CherryMX_PCB_KailhSocket_LTST-A683CEGBW:CherryMX_1.00u_PCB_KailhSocket_LTST-A683CEGBW -> MX_Only:MXOnly-1.25U-Hotswap
- MX83: renamed from MX38; footprint CherryMX_PCB_KailhSocket_LTST-A683CEGBW:CherryMX_1.00u_PCB_KailhSocket_LTST-A683CEGBW -> MX_Only:MXOnly-6.25U-Hotswap
- MX84: renamed from MX59; footprint CherryMX_PCB_KailhSocket_LTST-A683CEGBW:CherryMX_1.00u_PCB_KailhSocket_LTST-A683CEGBW -> MX_Only:MXOnly-1.25U-Hotswap
- MX85: renamed from MX65; footprint CherryMX_PCB_KailhSocket_LTST-A683CEGBW:CherryMX_1.00u_PCB_KailhSocket_LTST-A683CEGBW -> MX_Only:MXOnly-1.25U-Hotswap
- MX86: renamed from MX73; footprint CherryMX_PCB_KailhSocket_LTST-A683CEGBW:CherryMX_1.00u_PCB_KailhSocket_LTST-A683CEGBW -> MX_Only:MXOnly-1.25U-Hotswap
- MX87: renamed from MX79; footprint CherryMX_PCB_KailhSocket_LTST-A683CEGBW:CherryMX_1.00u_PCB_KailhSocket_LTST-A683CEGBW -> MX_Only:MXOnly-1.25U-Hotswap
- MX88: renamed from MX83; footprint CherryMX_PCB_KailhSocket_LTST-A683CEGBW:CherryMX_1.00u_PCB_KailhSocket_LTST-A683CEGBW -> MX_Only:MXOnly-1U-Hotswap
- MX89: renamed from MX87; footprint CherryMX_PCB_KailhSocket_LTST-A683CEGBW:CherryMX_1.00u_PCB_KailhSocket_LTST-A683CEGBW -> MX_Only:MXOnly-1U-Hotswap
- MX9: renamed from MX54; footprint CherryMX_PCB_KailhSocket_LTST-A683CEGBW:CherryMX_1.00u_PCB_KailhSocket_LTST-A683CEGBW -> MX_Only:MXOnly-1U-Hotswap
- OL1: footprint Resistor_SMD:R_0805_2012Metric -> kbd:OLED_v2
- renumbered C6 to C1, C74 to C10, C119 to C11, C121 to C12, C4 to C13, C7 to C14, C131 to C15, C118 to C16, C120 to C17, C23 to C18, C117 to C19, C5 to C2, C96 to C20, C50 to C21, C61 to C22, C72 to C23, C45 to C24, C46 to C25, C47 to C26, C48 to C27, C73 to C28, C128 to C29, C129 to C3, C24 to C30, C2 to C31, C3 to C32, C9 to C33, C10 to C34, C11 to C35, C22 to C36, C126 to C37, C49 to C38, C127 to C39, C122 to C4, C1 to C40, C8 to C41, C124 to C5, C130 to C6, C125 to C7, C85 to C8, C123 to C9, D111 to D1, D160 to D10, D112 to D2, D124 to D3, D136 to D4, D148 to D5, D161 to D6, D193 to D7, D195 to D8, D197 to D9, F5 to F2, F6 to F3, F7 to F4, F4 to F5, F2 to F6, F3 to F7, FB5 to FB2, FB6 to FB3, FB7 to FB4, FB4 to FB5, FB2 to FB6, FB3 to FB7, J3 to J2, J4 to J3, J5 to J4, J2 to J5, KD6 to KD1, KD60 to KD10, KD66 to KD11, KD70 to KD12, KD74 to KD13, KD80 to KD14, KD1 to KD15, KD7 to KD16, KD12 to KD17, KD24 to KD19, KD17 to KD2, KD29 to KD20, KD34 to KD21, KD40 to KD22, KD45 to KD23, KD50 to KD24, KD55 to KD25, KD61 to KD26, KD67 to KD27, KD71 to KD28, KD75 to KD29, KD23 to KD3, KD81 to KD30, KD84 to KD31, KD88 to KD32, KD2 to KD33, KD8 to KD34, KD13 to KD35, KD19 to KD36, KD25 to KD37, KD30 to KD38, KD35 to KD39, KD28 to KD4, KD41 to KD40, KD46 to KD41, KD51 to KD42, KD56 to KD43, KD62 to KD44, KD68 to KD45, KD72 to KD46, KD76 to KD47, KD82 to KD48, KD85 to KD49, KD33 to KD5, KD89 to KD50, KD3 to KD51, KD9 to KD52, KD14 to KD53, KD20 to KD54, KD26 to KD55, KD31 to KD56, KD36 to KD57, KD42 to KD58, KD47 to KD59, KD39 to KD6, KD52 to KD60, KD57 to KD61, KD63 to KD62, KD69 to KD63, KD77 to KD64, KD4 to KD65, KD10 to KD66, KD15 to KD67, KD21 to KD68, KD27 to KD69, KD44 to KD7, KD32 to KD70, KD37 to KD71, KD43 to KD72, KD48 to KD73, KD53 to KD74, KD58 to KD75, KD64 to KD76, KD78 to KD77, KD86 to KD78, KD5 to KD79, KD49 to KD8, KD11 to KD80, KD16 to KD81, KD22 to KD82, KD38 to KD83, KD59 to KD84, KD65 to KD85, KD73 to KD86, KD79 to KD87, KD83 to KD88, KD87 to KD89, KD54 to KD9, LC82 to LC10, LC2 to LC11, LC11 to LC12, LC20 to LC13, LC29 to LC14, LC38 to LC15, LC47 to LC16, LC56 to LC17, LC65 to LC18, LC74 to LC19, LC10 to LC2, LC83 to LC20, LC3 to LC21, LC12 to LC22, LC21 to LC23, LC30 to LC24, LC39 to LC25, LC48 to LC26, LC57 to LC27, LC66 to LC28, LC75 to LC29, LC19 to LC3, LC84 to LC30, LC4 to LC31, LC13 to LC32, LC22 to LC33, LC31 to LC34, LC40 to LC35, LC49 to LC36, LC58 to LC37, LC67 to LC38, LC76 to LC39, LC28 to LC4, LC85 to LC40, LC5 to LC41, LC14 to LC42, LC23 to LC43, LC32 to LC44, LC41 to LC45, LC50 to LC46, LC59 to LC47, LC68 to LC48, LC77 to LC49, LC37 to LC5, LC86 to LC50, LC6 to LC51, LC15 to LC52, LC24 to LC53, LC33 to LC54, LC42 to LC55, LC51 to LC56, LC60 to LC57, LC69 to LC58, LC78 to LC59, LC46 to LC6, LC87 to LC60, LC7 to LC61, LC16 to LC62, LC25 to LC63, LC34 to LC64, LC43 to LC65, LC52 to LC66, LC61 to LC67, LC70 to LC68, LC79 to LC69, LC55 to LC7, LC88 to LC70, LC8 to LC71, LC17 to LC72, LC26 to LC73, LC35 to LC74, LC44 to LC75, LC53 to LC76, LC62 to LC77, LC71 to LC78, LC80 to LC79, LC64 to LC8, LC89 to LC80, LC9 to LC81, LC18 to LC82, LC27 to LC83, LC36 to LC84, LC45 to LC85, LC54 to LC86, LC63 to LC87, LC72 to LC88, LC81 to LC89, LC73 to LC9, LED82 to LED10, LED2 to LED11, LED11 to LED12, LED20 to LED13, LED29 to LED14, LED38 to LED15, LED47 to LED16, LED56 to LED17, LED65 to LED18, LED74 to LED19, LED10 to LED2, LED83 to LED20, LED3 to LED21, LED12 to LED22, LED21 to LED23, LED30 to LED24, LED39 to LED25, LED48 to LED26, LED57 to LED27, LED66 to LED28, LED75 to LED29, LED19 to LED3, LED84 to LED30, LED4 to LED31, LED13 to LED32, LED22 to LED33, LED31 to LED34, LED40 to LED35, LED49 to LED36, LED58 to LED37, LED67 to LED38, LED76 to LED39, LED28 to LED4, LED85 to LED40, LED5 to LED41, LED14 to LED42, LED23 to LED43, LED32 to LED44, LED41 to LED45, LED50 to LED46, LED59 to LED47, LED68 to LED48, LED77 to LED49, LED37 to LED5, LED86 to LED50, LED6 to LED51, LED15 to LED52, LED24 to LED53, LED33 to LED54, LED42 to LED55, LED51 to LED56, LED60 to LED57, LED69 to LED58, LED78 to LED59, LED46 to LED6, LED87 to LED60, LED7 to LED61, LED16 to LED62, LED25 to LED63, LED34 to LED64, LED43 to LED65, LED52 to LED66, LED61 to LED67, LED70 to LED68, LED79 to LED69, LED55 to LED7, LED88 to LED70, LED8 to LED71, LED17 to LED72, LED26 to LED73, LED35 to LED74, LED44 to LED75, LED53 to LED76, LED62 to LED77, LED71 to LED78, LED80 to LED79, LED64 to LED8, LED89 to LED80, LED9 to LED81, LED18 to LED82, LED27 to LED83, LED36 to LED84, LED45 to LED85, LED54 to LED86, LED63 to LED87, LED72 to LED88, LED81 to LED89, LED73 to LED9, R4 to R1, R40 to R10, R41 to R11, R15 to R12, R43 to R13, R44 to R14, R17 to R15, R25 to R16, R26 to R17, R27 to R18, R28 to R19, R3 to R2, R29 to R20, R14 to R21, R30 to R22, R36 to R23, R39 to R24, R21 to R25, R24 to R26, R34 to R27, R37 to R28, R31 to R29, R5 to R3, R32 to R30, R38 to R31, R16 to R32, R19 to R33, R22 to R34, R42 to R35, R45 to R36, R13 to R37, R18 to R38, R33 to R39, R2 to R4, R35 to R40, R49 to R41, R20 to R42, R23 to R43, R12 to R44, R1 to R45, R8 to R46, R51 to R47, R11 to R5, R9 to R6, R10 to R7, R6 to R8, R7 to R9, SW91 to SW1, U8 to U10, U3 to U11, U5 to U12, U10 to U3, U11 to U4, U12 to U5, U9 to U6, U6 to U8, U4 to U9, USB4 to USB2, USB2 to USB3, USB3 to USB4
Connections:
- net ENCODER_B1: now also R18.1; no longer R20.1
- net ENCODER_B2: now also R20.1; no longer R18.1
- net GND: now also C35.1, C36.2

Commit message: Placed some of the LEDs
Parts:
- IC1: footprint FE2.1:LQFP-48_L7.0-W7.0-P0.50-LS9.0-BL -> custom-footprints:FE2.1
- LED1, LED10, LED11, LED12, LED13, LED14, LED15, LED16, LED17, LED18, LED19, LED2, LED20, LED21, LED22, LED23, LED24, LED25, LED26, LED27, LED28, LED29, LED3, LED30, LED31, LED32, LED33, LED34, LED35, LED36, LED37, LED38, LED39, LED4, LED40, LED41, LED42, LED43, LED44, LED45, LED46, LED47, LED48, LED49, LED5, LED50, LED51, LED52, LED53, LED54, LED55, LED56, LED57, LED58, LED59, LED6, LED60, LED61, LED62, LED63, LED64, LED65, LED66, LED67, LED68, LED69, LED7, LED70, LED71, LED72, LED73, LED74, LED75, LED76, LED77, LED78, LED79, LED8, LED80, LED81, LED82, LED83, LED84, LED85, LED86, LED87, LED88, LED89, LED9, LED90: footprint LED_SMD:LED_WS2812B_PLCC4_5.0x5.0mm_P3.2mm -> custom-footprints:WS2812BMINI_With_Hole

Commit message: New version with combined footprint
Parts:
- LED1, LED10, LED11, LED12, LED13, LED14, LED15, LED16, LED17, LED18, LED19, LED2, LED20, LED21, LED22, LED23, LED24, LED25, LED26, LED27, LED28, LED29, LED3, LED30, LED31, LED32, LED33, LED34, LED35, LED36, LED37, LED38, LED39, LED4, LED40, LED41, LED42, LED43, LED44, LED45, LED46, LED47, LED48, LED49, LED5, LED50, LED51, LED52, LED53, LED54, LED55, LED56, LED57, LED58, LED59, LED6, LED60, LED61, LED62, LED63, LED64, LED65, LED66, LED67, LED68, LED69, LED7, LED70, LED71, LED72, LED73, LED74, LED75, LED76, LED77, LED78, LED79, LED8, LED80, LED81, LED82, LED83, LED84, LED85, LED86, LED87, LED88, LED89, LED9, LED90: footprint custom-footprints:WS2812BMINI_With_Hole -> custom-footprints:SK6812MINI

Commit message: Updated footprints
Parts:
- LED1, LED10, LED11, LED12, LED13, LED14, LED15, LED16, LED17, LED18, LED19, LED2, LED20, LED21, LED22, LED23, LED24, LED25, LED26, LED27, LED28, LED29, LED3, LED30, LED31, LED32, LED33, LED34, LED35, LED36, LED37, LED38, LED39, LED4, LED40, LED41, LED42, LED43, LED44, LED45, LED46, LED47, LED48, LED49, LED5, LED50, LED51, LED52, LED53, LED54, LED55, LED56, LED57, LED58, LED59, LED6, LED60, LED61, LED62, LED63, LED64, LED65, LED66, LED67, LED68, LED69, LED7, LED70, LED71, LED72, LED73, LED74, LED75, LED76, LED77, LED78, LED79, LED8, LED80, LED81, LED82, LED83, LED84, LED85, LED86, LED87, LED88, LED89, LED9, LED90: footprint custom-footprints:SK6812MINI -> LED_SMD:LED_SK6812MINI_PLCC4_3.5x3.5mm_P1.75mm
