File: PCB/custom_keyboard (4).sch (KiCad schematic (older format))
At the start: 417 parts, among them IC1 FE2.1, J1 USB_A, J2 Conn_01x03_Male, J3 USB_A, J4 USB_A, J5 AVR-ISP-6, Q1 DTC123J, SW1 SW_Push, U1 24LC02, U10 PRTR5V0U2X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

Commit message: Mapped columns to microcontroller
Connections:
- wire segments 2519 -> 2521
Changed lines of the file:
@@
 Text GLabel 2100 2450 1    50   Input ~ 0
 COL0
-Text GLabel 5150 17000 2    50   Input ~ 0
+Text GLabel 5500 18000 2    50   Input ~ 0
 COL3
 Text GLabel 5500 18100 2    50   Input ~ 0
@@
 Text GLabel 3450 17000 0    50   Input ~ 0
 COL0
-Text GLabel 3450 16800 0    50   Input ~ 0
+Text GLabel 5150 17200 2    50   Input ~ 0
 COL9
-Text GLabel 5150 17500 2    50   Input ~ 0
+Text GLabel 5150 17100 2    50   Input ~ 0
 COL8
-Text GLabel 5150 17400 2    50   Input ~ 0
+Text GLabel 5150 17000 2    50   Input ~ 0
 COL7
-Text GLabel 5150 17300 2    50   Input ~ 0
+Text GLabel 5150 16900 2    50   Input ~ 0
 COL6
-Text GLabel 5150 17200 2    50   Input ~ 0
+Text GLabel 5150 16800 2    50   Input ~ 0
 COL5
-Text GLabel 5150 17100 2    50   Input ~ 0
+Text GLabel 5150 16700 2    50   Input ~ 0
 COL4
-Text GLabel 3450 16700 0    50   Input ~ 0
+Text GLabel 5150 17300 2    50   Input ~ 0
 COL10
-Text GLabel 5150 16700 2    50   Input ~ 0
+Text GLabel 5150 17400 2    50   Input ~ 0
 COL11
-Text GLabel 5500 18000 2    50   Input ~ 0
+Text GLabel 3450 17900 0    50   Input ~ 0
 COL17
-Text GLabel 5150 16800 2    50   Input ~ 0
+Text GLabel 3450 17800 0    50   Input ~ 0
 COL16
-Text GLabel 5150 16900 2    50   Input ~ 0
+Text GLabel 3450 17700 0    50   Input ~ 0
 COL15
-Text GLabel 3450 17800 0    50   Input ~ 0
+Text GLabel 3450 16900 0    50   Input ~ 0
 COL14
-Text GLabel 3450 17700 0    50   Input ~ 0
+Text GLabel 3450 16800 0    50   Input ~ 0
 COL13
-Text GLabel 3450 16900 0    50   Input ~ 0
+Text GLabel 3450 16700 0    50   Input ~ 0
 COL12
 Text GLabel 3450 17200 0    50   Input ~ 0
@@
 Text GLabel 3450 17600 0    50   Input ~ 0
 ROW0
-Text GLabel 3450 17900 0    50   Input ~ 0
+Text GLabel 5150 17500 2    50   Input ~ 0
 BKL_DATA_IN_3V3
 Text GLabel 3450 18000 0    50   Input ~ 0
@@
 HUB_LED1
 Wire Wire Line
-	25900 4000 25900 2450
+	25900 4000 25900 3200
 Wire Wire Line
 	2200 3200 2100 3200
@@
 Wire Wire Line
 	13200 20200 13600 20200
+Wire Wire Line
+	26000 3200 25900 3200
+Connection ~ 25900 3200
+Wire Wire Line
+	25900 3200 25900 2450
 $EndSCHEMATC

Commit message: Routed Rotary Encoders
Parts:
- added R39, R40, R48, R49: 10k, Resistor_SMD:R_0805_2012Metric, symbol Device:R_Small
Connections:
- wire segments 2521 -> 2533
Other:
- moved on the sheet: C7, C8, D2, D3, R14, R15, ROT1, ROT2
