File: PCB/custom_keyboard (f303, fe2.1).kicad_pcb (KiCad board)
At the start: 2 copper layers, 390.5 x 135.7 mm, 373 parts, among them IC1 FE2.1, J2 Conn_01x03_Male, Q1 DTC123J, SW1 SW_Push, U1 24LC02BT-I/SN, U10 PRTR5V0U2X, U11 XC6206P332MR, U12 74LVC1G34, U2 PRTR5V0U2X, U4 PRTR5V0U2X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

Commit message: Made some traces shorter
Routing:
- net BKL_DATA_IN_3V3: track 664.6 -> 330.9 mm
- net ENCODER_B1: track 641.3 -> 352.3 mm
- net COL16: track 362.4 -> 262.0 mm
- net GND: track 694.8 -> 652.0 mm, vias 291 -> 304
- net Earth: track 489.0 -> 518.4 mm, vias 30 -> 26
- net ENCODER_A: track 642.4 -> 639.6 mm
- net COL0: track 330.5 -> 333.2 mm
- net COL2: track 310.0 -> 312.3 mm
- net COL1: track 315.7 -> 317.2 mm
- net ROW2: track 619.8 -> 618.4 mm
- net ROW4: track 558.7 -> 557.2 mm
- net ROW3: track 516.1 -> 514.7 mm
- net COL17: track 302.4 -> 303.1 mm
- net ROW5: track 546.7 -> 546.0 mm
- net COL15: track 271.2 -> 271.9 mm

Commit message: Tidied up some traces
Parts:
- moved C15 1.77 mm to (202.8, 269.1)
- moved C22 1.77 mm to (202.0, 273.0)
- moved DRST1 1.77 mm to (196.4, 270.7)
- moved Q1 1.77 mm to (199.6, 268.3)
- moved R30 1.77 mm to (199.6, 273.0)
- moved SW1 1.77 mm to (192.1, 270.7)
Routing:
- net GND: track 652.0 -> 640.8 mm, vias 304 -> 305
- net EXTRA_1: track 55.6 -> 52.8 mm
- net +3V3: track 287.9 -> 289.1 mm
- net KEYBOARD_D+: track 183.8 -> 184.5 mm
- net KEYBOARD_D-: track 178.6 -> 179.3 mm
- net BOOT0: track 90.0 -> 90.5 mm

Commit message: Draft 1-2
Parts:
- moved SW1 5.61 mm to (192.9, 276.2), turned to 180 degrees
- moved DRST1 1.98 mm to (194.5, 270.7), turned to 180 degrees
- moved D2 1.77 mm to (83.3, 177.0), turned to 180 degrees
Routing:
- net Net-(D2-Pad2): track 2.41 -> 5.82 mm
- net Net-(DRST1-Pad2): track 9.08 -> 11.7 mm
- net ROT1_ROW: track 661.2 -> 658.7 mm
- net +3V3: track 289.1 -> 290.6 mm
- net BOOT0: track 90.5 -> 91.7 mm
- net GND: vias 305 -> 304

Commit message: Added a ferrite bead
Parts:
- added FB8: 60 @ 100 MHz, Inductor_SMD:L_0805_2012Metric, B.Cu at (238.5, 155.6)
- moved FB7 0.92 mm to (456.4, 243.5)
- moved FB4 0.79 mm to (416.7, 157.2)
- moved FB6 0.79 mm to (121.4, 157.2)
- moved C18 0.40 mm to (261.1, 282.2)
- moved C19 0.40 mm to (258.7, 282.2)
Connections:
- R19 pad 1: D+ -> Net-(R19-Pad1)
- R2 pad 1: D- -> Net-(R2-Pad1)
- R20 pad 1: D- -> Net-(R20-Pad1)
- R24 pad 1: D+ -> Net-(R24-Pad1)
- R25 pad 1: D- -> Net-(R25-Pad1)
- R3 pad 2: D- -> Net-(R3-Pad2)
- R31 pad 1: D- -> Net-(R31-Pad1)
- R33 pad 1: D+ -> Net-(R33-Pad1)
- R34 pad 1: D+ -> Net-(R34-Pad1)
- R37 pad 1: D- -> Net-(R37-Pad1)
- R4 pad 1: D+ -> Net-(R4-Pad1)
- R43 pad 1: KEYBOARD_D- -> Net-(R43-Pad1)
- R44 pad 1: KEYBOARD_D+ -> Net-(R44-Pad1)
- R45 pad 1: D+ -> Net-(R45-Pad1)
- R46 pad 1: D- -> Net-(R46-Pad1)
- R6 pad 2: D+ -> Net-(R6-Pad2)
- U10 pad 2: D+ -> Net-(R45-Pad1)
- U10 pad 3: D- -> Net-(R46-Pad1)
- U2 pad 2: D+ -> Net-(R4-Pad1)
- U2 pad 3: D- -> Net-(R2-Pad1)
- U4 pad 2: D+ -> Net-(R19-Pad1)
- U4 pad 3: D- -> Net-(R20-Pad1)
- U5 pad 2: D+ -> Net-(R24-Pad1)
- U5 pad 3: D- -> Net-(R25-Pad1)
- U6 pad 2: D+ -> Net-(R33-Pad1)
- U6 pad 3: D- -> Net-(R31-Pad1)
- U9 pad 32: KEYBOARD_D- -> Net-(R43-Pad1)
- U9 pad 33: KEYBOARD_D+ -> Net-(R44-Pad1)
- USB1 pad 5: D- -> Net-(R2-Pad1)
- USB1 pad 6: D+ -> Net-(R4-Pad1)
- USB1 pad 7: D- -> Net-(R2-Pad1)
- USB1 pad 8: D+ -> Net-(R4-Pad1)
- USB2 pad 5: D- -> Net-(R31-Pad1)
- USB2 pad 6: D+ -> Net-(R33-Pad1)
- USB2 pad 7: D- -> Net-(R31-Pad1)
- USB2 pad 8: D+ -> Net-(R33-Pad1)
- USB3 pad 2: D- -> Net-(R37-Pad1)
- USB3 pad 3: D+ -> Net-(R34-Pad1)
- USB4 pad 2: D- -> Net-(R46-Pad1)
- USB4 pad 3: D+ -> Net-(R45-Pad1)
- USB5 pad 5: D- -> Net-(R3-Pad2)
- USB5 pad 6: D+ -> Net-(R6-Pad2)
- USB5 pad 7: D- -> Net-(R3-Pad2)
- USB5 pad 8: D+ -> Net-(R6-Pad2)
- USB6 pad 2: D- -> Net-(R25-Pad1)
- USB6 pad 3: D+ -> Net-(R24-Pad1)
- USB7 pad 5: D- -> Net-(R20-Pad1)
- USB7 pad 6: D+ -> Net-(R19-Pad1)
- USB7 pad 7: D- -> Net-(R20-Pad1)
- USB7 pad 8: D+ -> Net-(R19-Pad1)
Routing:
- net D+: track 339.8 -> 0.00 mm
- net D-: track 335.7 -> 0.00 mm
- net Net-(R4-Pad1): track 0.00 -> 240.2 mm
- net Net-(R2-Pad1): track 0.00 -> 238.9 mm
- net Net-(R19-Pad1): track 0.00 -> 22.0 mm
- net Net-(R6-Pad2): track 0.00 -> 21.1 mm
- net Net-(R20-Pad1): track 0.00 -> 20.8 mm
- net Net-(R3-Pad2): track 0.00 -> 19.8 mm
- net Net-(R33-Pad1): track 0.00 -> 19.4 mm
- net Net-(R31-Pad1): track 0.00 -> 18.2 mm
- net Net-(R46-Pad1): track 0.00 -> 13.3 mm
- net Net-(R37-Pad1): track 0.00 -> 12.5 mm
- net Net-(R24-Pad1): track 0.00 -> 12.4 mm
- net Net-(R34-Pad1): track 0.00 -> 12.4 mm
- net Net-(R25-Pad1): track 0.00 -> 12.4 mm
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Other:
- board text added: "JLCJLCJLCJLC"
