File: PCB/custom_keyboard (f303, fe2.1).kicad_pcb (KiCad board)
At the start: 2 copper layers, 395.3 x 138.1 mm, 444 parts, among them IC1 FE2.1, J2 Conn_01x03_Male, J5 AVR-ISP-6, Q1 DTC123J, SW1 SW_Push, U1 24LC02BT-I/SN, U10 PRTR5V0U2X, U11 XC6206P332MR, U12 74LVC1G34, U13 XC6206P332MR, U14 MIC2505, U15 MIC2505, U2 PRTR5V0U2X, U4 PRTR5V0U2X, U5 PRTR5V0U2X, U6 PRTR5V0U2X, U8 PRTR5V0U2X, U9 STM32F303CBT6, Y1 8MHz, Y2 32.768KHz, Y3 12MHz

Commit message: connected microcontroller testpoints in PCB
Parts:
- removed TP21, TP22, TP23, TP25: TestPoint_Small, TestPoint:TestPoint_THTPad_D1.0mm_Drill0.5mm
- added D1: Red, LED_SMD:LED_0805_2012Metric, B.Cu at (77.8, 193.7)
- added D4: Red, LED_SMD:LED_0805_2012Metric, B.Cu at (127.8, 165.9)
- added D5: Red, LED_SMD:LED_0805_2012Metric, B.Cu at (449.2, 248.4)
- added D6: Red, LED_SMD:LED_0805_2012Metric, B.Cu at (298.4, 157.9)
- added D7: Red, LED_SMD:LED_0805_2012Metric, B.Cu at (423.0, 165.1)
- added D8: Red, LED_SMD:LED_0805_2012Metric, B.Cu at (455.6, 176.2)
- added D9: Red, LED_SMD:LED_0805_2012Metric, B.Cu at (232.6, 157.9)
- added R57: 330, Resistor_SMD:R_0805_2012Metric, B.Cu at (127.8, 169.9)
- added R58: 330, Resistor_SMD:R_0805_2012Metric, B.Cu at (77.8, 197.6)
- added R59: 330, Resistor_SMD:R_0805_2012Metric, B.Cu at (450.0, 245.3)
- added R60: 330, Resistor_SMD:R_0805_2012Metric, B.Cu at (294.5, 157.9)
- added R61: 330, Resistor_SMD:R_0805_2012Metric, B.Cu at (423.0, 169.1)
- added R62: 330, Resistor_SMD:R_0805_2012Metric, B.Cu at (458.0, 173.0)
- added R63: 330, Resistor_SMD:R_0805_2012Metric, B.Cu at (232.6, 160.3)
- added TP3: TestPoint_Small, TestPoint:TestPoint_THTPad_D1.0mm_Drill0.5mm, B.Cu at (254.0, 273.0)
- moved TP20 95.0 mm to (292.9, 272.2), turned to 90 degrees
- moved TP19 94.6 mm to (289.7, 269.9)
- moved TP18 91.9 mm to (287.3, 269.9), turned to 180 degrees
- moved TP39 87.5 mm to (296.1, 273.8), turned to 180 degrees
- moved TP36 87.1 mm to (292.1, 269.9), turned to 180 degrees
- moved TP40 86.6 mm to (297.6, 276.2), turned to 270 degrees
- moved TP37 68.7 mm to (279.4, 282.6), turned to 180 degrees
- moved TP38 66.6 mm to (277.0, 282.6)
- moved TP24 63.6 mm to (256.4, 272.2)
- moved TP26 62.0 mm to (258.0, 276.2)
- moved TP27 59.4 mm to (249.2, 273.8)
- moved TP8 22.2 mm to (79.4, 169.1)
- moved C25 5.32 mm to (127.8, 173.0), turned to 0 degrees
- moved F4 3.55 mm to (425.4, 168.3)
- moved F6 3.55 mm to (130.2, 169.1)
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Connections:
- C11 pad 2: +5V -> PORT1-4_PWR
- C12 pad 2: +5V -> PORT1-4_PWR
- C45 pad 1: +5V -> PORT1-4_PWR
- C47 pad 1: +5V -> PORT1-4_PWR
- FB16 pad 1: +5V -> PORT1-4_PWR
- FB16 pad 2: +5V -> PORT1-4_PWR
- FB8 pad 1: +5V -> PORT1-4_PWR
- FB8 pad 2: +5V -> PORT1-4_PWR
- IC1 pad 8: +5V -> PORT1-4_PWR
- LC1 pad 2: +5V -> PORT1-4_PWR
- LC10 pad 2: +5V -> PORT1-4_PWR
- LC11 pad 2: +5V -> PORT1-4_PWR
- LC12 pad 2: +5V -> PORT1-4_PWR
- LC13 pad 2: +5V -> PORT1-4_PWR
- LC14 pad 2: +5V -> PORT1-4_PWR
- LC15 pad 2: +5V -> PORT1-4_PWR
- LC16 pad 2: +5V -> PORT1-4_PWR
- LC17 pad 2: +5V -> PORT1-4_PWR
- LC18 pad 2: +5V -> PORT1-4_PWR
- LC19 pad 2: +5V -> PORT1-4_PWR
- LC2 pad 2: +5V -> PORT1-4_PWR
- LC20 pad 2: +5V -> PORT1-4_PWR
- LC21 pad 2: +5V -> PORT1-4_PWR
- LC22 pad 2: +5V -> PORT1-4_PWR
- LC23 pad 2: +5V -> PORT1-4_PWR
- LC24 pad 2: +5V -> PORT1-4_PWR
- LC25 pad 2: +5V -> PORT1-4_PWR
- LC26 pad 2: +5V -> PORT1-4_PWR
- LC27 pad 2: +5V -> PORT1-4_PWR
- LC28 pad 2: +5V -> PORT1-4_PWR
- LC29 pad 2: +5V -> PORT1-4_PWR
- LC3 pad 2: +5V -> PORT1-4_PWR
- LC30 pad 2: +5V -> PORT1-4_PWR
- LC31 pad 2: +5V -> PORT1-4_PWR
- LC32 pad 2: +5V -> PORT1-4_PWR
- LC33 pad 2: +5V -> PORT1-4_PWR
- LC34 pad 2: +5V -> PORT1-4_PWR
- LC35 pad 2: +5V -> PORT1-4_PWR
- LC36 pad 2: +5V -> PORT1-4_PWR
- LC37 pad 2: +5V -> PORT1-4_PWR
- LC38 pad 2: +5V -> PORT1-4_PWR
- LC39 pad 2: +5V -> PORT1-4_PWR
- LC4 pad 2: +5V -> PORT1-4_PWR
- LC40 pad 2: +5V -> PORT1-4_PWR
- LC41 pad 2: +5V -> PORT1-4_PWR
- LC42 pad 2: +5V -> PORT1-4_PWR
- LC43 pad 2: +5V -> PORT1-4_PWR
- LC44 pad 2: +5V -> PORT1-4_PWR
- LC45 pad 2: +5V -> PORT1-4_PWR
- LC46 pad 2: +5V -> PORT1-4_PWR
- LC47 pad 2: +5V -> PORT1-4_PWR
- LC48 pad 2: +5V -> PORT1-4_PWR
- LC49 pad 2: +5V -> PORT1-4_PWR
- LC5 pad 2: +5V -> PORT1-4_PWR
- LC50 pad 2: +5V -> PORT1-4_PWR
- LC51 pad 2: +5V -> PORT1-4_PWR
- LC52 pad 2: +5V -> PORT1-4_PWR
- LC53 pad 2: +5V -> PORT1-4_PWR
- LC54 pad 2: +5V -> PORT1-4_PWR
- LC55 pad 2: +5V -> PORT1-4_PWR
- LC56 pad 2: +5V -> PORT1-4_PWR
- LC57 pad 2: +5V -> PORT1-4_PWR
- LC58 pad 2: +5V -> PORT1-4_PWR
- LC59 pad 2: +5V -> PORT1-4_PWR
- LC6 pad 2: +5V -> PORT1-4_PWR
- LC60 pad 2: +5V -> PORT1-4_PWR
- LC61 pad 2: +5V -> PORT1-4_PWR
- LC62 pad 2: +5V -> PORT1-4_PWR
- LC63 pad 2: +5V -> PORT1-4_PWR
- LC64 pad 2: +5V -> PORT1-4_PWR
- LC65 pad 2: +5V -> PORT1-4_PWR
- LC66 pad 2: +5V -> PORT1-4_PWR
- LC67 pad 2: +5V -> PORT1-4_PWR
- LC68 pad 2: +5V -> PORT1-4_PWR
- LC69 pad 2: +5V -> PORT1-4_PWR
- LC7 pad 2: +5V -> PORT1-4_PWR
- LC70 pad 2: +5V -> PORT1-4_PWR
- LC71 pad 2: +5V -> PORT1-4_PWR
- LC72 pad 2: +5V -> PORT1-4_PWR
- LC73 pad 2: +5V -> PORT1-4_PWR
- LC74 pad 2: +5V -> PORT1-4_PWR
- LC75 pad 2: +5V -> PORT1-4_PWR
- LC76 pad 2: +5V -> PORT1-4_PWR
- LC77 pad 2: +5V -> PORT1-4_PWR
- LC78 pad 2: +5V -> PORT1-4_PWR
- LC79 pad 2: +5V -> PORT1-4_PWR
- LC8 pad 2: +5V -> PORT1-4_PWR
- LC80 pad 2: +5V -> PORT1-4_PWR
- LC81 pad 2: +5V -> PORT1-4_PWR
- LC82 pad 2: +5V -> PORT1-4_PWR
- LC83 pad 2: +5V -> PORT1-4_PWR
- LC84 pad 2: +5V -> PORT1-4_PWR
- LC85 pad 2: +5V -> PORT1-4_PWR
- LC86 pad 2: +5V -> PORT1-4_PWR
- LC87 pad 2: +5V -> PORT1-4_PWR
- LC88 pad 2: +5V -> PORT1-4_PWR
- LC89 pad 2: +5V -> PORT1-4_PWR
- LC9 pad 2: +5V -> PORT1-4_PWR
- LC90 pad 2: +5V -> PORT1-4_PWR
- MX1 pad 6: +5V -> PORT1-4_PWR
- MX10 pad 6: +5V -> PORT1-4_PWR
- MX11 pad 6: +5V -> PORT1-4_PWR
- MX12 pad 6: +5V -> PORT1-4_PWR
- MX13 pad 6: +5V -> PORT1-4_PWR
- MX14 pad 6: +5V -> PORT1-4_PWR
- MX15 pad 6: +5V -> PORT1-4_PWR
- MX16 pad 6: +5V -> PORT1-4_PWR
- MX17 pad 6: +5V -> PORT1-4_PWR
- MX18 pad 6: +5V -> PORT1-4_PWR
- MX19 pad 6: +5V -> PORT1-4_PWR
- MX2 pad 6: +5V -> PORT1-4_PWR
- MX20 pad 6: +5V -> PORT1-4_PWR
- MX21 pad 6: +5V -> PORT1-4_PWR
- MX22 pad 6: +5V -> PORT1-4_PWR
- MX23 pad 6: +5V -> PORT1-4_PWR
- MX24 pad 6: +5V -> PORT1-4_PWR
- MX25 pad 6: +5V -> PORT1-4_PWR
- MX26 pad 6: +5V -> PORT1-4_PWR
- MX27 pad 6: +5V -> PORT1-4_PWR
- MX28 pad 6: +5V -> PORT1-4_PWR
- MX29 pad 6: +5V -> PORT1-4_PWR
- MX3 pad 6: +5V -> PORT1-4_PWR
- MX30 pad 6: +5V -> PORT1-4_PWR
- MX31 pad 6: +5V -> PORT1-4_PWR
- MX32 pad 6: +5V -> PORT1-4_PWR
- MX33 pad 6: +5V -> PORT1-4_PWR
- MX34 pad 6: +5V -> PORT1-4_PWR
- MX35 pad 6: +5V -> PORT1-4_PWR
- MX36 pad 6: +5V -> PORT1-4_PWR
- MX37 pad 6: +5V -> PORT1-4_PWR
- MX38 pad 6: +5V -> PORT1-4_PWR
- MX39 pad 6: +5V -> PORT1-4_PWR
- MX4 pad 6: +5V -> PORT1-4_PWR
- MX40 pad 6: +5V -> PORT1-4_PWR
- MX41 pad 6: +5V -> PORT1-4_PWR
- MX42 pad 6: +5V -> PORT1-4_PWR
- MX43 pad 6: +5V -> PORT1-4_PWR
- MX45 pad 6: +5V -> PORT1-4_PWR
- MX46 pad 6: +5V -> PORT1-4_PWR
- MX48 pad 6: +5V -> PORT1-4_PWR
- MX49 pad 6: +5V -> PORT1-4_PWR
- MX5 pad 6: +5V -> PORT1-4_PWR
- MX51 pad 6: +5V -> PORT1-4_PWR
- MX52 pad 6: +5V -> PORT1-4_PWR
- MX53 pad 6: +5V -> PORT1-4_PWR
- MX54 pad 6: +5V -> PORT1-4_PWR
- MX55 pad 6: +5V -> PORT1-4_PWR
- MX56 pad 6: +5V -> PORT1-4_PWR
- MX57 pad 6: +5V -> PORT1-4_PWR
- MX59 pad 6: +5V -> PORT1-4_PWR
- MX6 pad 6: +5V -> PORT1-4_PWR
- MX60 pad 6: +5V -> PORT1-4_PWR
- MX61 pad 6: +5V -> PORT1-4_PWR
- MX7 pad 6: +5V -> PORT1-4_PWR
- MX78 pad 6: +5V -> PORT1-4_PWR
- MX8 pad 6: +5V -> PORT1-4_PWR
- MX83 pad 6: +5V -> PORT1-4_PWR
- MX84 pad 6: +5V -> PORT1-4_PWR
- MX9 pad 6: +5V -> PORT1-4_PWR
- OL1 pad 3: +5V -> PORT1-4_PWR
- R13 pad 1: +5V -> PORT1-4_PWR
- R15 pad 1: +5V -> PORT5-7PWR
- R22 pad 1: +5V -> PORT1-4_PWR
- R39 pad 1: +5V -> PORT5-7PWR
- R48 pad 1: +5V -> PORT1-4_PWR
- U12 pad 5: +5V -> PORT1-4_PWR
- U13 pad 3: +5V -> PORT1-4_PWR
- U14 pad 5: +5V -> PORT1-4_PWR
- U14 pad 7: +5V -> PORT1-4_PWR
- U15 pad 5: +5V -> PORT1-4_PWR
- U15 pad 7: +5V -> PORT1-4_PWR
- U2 pad 4: +5V -> PORT1-4_PWR
- USB1 pad 11: +5V -> PORT1-4_PWR
- USB1 pad 2: +5V -> PORT1-4_PWR
Routing:
- net PORT1-4_PWR: track 794.4 -> 3949.0 mm, vias 7 -> 24
- net +5V: track 3110.0 -> 0.00 mm, vias 13 -> 0
- net BKL_DATA_IN_3V3: track 330.0 -> 349.3 mm
- net PORT5-7PWR: track 341.6 -> 358.6 mm
- net KEYBOARD_SDA: track 233.6 -> 249.0 mm
- net KEYBOARD_SCL: track 238.8 -> 252.7 mm, vias 1 -> 2
- net ENCODER_B2: track 291.7 -> 304.6 mm
- net ENCODER_B1: track 347.6 -> 359.3 mm
- net Net-(KD14-Pad2): track 10.7 -> 4.30 mm
- net ENCODER_A: track 642.8 -> 648.8 mm
- net Net-(D8-Pad1): track 0.00 -> 2.85 mm
- net COL0: track 336.3 -> 338.9 mm
- net GND: track 754.7 -> 752.3 mm, vias 309 -> 312
- net Net-(D9-Pad1): track 0.00 -> 2.39 mm
- net HUB_PORT3_D-: track 330.5 -> 328.1 mm
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
Commit message: Added fuse to LED matrix
Parts:
- removed FB16: 60 @ 100 MHz, Inductor_SMD:L_0805_2012Metric
- added C48: 100uF, Capacitor_SMD:C_1206_3216Metric, B.Cu at (234.9, 178.6)
- added F8: 500mA, Fuse:Fuse_1206_3216Metric, B.Cu at (229.4, 178.6)
- moved C17 0.79 mm to (275.4, 278.6), turned to 0 degrees
- moved J5 0.40 mm to (210.3, 272.2)
Routing:
- net GND: track 752.3 -> 904.9 mm, vias 312 -> 322
- net PORT1-4_PWR: track 3949.0 -> 3953.6 mm
- net +3V3: track 374.1 -> 372.7 mm
- net COL3: track 280.1 -> 281.0 mm
- net BOOT0: track 91.4 -> 92.0 mm
- net PORT5-7PWR: track 358.6 -> 358.2 mm, vias 2 -> 4

Commit message: Added JLCPCB Part numbers
Parts:
- C45, C47, C7, C8: value 0.1uF -> 100nF
- TP1: value HUB_D- -> TestPoint_Small
- TP2: value HUB_D+ -> TestPoint_Small
- TP4: value EXTRA_1 -> TestPoint_Small
- turned TP1 to 0 degrees
- turned TP2 to 0 degrees
- turned TP4 to 90 degrees
