File: PCB/custom_keyboard (f103, fe2.1).sch (KiCad schematic (older format))
At the start: 505 parts, among them IC1 FE2.1, J2 Conn_01x04, SW1 SW_Push, U1 24LC02BT-I/SN, U10 PRTR5V0U2X, U11 XC6206P332MR, U12 74LVC1G34, U13 XC6206P332MR, U14 MIC2505, U15 MIC2505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

Commit message: Changed USB test pads to pad style, moved resistors
Parts:
- FB1, FB10, FB11, FB12, FB13, FB14, FB15, FB2, FB3, FB4, FB5, FB6, FB7, FB8, FB9: LCSC Part C18305 -> C237300
- TP1, TP2, TP21, TP22, TP23, TP25, TP39, TP40, TP44, TP45, TP46, TP47, TP48, TP49, TP50, TP51: footprint TestPoint:TestPoint_THTPad_D1.0mm_Drill0.5mm -> TestPoint:TestPoint_Pad_1.0x1.0mm
Connections:
- net labels added: HUB_PORT1_D+, HUB_PORT1_D-, KEYBOARD_5V
- wire segments 2705 -> 2697
Other:
- note added: "Keyboard 3.3v"
- note added: "Keyboard ESD"
- note added: "Upstream 3.3v\n"
- note removed: "Keyboard Power"
- note removed: "Keyboard Protection"
- note removed: "USB Hub 3V3\n"
- moved on the sheet: C1, C10, C13, C16, C17, C18, C19, C2, C20, C21, C23, C25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
