File: PCB/_autosave-custom_keyboard (f103, fe2.1).kicad_pcb (KiCad board)
At the start: 2 copper layers, 395.3 x 138.1 mm, 464 parts, among them IC1 FE2.1, J2 Conn_01x04, U1 24LC02BT-I/SN, U10 PRTR5V0U2X, U11 XC6206P332MR, U12 74LVC1G34, U14 MIC2505, U15 MIC2505, U2 PRTR5V0U2X, U4 PRTR5V0U2X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

Commit message: Changed reset circuit
Parts:
- moved C8 0.79 mm to (449.2, 166.3)
- moved R49 0.79 mm to (445.7, 167.5)
Routing:
- net ENCODER_A: track 651.9 -> 668.6 mm
- net Net-(C5-Pad2): track 15.7 -> 6.62 mm
- net Net-(C6-Pad1): track 16.1 -> 7.06 mm
- net ENCODER_B1: track 355.1 -> 348.0 mm
- net GND: track 727.9 -> 726.7 mm, vias 323 -> 325
