File: PCB/_autosave-custom_keyboard (f103, fe2.1).sch (KiCad schematic (older format))
At the start: 504 parts, among them IC1 FE2.1, J2 Conn_01x04, U1 24LC02BT-I/SN, U10 PRTR5V0U2X, U11 XC6206P332MR, U12 74LVC1G34, U14 MIC2505, U15 MIC2505, U2 PRTR5V0U2X, U3 PRTR5V0U2X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

Commit message: Changed reset circuit
Connections:
- net Earth: no longer FB7.2, USB4.5 (Shield)
- new net: FB7.2, USB4.5 (Shield)
Other:
- note added: "Circuit Breaker"
- moved on the sheet: BOOT0, C1, C10, C11, C12, C13, C14, C2, C23, C24, C25, C26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
