File: PCB/custom_keyboard (f303, fe2.1).sch (KiCad schematic (older format))
At the start: 509 parts, among them IC1 FE2.1, J2 Conn_01x03_Male, J5 AVR-ISP-6, Q1 DTC123J, SW1 SW_Push, U1 24LC02BT-I/SN, U10 PRTR5V0U2X, U11 XC6206P332MR, U12 74LVC1G34, U13 XC6206P332MR, U14 MIC2505, U15 MIC2505, U2 PRTR5V0U2X, U3 PRTR5V0U2X, U4 PRTR5V0U2X, U5 PRTR5V0U2X, U6 PRTR5V0U2X, U7 PRTR5V0U2X, U8 PRTR5V0U2X, U9 STM32F303CBT6, Y1 8MHz, Y2 32.768KHz, Y3 12MHz

Commit message: Reassigned pins on microcontroller
- they were all completely incorrect
Parts:
- removed J2: Conn_01x03_Male, Connector_JST:JST_SH_SM03B-SRSS-TB_1x03-1MP_P1.00mm_Horizontal, symbol Connector:Conn_01x03_Male
- removed J5: AVR-ISP-6, random-keyboard-parts:Reset_Pretty-Mask, symbol Connector:AVR-ISP-6
- removed Q1: DTC123J, Package_TO_SOT_SMD:SOT-23, symbol Transistor_BJT:DTC123J
- removed TP4: TestPoint_Small, TestPoint:TestPoint_THTPad_D1.0mm_Drill0.5mm, symbol Connector:TestPoint_Small
- added J1: Conn_02x03_Odd_Even, Connector_PinSocket_2.54mm:PinSocket_2x03_P2.54mm_Vertical, symbol Connector_Generic:Conn_02x03_Odd_Even
- added Q1: MMBT3904, Package_TO_SOT_SMD:SOT-23, symbol Transistor_BJT:MMBT3904
- added R13, R15: 100k, Resistor_SMD:R_0603_1608Metric, symbol Device:R_Small
Connections:
- net EXTRA_1 is gone; now on net COL2: U9.2 (PC13)
- net +3V3: now also J1.1 (Pin_1); no longer R54.1, R55.1, R56.1
- net +5V: now also R54.1, R55.1, R56.1, R13.1, R15.1
- net BKL_DATA_IN_3V3: now also U9.31 (PA10); no longer U9.29 (PA8)
- net BOOT0: now also J1.3 (Pin_3)
- net COL0: now also U9.37 (PA14), J1.4 (Pin_4); no longer U9.39 (PB3)
- net COL1: now also U9.34 (PA13), J1.2 (Pin_2); no longer U9.38 (PA15)
- net COL10: now also U9.21 (PB10); no longer U9.16 (PA6)
- net COL11: now also U9.22 (PB11); no longer U9.17 (PA7)
- net COL12: now also U9.25 (PB12); no longer U9.18 (PB0)
- net COL13: now also U9.26 (PB13); no longer U9.19 (PB1)
- net COL14: now also TP41.1, U9.27 (PB14); no longer TP7.1, U9.20 (PB2)
- net COL15: now also U9.28 (PB15); no longer U9.21 (PB10)
- net COL16: now also U9.29 (PA8); no longer U9.22 (PB11)
- net COL17: now also U9.30 (PA9); no longer U9.25 (PB12)
- net COL2: no longer U9.37 (PA14)
- net COL3: now also TP7.1, U9.10 (PA0); no longer TP41.1, U9.34 (PA13)
- net COL4: now also U9.11 (PA1); no longer U9.10 (PA0)
- net COL5: now also U9.12 (PA2); no longer U9.11 (PA1)
- net COL6: now also U9.13 (PA3); no longer U9.12 (PA2)
- net COL7: now also U9.14 (PA4); no longer U9.13 (PA3)
- net COL8: now also U9.15 (PA5); no longer U9.14 (PA4)
- net COL9: now also U9.16 (PA6); no longer U9.15 (PA5)
- net ENCODER_A: now also U9.17 (PA7); no longer U9.26 (PB13)
- net ENCODER_B1: now also U9.18 (PB0); no longer U9.27 (PB14)
- net ENCODER_B2: now also U9.19 (PB1); no longer U9.28 (PB15)
- net GND: now also R61.1, J1.6 (Pin_6), Q1.2 (E)
- net KEYBOARD_RESET: now also J1.5 (Pin_5), Q1.3 (C)
- net KEYBOARD_SCL: now also U9.42 (PB6); no longer U9.30 (PA9)
- net KEYBOARD_SDA: now also U9.43 (PB7); no longer U9.31 (PA10)
- net PORT5-7PWR: now also R15.2
- net ROW2: now also U9.41 (PB5); no longer U9.43 (PB7)
- net ROW3: now also U9.40 (PB4); no longer U9.42 (PB6)
- net ROW4: now also U9.39 (PB3); no longer U9.41 (PB5)
- net ROW5: now also U9.38 (PA15); no longer U9.40 (PB4)
- net VCC: now also R13.2
- net at DRST1.2 (A), SW1.2: now also Q1.1 (B)
- no-connect marks 9 -> 10
Other:
- moved on the sheet: C1, C15, C22, C3, C4, C40, C41, C7, C8, C9, D3, DRST1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

Commit message: Changes to F303 schematic and PCB before switch to F103
Parts:
- removed R5: 390, Resistor_SMD:R_0805_2012Metric, symbol Device:R_Small
- removed Y1: 8MHz, Crystal:Crystal_SMD_3225-4Pin_3.2x2.5mm, symbol Device:Crystal_GND24_Small
- added Y1: 8MHz, Crystal:Crystal_SMD_HC49-SD, symbol Device:Crystal_Small
Connections:
- net KEYBOARD_XTAL1: now also Y1.1
- net KEYBOARD_XTAL2: now also C3.1, Y1.2
Other:
- moved on the sheet: C1, C15, C22, C3, C5, C6, C7, C8, D2, D3, DRST1, J1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
