File: PCB/custom_keyboard (f103, fe2.1).kicad_pcb (KiCad board)
At the start: 2 copper layers, 395.3 x 138.1 mm, 464 parts, among them IC1 FE2.1, J2 Conn_01x04, U1 24LC02BT-I/SN, U10 PRTR5V0U2X, U11 XC6206P332MR, U12 74LVC1G34, U14 MIC2505, U15 MIC2505, U2 PRTR5V0U2X, U4 PRTR5V0U2X, U5 PRTR5V0U2X, U6 PRTR5V0U2X, U8 SD00HA, U9 STM32F103C8T6, Y1 8MHz, Y3 12MHz

Commit message: Tidied up components on schematic and PCB
Parts:
- moved C30 8.74 mm to (395.3, 250.0), turned to 90 degrees
- moved C28 3.99 mm to (397.6, 250.0), turned to 270 degrees
- moved C37 3.76 mm to (395.7, 246.8), turned to 0 degrees
- moved R15 1.77 mm to (426.2, 228.6)
- moved TP53 1.59 mm to (428.6, 227.8), turned to 180 degrees
- moved C27 0.89 mm to (400.0, 250.0), turned to 270 degrees
- moved C8 0.79 mm to (449.2, 166.3)
- moved R49 0.79 mm to (445.7, 167.5)
- renumbered IC1 to FE2.1, U9 to STM32
Routing:
- net GND: track 727.9 -> 751.1 mm, vias 323 -> 325
- net ENCODER_A: track 651.9 -> 668.6 mm
- net Net-(C5-Pad2): track 15.7 -> 6.62 mm
- net Net-(C6-Pad1): track 16.1 -> 7.06 mm
- net ENCODER_B1: track 355.1 -> 348.0 mm
- net PORT5-7PWR: track 280.4 -> 278.6 mm
- net HUB_LED1: track 42.4 -> 41.0 mm
- net +5V: track 3263.2 -> 3264.4 mm

Commit message: Reannotated components
Parts:
- moved FB15 15.1 mm to (210.3, 268.3), turned to 90 degrees
- moved C23 4.27 mm to (258.7, 269.1), turned to 0 degrees
- moved C24 4.27 mm to (258.7, 266.7), turned to 180 degrees
- moved F8 2.38 mm to (210.3, 280.2), turned to 90 degrees
- moved R25 1.77 mm to (203.2, 276.2), turned to 270 degrees
- moved C1 0.79 mm to (235.7, 178.6)
- moved F1 0.79 mm to (230.2, 178.6)
- turned TP19 to 180 degrees
- turned TP21 to 0 degrees
- turned TP23 to 180 degrees
- turned TP36 to 180 degrees
- turned TP43 to 0 degrees
- renumbered C48 to C1, C7 to C10, C8 to C11, C34 to C12, C9 to C13, C11 to C14, C12 to C15, C14 to C16, C2 to C17, C4 to C18, C16 to C19, C32 to C2, C17 to C20, C18 to C21, C19 to C22, C20 to C23, C21 to C24, C13 to C25, C24 to C26, C26 to C27, C27 to C28, C28 to C29, C1 to C3, C10 to C30, C29 to C31, C30 to C32, C31 to C33, C44 to C34, C45 to C35, C35 to C38, C38 to C39, C25 to C4, C39 to C40, C46 to C41, C47 to C42, C40 to C43, C41 to C44, C33 to C5, C23 to C6, C3 to C7, D9 to D2, D2 to D3, D3 to D4, D4 to D5, D5 to D7, D7 to D8, D8 to D9, F8 to F1, F6 to F2, F5 to F3, F7 to F4, F2 to F5, F4 to F6, F3 to F7, F1 to F8, FB9 to FB1, FB13 to FB10, FB2 to FB11, FB4 to FB12, FB14 to FB13, FB3 to FB14, FB8 to FB2, FB10 to FB3, FB6 to FB4, FB1 to FB5, FB11 to FB6, FB5 to FB7, FB12 to FB8, FB7 to FB9, J2 to J1, R57 to R10, R33 to R11, R8 to R12, R9 to R13, R28 to R14, R14 to R16, R49 to R18, R30 to R19, R58 to R2, R53 to R20, R52 to R21, R5 to R22, R45 to R23, R48 to R24, R39 to R25, R46 to R26, R16 to R27, R60 to R28, R21 to R29, R2 to R3, R59 to R30, R22 to R31, R23 to R32, R10 to R33, R3 to R34, R6 to R35, R11 to R36, R1 to R37, R50 to R38, R51 to R39, R24 to R40, R43 to R41, R25 to R42, R44 to R43, R7 to R44, R61 to R45, R17 to R46, R18 to R47, R62 to R48, R26 to R49, R34 to R5, R35 to R50, R41 to R51, R20 to R52, R19 to R53, R29 to R54, R13 to R55, R36 to R56, R54 to R57, R42 to R58, R32 to R59, R37 to R6, R55 to R60, R15 to R61, R56 to R62, R38 to R63, R27 to R7, R63 to R8, R31 to R9, TP47 to TP10, TP48 to TP11, TP49 to TP12, TP26 to TP13, TP3 to TP14, TP24 to TP15, TP42 to TP16, TP8 to TP17, TP43 to TP18, TP7 to TP20, TP20 to TP21, TP28 to TP22, TP27 to TP23, TP29 to TP24, TP10 to TP25, TP30 to TP26, TP11 to TP27, TP31 to TP28, TP50 to TP29, TP21 to TP3, TP12 to TP30, TP32 to TP31, TP51 to TP32, TP37 to TP33, TP33 to TP34, TP38 to TP35, TP18 to TP36, TP13 to TP37, TP16 to TP38, TP52 to TP39, TP22 to TP4, TP14 to TP40, TP17 to TP41, TP34 to TP42, TP36 to TP43, TP35 to TP44, TP39 to TP45, TP5 to TP46, TP40 to TP47, TP6 to TP48, TP41 to TP49, TP23 to TP5, TP15 to TP50, TP9 to TP51, TP53 to TP52, TP54 to TP53, TP25 to TP6, TP44 to TP7, TP45 to TP8, TP46 to TP9, U8 to U1, U4 to U10, U15 to U11, U11 to U12, U12 to U13, U6 to U4, U1 to U5, U10 to U6, U5 to U8, U14 to U9, Y3 to Y1, Y1 to Y2
Routing:
- net +5V: track 3264.4 -> 3216.3 mm
- net Net-(F8-Pad2): track 2.30 -> 9.44 mm
- net +3V3: track 338.7 -> 334.2 mm
- net KEYBOARD_5V: track 226.3 -> 228.2 mm
- net GND: track 751.1 -> 752.3 mm, vias 325 -> 327
- net COL10: track 171.5 -> 172.6 mm

Commit message: Added logo, copyright, and credits
Parts:
- added logo: G***, custom-footprints:logo, F.Cu at (406.4, 253.2)
- FE2.1: value FE2.1 -> LQFP-48_L7.0-W7.0-P0.50-LS9.0-BL
- U11, U9: value MIC2505 -> SOIC-8_L5.0-W4.0-P1.27-LS6.0-BL
Routing:
- net GND: track 752.3 -> 736.1 mm
