File: PCB/custom_keyboard (f103, fe2.1).kicad_pcb (KiCad board)
At the start: 2 copper layers, 395.3 x 138.1 mm, 465 parts, among them J1 Conn_01x04, U1 SD00HA, U10 PRTR5V0U2X, U11 SOIC-8_L5.0-W4.0-P1.27-LS6.0-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, U12 XC6206P332MR, U13 74LVC1G34, U2 PRTR5V0U2X, U4 PRTR5V0U2X, U5 24LC02BT-I/SN, U6 PRTR5V0U2X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

Commit message: Moved resistors closer to usb hub ic
Parts:
- removed logo: G***, custom-footprints:logo
- added MX64: ENTER, custom-footprints:CherryMX_2.25u_PCB_KailhSocket_LTST-A683CEGBW, F.Cu at (367.5, 234.9)
- added TP54: Logo, custom-footprints:logo, F.Cu at (406.4, 252.4)
- FE2.1: value LQFP-48_L7.0-W7.0-P0.50-LS9.0-BL -> FE2.1
- U11, U9: value SOIC-8_L5.0-W4.0-P1.27-LS6.0-BL -> MIC2505
- U5: value 24LC02BT-I/SN -> 24LC04BT-I/SN
- moved R52 26.2 mm to (398.8, 229.0)
- moved R53 26.2 mm to (401.2, 229.0)
- moved R9 22.3 mm to (384.9, 237.3), turned to 0 degrees
- moved R11 20.2 mm to (384.9, 234.9), turned to 0 degrees
- moved C38 15.2 mm to (387.3, 229.4)
- moved R40 15.1 mm to (398.8, 223.8)
- moved R42 15.1 mm to (396.5, 223.8)
- moved R23 5.61 mm to (389.3, 251.6)
- moved R26 5.61 mm to (391.7, 251.6)
- moved C39 4.86 mm to (384.2, 245.9), turned to 270 degrees
- moved C31 4.76 mm to (388.9, 246.8), turned to 270 degrees
- moved C40 3.37 mm to (386.5, 246.8), turned to 270 degrees
- moved C33 3.31 mm to (387.3, 227.0)
- moved R51 3.30 mm to (387.3, 224.6)
- moved C26 2.51 mm to (406.4, 228.6), turned to 90 degrees
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Routing:
- net HUB_PORT2_D-: track 37.2 -> 3.73 mm, vias 2 -> 0
- net HUB_PORT2_D+: track 36.2 -> 4.30 mm, vias 2 -> 0
- net Net-(R9-Pad1): track 345.1 -> 376.8 mm, vias 0 -> 2
- net HUB_PORT7_D-: track 35.8 -> 5.06 mm, vias 2 -> 0
- net Net-(R11-Pad1): track 347.1 -> 377.7 mm, vias 0 -> 2
- net HUB_PORT7_D+: track 36.3 -> 5.81 mm, vias 2 -> 0
- net GND: track 736.1 -> 706.4 mm, vias 327 -> 328
- net Net-(R53-Pad1): track 82.8 -> 109.9 mm
- net Net-(R52-Pad1): track 82.2 -> 109.4 mm
- net HUB_PORT6_D+: track 24.0 -> 7.97 mm
- net HUB_PORT6_D-: track 24.0 -> 7.97 mm
- net Net-(R40-Pad1): track 81.3 -> 96.7 mm
- net Net-(R42-Pad1): track 81.3 -> 96.7 mm
- net Net-(R23-Pad1): track 73.8 -> 79.7 mm
- net Net-(R26-Pad1): track 73.2 -> 79.0 mm
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
Commit message: Added indicator LEDs to keyboard power
Parts:
- added D11: Red, LED_SMD:LED_0805_2012Metric, B.Cu at (206.4, 281.8)
- added D12: Red, LED_SMD:LED_0805_2012Metric, B.Cu at (227.8, 178.6)
- added R64: 330, Resistor_SMD:R_0805_2012Metric, B.Cu at (202.4, 281.8)
- added R65: 330, Resistor_SMD:R_0805_2012Metric, B.Cu at (230.2, 178.6)
- moved F1 5.61 mm to (235.7, 179.4)
- moved C1 5.61 mm to (241.3, 179.4)
- moved TP54 0.79 mm to (406.4, 253.2)
- turned TP13 to 180 degrees
Routing:
- net GND: track 706.4 -> 722.0 mm, vias 328 -> 329
- net Net-(D12-Pad2): track 4.78 -> 9.33 mm
- net KEYBOARD_5V: track 228.1 -> 231.2 mm
- net Net-(D12-Pad1): track 0.00 -> 2.39 mm
- net Net-(D11-Pad1): track 0.00 -> 2.14 mm
- net +5V: track 3213.9 -> 3214.7 mm
- net +3V3: track 337.9 -> 338.5 mm

Commit message: Added guard traces, double checked part numbers
Parts:
- turned TP13 to 0 degrees
Routing:
- net GND: track 722.0 -> 1376.6 mm, vias 329 -> 352
- net Net-(R9-Pad1): track 376.8 -> 374.1 mm
- net Net-(R11-Pad1): track 377.7 -> 375.0 mm
- net Net-(R6-Pad1): track 347.4 -> 345.8 mm
- net Net-(R5-Pad1): track 346.3 -> 344.7 mm
- net DOUT5: track 375.2 -> 374.1 mm
- net KEYBOARD_D-: track 154.6 -> 153.6 mm
- net KEYBOARD_D+: track 154.4 -> 153.4 mm
