File: PCB/custom_keyboard (f103, fe2.1).kicad_pcb (KiCad board)
At the start: 2 copper layers, 395.3 x 138.1 mm, 470 parts, among them J1 Conn_01x04, SW1 SW_Push, SW2 SW_Push, U1 SD00HA, U10 PRTR5V0U2X, U11 MIC2505, U12 XC6206P332MR, U13 74LVC1G34, U2 PRTR5V0U2X, U4 PRTR5V0U2X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

Commit message: Removed open load detect resistors
Parts:
- removed R55, R61: 100k, Resistor_SMD:R_0603_1608Metric
- U11, U9: value MIC2505 -> MIC2505-1YM
Routing:
- net +5V: track 3214.2 -> 3210.0 mm
- net PORT1-4_PWR: track 643.5 -> 640.4 mm
- net PORT5-7PWR: track 278.6 -> 277.9 mm
- net GND: vias 354 -> 355

Commit message: Draft 1-5 with MCU swapped with F303
Parts:
- removed STM32: STM32F103C8T6, Package_QFP:LQFP-48_7x7mm_P0.5mm
- added U14: STM32F303CBTx, Package_QFP:LQFP-48_7x7mm_P0.5mm, B.Cu at (268.3, 273.0)
- moved ROW3 1.12 mm to (99.2, 231.0)
- moved ROW5 1.12 mm to (98.4, 269.1)
- moved ROW1 0.89 mm to (100.4, 192.9)
- moved ROW4 0.89 mm to (98.8, 250.0)
- moved D+5 0.79 mm to (309.1, 175.8)
- moved D-5 0.79 mm to (306.8, 175.8)
- moved R60 0.79 mm to (427.8, 233.4)
- moved ROW2 0.79 mm to (100.0, 211.9)
Routing:
- net GND: track 1431.3 -> 1924.8 mm, vias 355 -> 488
- net COL13: track 204.2 -> 213.5 mm
- net COL12: track 193.7 -> 203.0 mm
- net COL11: track 199.2 -> 205.3 mm
- net DOUT1: track 363.1 -> 368.7 mm
- net BKL_DATA_IN_3V3: track 324.0 -> 329.1 mm
- net +5V: track 3210.0 -> 3214.9 mm
- net COL7: track 157.7 -> 161.9 mm
- net OVCJ1: track 41.4 -> 37.6 mm
- net COL9: track 148.2 -> 151.9 mm
- net COL8: track 138.7 -> 142.4 mm
- net COL10: track 172.6 -> 176.3 mm
- net KEYBOARD_RESET: track 70.3 -> 73.5 mm
- net KEYBOARD_D-: track 153.6 -> 150.7 mm
- net COL3: track 249.9 -> 251.8 mm
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
Commit message: Slightly adjusted USB traces
Parts:
- U14: value STM32F303CBTx -> STM32F303CBT6
- moved COL15 1.77 mm to (401.6, 188.9)
Connections:
- D+6 pad 1: Net-(D+6-Pad1) -> HUB_PORT6_D+
- D+7 pad 1: Net-(D+7-Pad1) -> HUB_PORT7_D+
- D-6 pad 1: Net-(D-6-Pad1) -> HUB_PORT6_D-
- D-7 pad 1: Net-(D-7-Pad1) -> HUB_PORT7_D-
- R40 pad 1: Net-(D+6-Pad1) -> HUB_PORT6_D+
- R42 pad 1: Net-(D-6-Pad1) -> HUB_PORT6_D-
- R52 pad 1: Net-(D-7-Pad1) -> HUB_PORT7_D-
- R53 pad 1: Net-(D+7-Pad1) -> HUB_PORT7_D+
- U10 pad 2: Net-(D+7-Pad1) -> HUB_PORT7_D+
- U10 pad 3: Net-(D-7-Pad1) -> HUB_PORT7_D-
- U8 pad 2: Net-(D+6-Pad1) -> HUB_PORT6_D+
- U8 pad 3: Net-(D-6-Pad1) -> HUB_PORT6_D-
- USB6 pad 2: Net-(D-6-Pad1) -> HUB_PORT6_D-
- USB6 pad 3: Net-(D+6-Pad1) -> HUB_PORT6_D+
- USB7 pad 5: Net-(D-7-Pad1) -> HUB_PORT7_D-
- USB7 pad 6: Net-(D+7-Pad1) -> HUB_PORT7_D+
- USB7 pad 7: Net-(D-7-Pad1) -> HUB_PORT7_D-
- USB7 pad 8: Net-(D+7-Pad1) -> HUB_PORT7_D+
Routing:
- net Net-(D+7-Pad1): track 110.4 -> 0.00 mm
- net Net-(D-7-Pad1): track 109.8 -> 0.00 mm
- net HUB_PORT7_D+: track 5.81 -> 114.8 mm
- net HUB_PORT7_D-: track 5.06 -> 113.6 mm
- net Net-(D+6-Pad1): track 96.7 -> 0.00 mm
- net Net-(D-6-Pad1): track 96.7 -> 0.00 mm
- net HUB_PORT6_D+: track 7.97 -> 104.2 mm
- net HUB_PORT6_D-: track 7.97 -> 104.2 mm
- net GND: track 1924.8 -> 1980.7 mm, vias 488 -> 496
- net +5V: track 3214.9 -> 3214.0 mm
