File: PCB/custom_keyboard plate.kicad_pcb (KiCad board)
At the start: 2 copper layers, 393.7 x 141.3 mm, 0 parts

Commit message: Exported keyboard plate files
Parts:
- added logo: G***, custom-footprints:logo, F.Cu at (416.7, 255.6)
Other:
- board text added: "kb.ht12345.xyz/0"
- board text added: "keyboard0 FR4 plate"
- board text added: "© 2021 Howard Tseng"
Changed lines of the file:
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@@
   (general
     (thickness 1.6)
-    (drawings 1112)
+    (drawings 1115)
     (tracks 1)
     (zones 0)
-    (modules 0)
+    (modules 1)
     (nets 1)
   )
@@
     (uvia_drill 0.1)
   )
+  (module custom-footprints:logo (layer F.Cu)
+    (at 416.6925 255.5714)
+    (descr "Converted using: svg2mod -i Untitled-1.svg -o ./custom-footprints.pretty/logo -f 1 --name logo")
+    (tags svg2mod)
+    (attr virtual)
+    (fp_text reference logo (at 0 -3.048) (layer F.SilkS) hide
+      (effects (font (size 1.524 1.524) (thickness 0.3048)))
+    )
+    (fp_text value G*** (at 0 9.474729) (layer F.SilkS) hide
+      (effects (font (size 1.524 1.524) (thickness 0.3048)))
+    )
+    (fp_poly (pts (xy -2.19075 3.172354) (xy -1.296458 2.278063) (xy -1.613958 1.947333) (xy -3.81 4.146021)
+      (xy -3.479271 4.474104) (xy -2.590271 3.582458) (xy 0.238125 6.426729) (xy 0.648229 6.013979)
+      (xy -2.19075 3.172354)) (layer B.SilkS) (width 0))
+    (fp_poly (pts (xy 0.502708 5.606521) (xy 3.677708 2.431521) (xy 3.264958 2.026708) (xy 1.899708 3.394604)
+      (xy 0.293687 1.785938) (xy 1.661583 0.415396) (xy 1.246187 0) (xy -1.928813 3.175)
+      (xy -1.508125 3.585104) (xy -0.047625 2.119313) (xy 1.561042 3.722688) (xy 0.09525 5.188479)
+      (xy 0.502708 5.606521)) (layer B.SilkS) (width 0))
+  )
+  (gr_text "© 2021 Howard Tseng" (at 411.9303 260.3336) (layer B.SilkS)
+    (effects (font (size 1 1) (thickness 0.15)) (justify left mirror))
+  )
+  (gr_text kb.ht12345.xyz/0 (at 411.9303 258.7462) (layer B.SilkS)
+    (effects (font (size 1 1) (thickness 0.15)) (justify left mirror))
+  )
+  (gr_text "keyboard0 FR4 plate" (at 411.9303 257.1588) (layer B.SilkS)
+    (effects (font (size 1 1) (thickness 0.15)) (justify left mirror))
+  )
   (gr_text "JLCJLCJLCJLC\n" (at 405.5807 294.4627) (layer B.SilkS)
