File: PCB/custom_keyboard (f303).kicad_pcb (KiCad board)
At the start: 2 copper layers, 395.3 x 138.1 mm, 468 parts, among them J1 Conn_01x04, SW1 SW_Push, SW2 SW_Push, U1 SD00HA, U10 PRTR5V0U2X, U11 MIC2505-1YM, U12 XC6206P332MR, U13 74LVC1G34, U14 STM32F303CBT6, U2 PRTR5V0U2X, U4 PRTR5V0U2X, U5 24LC04BT-I/SN, U6 PRTR5V0U2X, U8 PRTR5V0U2X, U9 MIC2505-1YM, X1 TestPoint_Small, X2 TestPoint_Small, Y1 12MHz, Y2 8MHz

Commit message: Exported files for first prototype
Parts:
- added UD10: Amber, LED_SMD:LED_0805_2012Metric, B.Cu at (424.6, 242.9)
- added UD11: Amber, LED_SMD:LED_0805_2012Metric, B.Cu at (428.6, 242.9)
- added UD12: Amber, LED_SMD:LED_0805_2012Metric, B.Cu at (433.4, 242.9)
- added UD13: Amber, LED_SMD:LED_0805_2012Metric, B.Cu at (437.3, 242.9)
- added UD14: Amber, LED_SMD:LED_0805_2012Metric, B.Cu at (441.3, 242.9)
- added UD8: Amber, LED_SMD:LED_0805_2012Metric, B.Cu at (416.7, 242.9)
- added UD9: Amber, LED_SMD:LED_0805_2012Metric, B.Cu at (420.7, 242.9)
- moved C12 2.86 mm to (444.5, 245.3), turned to 90 degrees
- moved R37 2.38 mm to (416.7, 245.3)
- moved R44 2.38 mm to (420.7, 245.3)
- moved R46 2.38 mm to (424.6, 245.3)
- moved R47 2.38 mm to (428.6, 245.3)
- moved UD5 2.38 mm to (433.4, 245.3)
- moved UD6 2.38 mm to (437.3, 245.3)
- moved UD7 2.38 mm to (441.3, 245.3)
- moved ENCA1 0.79 mm to (269.1, 264.3), turned to 180 degrees
- moved ENCB1 0.79 mm to (273.8, 264.3)
- moved ENCB2 0.79 mm to (271.4, 264.3)
- moved R62 0.40 mm to (415.5, 232.6)
- turned 1-4 to 90 degrees
Connections:
- D+6 pad 1: HUB_PORT6_D+ -> Net-(D+6-Pad1)
- D+7 pad 1: HUB_PORT7_D+ -> Net-(D+7-Pad1)
- D-6 pad 1: HUB_PORT6_D- -> Net-(D-6-Pad1)
- D-7 pad 1: HUB_PORT7_D- -> Net-(D-7-Pad1)
- R40 pad 1: HUB_PORT6_D+ -> Net-(D+6-Pad1)
- R42 pad 1: HUB_PORT6_D- -> Net-(D-6-Pad1)
- R52 pad 1: HUB_PORT7_D- -> Net-(D-7-Pad1)
- R53 pad 1: HUB_PORT7_D+ -> Net-(D+7-Pad1)
- U10 pad 2: HUB_PORT7_D+ -> Net-(D+7-Pad1)
- U10 pad 3: HUB_PORT7_D- -> Net-(D-7-Pad1)
- U8 pad 2: HUB_PORT6_D+ -> Net-(D+6-Pad1)
- U8 pad 3: HUB_PORT6_D- -> Net-(D-6-Pad1)
- USB6 pad 2: HUB_PORT6_D- -> Net-(D-6-Pad1)
- USB6 pad 3: HUB_PORT6_D+ -> Net-(D+6-Pad1)
- USB7 pad 5: HUB_PORT7_D- -> Net-(D-7-Pad1)
- USB7 pad 6: HUB_PORT7_D+ -> Net-(D+7-Pad1)
- USB7 pad 7: HUB_PORT7_D- -> Net-(D-7-Pad1)
- USB7 pad 8: HUB_PORT7_D+ -> Net-(D+7-Pad1)
Routing:
- net Net-(D+7-Pad1): track 0.00 -> 109.0 mm
- net HUB_PORT7_D+: track 114.8 -> 5.81 mm
- net HUB_PORT7_D-: track 113.6 -> 5.06 mm
- net Net-(D-7-Pad1): track 0.00 -> 108.5 mm
- net Net-(D+6-Pad1): track 0.00 -> 96.2 mm
- net HUB_PORT6_D+: track 104.2 -> 7.97 mm
- net HUB_PORT6_D-: track 104.2 -> 7.97 mm
- net Net-(D-6-Pad1): track 0.00 -> 96.2 mm
- net HUB_DRV: track 68.3 -> 86.7 mm
- net GND: track 1980.7 -> 1973.6 mm, vias 496 -> 493
- net HUB_LED2: track 33.0 -> 30.6 mm
- net Net-(R59-Pad1): track 2.39 -> 4.77 mm
- net Net-(R47-Pad1): track 2.39 -> 4.77 mm
- net Net-(R46-Pad1): track 2.39 -> 4.77 mm
- net HUB_LED4: track 52.9 -> 50.5 mm
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
Commit message: (not in 1st proto) Fixed rotary encoder locations
Parts:
- moved D3 12.9 mm to (96.0, 174.6), turned to 270 degrees
- moved ROT1 12.1 mm to (91.3, 160.7), turned to 270 degrees
- moved ROT2 11.4 mm to (448.4, 160.7), turned to 270 degrees
- moved R16 6.93 mm to (448.4, 164.3), turned to 0 degrees
- moved C11 4.91 mm to (444.5, 167.5), turned to 270 degrees
- moved C10 4.65 mm to (447.6, 167.5)
- moved R18 3.74 mm to (443.7, 164.3)
- moved D4 1.12 mm to (438.1, 177.0), turned to 0 degrees
Routing:
- net ROT1_ROW: track 660.0 -> 644.9 mm
- net COL0: track 345.8 -> 337.4 mm
- net ENCODER_A: track 668.2 -> 676.2 mm, vias 2 -> 3
- net Net-(D4-Pad2): track 3.53 -> 9.40 mm
- net ENCODER_B1: track 349.0 -> 343.8 mm
- net COL17: track 305.3 -> 301.4 mm
- net Net-(C10-Pad2): track 8.72 -> 6.22 mm
- net PORT5-7PWR: track 276.3 -> 274.5 mm
- net BKL_DATA_IN_3V3: track 329.1 -> 327.5 mm
- net ENCODER_B2: track 300.4 -> 301.7 mm
- net Net-(C11-Pad1): track 7.11 -> 6.32 mm
- net Net-(C9-Pad1): track 7.06 -> 6.32 mm
- net Net-(D3-Pad2): track 5.82 -> 5.19 mm
- net GND: vias 493 -> 498

Commit message: Halfway through converting to FE1.1s
Parts:
- removed 1-4, 5-7, BKL3, BKL5, BOOT1, COL0, COL1, COL10, COL11, COL12, COL13, COL14, COL15, COL16, COL17, COL2, COL3, COL4, COL5, COL6, COL7, COL8, COL9, ENCA1, ENCB1, ENCB2, KSCL1, KSDA1, ROW0, ROW1, ROW2, ROW3, ROW4, ROW5, X1, X2: TestPoint_Small, TestPoint:TestPoint_THTPad_D1.0mm_Drill0.5mm
- removed C1, C17, C25, C30: 100uF, Capacitor_SMD:C_1206_3216Metric
- removed C10, C11, C13, C16, C18, C19, C20, C22, C26, C27, C28, C29, C31, C32, C33, C34, C35, C38, C39, C40, C41, C42: 100nF, Capacitor_SMD:C_0805_2012Metric
- removed C21, LC1, LC10, LC11, LC12, LC13, LC14, LC15, LC16, LC17, LC18, LC19, LC2, LC20, LC21, LC22, LC23, LC24, LC25, LC26, LC27, LC28, LC29, LC3, LC30, LC31, LC32, LC33, LC34, LC35, LC36, LC37, LC38, LC39, LC4, LC40, LC41, LC42, LC43, LC44, LC45, LC46, LC47, LC48, LC49, LC5, LC50, LC51, LC52, LC53, LC54, LC55, LC56, LC57, LC58, LC59, LC6, LC60, LC61, LC62, LC63, LC64, LC65, LC66, LC67, LC68, LC69, LC7, LC70, LC71, LC72, LC73, LC74, LC75, LC76, LC77, LC78, LC79, LC8, LC80, LC81, LC82, LC83, LC84, LC85, LC86, LC87, LC88, LC89, LC9, LC90: 10uF, Capacitor_SMD:C_0805_2012Metric
- removed C23: 10nF, Capacitor_SMD:C_0805_2012Metric
- removed C24, C43, C44: 1uF, Capacitor_SMD:C_0805_2012Metric
- removed C3, C7: 20pF, Capacitor_SMD:C_0805_2012Metric
- removed D+5, D+6, D+7, D-5, D-6, D-7, KD+1, KD-1: TestPoint_Small, TestPoint:TestPoint_Pad_1.0x1.0mm
- removed D11, D12, D6, D8, D9: Red, LED_SMD:LED_0805_2012Metric
- removed D3, D4, KD1, KD10, KD11, KD12, KD13, KD14, KD15, KD16, KD17, KD18, KD19, KD2, KD20, KD21, KD22, KD23, KD24, KD25, KD26, KD27, KD28, KD29, KD3, KD30, KD31, KD32, KD33, KD34, KD35, KD36, KD37, KD38, KD39, KD4, KD40, KD41, KD42, KD43, KD44, KD45, KD46, KD47, KD48, KD49, KD5, KD50, KD51, KD52, KD53, KD54, KD55, KD56, KD57, KD58, KD59, KD6, KD60, KD61, KD62, KD63, KD64, KD65, KD66, KD67, KD68, KD69, KD7, KD70, KD71, KD72, KD73, KD74, KD75, KD76, KD77, KD78, KD79, KD8, KD80, KD81, KD82, KD83, KD84, KD85, KD86, KD87, KD88, KD89, KD9, KD90: SOD-123, Diode_SMD:D_SOD-123
- removed F1, F5, F6, F7, F8: 500mA, Fuse:Fuse_1206_3216Metric
- removed FB10, FB11, FB12, FB13, FB14, FB2, FB8: 60 @ 100 MHz, Inductor_SMD:L_0805_2012Metric
- removed FE2.1: FE2.1, custom-footprints:FE2.1
- removed J1: Conn_01x04, Connector_PinSocket_2.54mm:PinSocket_1x04_P2.54mm_Vertical
- removed LOGO0: Logo, custom-footprints:logo
- removed MX1: ESC, custom-footprints:CherryMX_1.00u_PCB_KailhSocket_LTST-A683CEGBW
- removed MX10: F9, custom-footprints:CherryMX_1.00u_PCB_KailhSocket_LTST-A683CEGBW
- removed MX11: F10, custom-footprints:CherryMX_1.00u_PCB_KailhSocket_LTST-A683CEGBW
- removed MX12: F11, custom-footprints:CherryMX_1.00u_PCB_KailhSocket_LTST-A683CEGBW
- removed MX13: F12, custom-footprints:CherryMX_1.00u_PCB_KailhSocket_LTST-A683CEGBW
- removed MX14: PSCR, custom-footprints:CherryMX_1.00u_PCB_KailhSocket_LTST-A683CEGBW
- removed MX15: M1, custom-footprints:CherryMX_1.00u_PCB_KailhSocket_LTST-A683CEGBW
- removed MX16: `/~, custom-footprints:CherryMX_1.00u_PCB_KailhSocket_LTST-A683CEGBW
- removed MX17: 1, custom-footprints:CherryMX_1.00u_PCB_KailhSocket_LTST-A683CEGBW
- removed MX18: 2, custom-footprints:CherryMX_1.00u_PCB_KailhSocket_LTST-A683CEGBW
- removed MX19: 3, custom-footprints:CherryMX_1.00u_PCB_KailhSocket_LTST-A683CEGBW
- removed MX2: F1, custom-footprints:CherryMX_1.00u_PCB_KailhSocket_LTST-A683CEGBW
- removed MX20: 4, custom-footprints:CherryMX_1.00u_PCB_KailhSocket_LTST-A683CEGBW
- removed MX21: 5, custom-footprints:CherryMX_1.00u_PCB_KailhSocket_LTST-A683CEGBW
- removed MX22: 6, custom-footprints:CherryMX_1.00u_PCB_KailhSocket_LTST-A683CEGBW
- removed MX23: 7, custom-footprints:CherryMX_1.00u_PCB_KailhSocket_LTST-A683CEGBW
- removed MX24: 8, custom-footprints:CherryMX_1.00u_PCB_KailhSocket_LTST-A683CEGBW
- removed MX25: 9, custom-footprints:CherryMX_1.00u_PCB_KailhSocket_LTST-A683CEGBW
- removed MX26: 0, custom-footprints:CherryMX_1.00u_PCB_KailhSocket_LTST-A683CEGBW
- removed MX27: -/_, custom-footprints:CherryMX_1.00u_PCB_KailhSocket_LTST-A683CEGBW
- removed MX28: =/+, custom-footprints:CherryMX_1.00u_PCB_KailhSocket_LTST-A683CEGBW
- removed MX29: BACKSPACE, custom-footprints:CherryMX_2.00u_PCB_KailhSocket_LTST-A683CEGBW
- removed MX3: F2, custom-footprints:CherryMX_1.00u_PCB_KailhSocket_LTST-A683CEGBW
- removed MX30: INS, custom-footprints:CherryMX_1.00u_PCB_KailhSocket_LTST-A683CEGBW
- removed MX31: HOME, custom-footprints:CherryMX_1.00u_PCB_KailhSocket_LTST-A683CEGBW
- removed MX32: PGUP, custom-footprints:CherryMX_1.00u_PCB_KailhSocket_LTST-A683CEGBW
- removed MX33: M2, custom-footprints:CherryMX_1.00u_PCB_KailhSocket_LTST-A683CEGBW
- removed MX34: TAB, custom-footprints:CherryMX_1.50u_PCB_KailhSocket_LTST-A683CEGBW
- removed MX35: Q, custom-footprints:CherryMX_1.00u_PCB_KailhSocket_LTST-A683CEGBW
- removed MX36: W, custom-footprints:CherryMX_1.00u_PCB_KailhSocket_LTST-A683CEGBW
- removed MX37: E, custom-footprints:CherryMX_1.00u_PCB_KailhSocket_LTST-A683CEGBW
- removed MX38: R, custom-footprints:CherryMX_1.00u_PCB_KailhSocket_LTST-A683CEGBW
- removed MX39: T, custom-footprints:CherryMX_1.00u_PCB_KailhSocket_LTST-A683CEGBW
- removed MX4: F3, custom-footprints:CherryMX_1.00u_PCB_KailhSocket_LTST-A683CEGBW
- removed MX40: Y, custom-footprints:CherryMX_1.00u_PCB_KailhSocket_LTST-A683CEGBW
- removed MX41: U, custom-footprints:CherryMX_1.00u_PCB_KailhSocket_LTST-A683CEGBW
- removed MX42: I, custom-footprints:CherryMX_1.00u_PCB_KailhSocket_LTST-A683CEGBW
- removed MX43: O, custom-footprints:CherryMX_1.00u_PCB_KailhSocket_LTST-A683CEGBW
- removed MX45: [/{, custom-footprints:CherryMX_1.00u_PCB_KailhSocket_LTST-A683CEGBW
- removed MX46: ]/}, custom-footprints:CherryMX_1.00u_PCB_KailhSocket_LTST-A683CEGBW
- removed MX48: DELETE, custom-footprints:CherryMX_1.00u_PCB_KailhSocket_LTST-A683CEGBW
- removed MX49: END, custom-footprints:CherryMX_1.00u_PCB_KailhSocket_LTST-A683CEGBW
- removed MX5: F4, custom-footprints:CherryMX_1.00u_PCB_KailhSocket_LTST-A683CEGBW
- removed MX51: M3, custom-footprints:CherryMX_1.00u_PCB_KailhSocket_LTST-A683CEGBW
- removed MX52: CAPS, custom-footprints:CherryMX_1.75u_PCB_KailhSocket_LTST-A683CEGBW
- removed MX54: S, custom-footprints:CherryMX_1.00u_PCB_KailhSocket_LTST-A683CEGBW
- removed MX55: D, custom-footprints:CherryMX_1.00u_PCB_KailhSocket_LTST-A683CEGBW
- removed MX56: F, custom-footprints:CherryMX_1.00u_PCB_KailhSocket_LTST-A683CEGBW
- removed MX57: G, custom-footprints:CherryMX_1.00u_PCB_KailhSocket_LTST-A683CEGBW
- removed MX59: J, custom-footprints:CherryMX_1.00u_PCB_KailhSocket_LTST-A683CEGBW
- removed MX6: F5, custom-footprints:CherryMX_1.00u_PCB_KailhSocket_LTST-A683CEGBW
- removed MX60: K, custom-footprints:CherryMX_1.00u_PCB_KailhSocket_LTST-A683CEGBW
- removed MX61: L, custom-footprints:CherryMX_1.00u_PCB_KailhSocket_LTST-A683CEGBW
- removed MX7: F6, custom-footprints:CherryMX_1.00u_PCB_KailhSocket_LTST-A683CEGBW
- removed MX8: F7, custom-footprints:CherryMX_1.00u_PCB_KailhSocket_LTST-A683CEGBW
- removed MX9: F8, custom-footprints:CherryMX_1.00u_PCB_KailhSocket_LTST-A683CEGBW
- removed OL1: OLED, kbd:OLED_v2
- removed R16, R18, R20, R21, R22, R25, R27, R38, R39: 10k, Resistor_SMD:R_0805_2012Metric
- removed R19: 1k, Resistor_SMD:R_0805_2012Metric
- removed R24, R45, R46, R47, R48, R49, R54, R59, R64, R65: 330, Resistor_SMD:R_0805_2012Metric
- removed R33, R36, R50, R56: 56K, Resistor_SMD:R_0805_2012Metric
- removed R34, R35, R40, R41, R42, R43, R52, R53: 22, Resistor_SMD:R_0805_2012Metric
- removed R57, R60, R62: 100k, Resistor_SMD:R_0603_1608Metric
- removed R58: 1.5k, Resistor_SMD:R_0805_2012Metric
- removed ROT1, ROT2: Rotary_Encoder_Switch, Rotary_Encoder:RotaryEncoder_Alps_EC11E-Switch_Vertical_H20mm
- removed SW1, SW2: SW_Push, random-keyboard-parts:SKQG-1155865
- removed U10, U8: PRTR5V0U2X, random-keyboard-parts:SOT143B
- removed U11, U9: MIC2505-1YM, custom-footprints:MIC2505
- removed U12: XC6206P332MR, Package_TO_SOT_SMD:SOT-23
- removed U13: 74LVC1G34, Package_TO_SOT_SMD:SOT-23-5
- removed U14: STM32F303CBT6, Package_QFP:LQFP-48_7x7mm_P0.5mm
- removed UD10, UD11, UD12, UD13, UD14, UD8, UD9: Amber, LED_SMD:LED_0805_2012Metric
- removed UD5, UD6, UD7: Green, LED_SMD:LED_0805_2012Metric
- removed USB5, USB7: HRO-TYPE-C-31-M-12, Type-C:HRO-TYPE-C-31-M-12-Assembly
- removed USB6: USB_A, random-keyboard-parts:USB-A-Generic
- removed Y2: 8MHz, Crystal:Crystal_SMD_HC49-SD
- added MX65: M4, CherryMX_PCB_KailhSocket_LTST-A683CEGBW:CherryMX_1.00u_PCB_KailhSocket_LTST-A683CEGBW, F.Cu at (88.9, 254.0)
- added MX66: LSHIFT, CherryMX_PCB_KailhSocket_StabWireBottom_LTST-A683CEGBW:CherryMX_2.25u_PCB_KailhSocket_StabWireBottom_LTST-A683CEGBW, F.Cu at (124.6, 254.0)
- added MX67: Z, CherryMX_PCB_KailhSocket_LTST-A683CEGBW:CherryMX_1.00u_PCB_KailhSocket_LTST-A683CEGBW, F.Cu at (155.6, 254.0)
- added MX68: X, CherryMX_PCB_KailhSocket_LTST-A683CEGBW:CherryMX_1.00u_PCB_KailhSocket_LTST-A683CEGBW, F.Cu at (174.6, 254.0)
- added MX69: C, CherryMX_PCB_KailhSocket_LTST-A683CEGBW:CherryMX_1.00u_PCB_KailhSocket_LTST-A683CEGBW, F.Cu at (193.7, 254.0)
- added MX70: V, CherryMX_PCB_KailhSocket_LTST-A683CEGBW:CherryMX_1.00u_PCB_KailhSocket_LTST-A683CEGBW, F.Cu at (212.7, 254.0)
- added MX71: B, CherryMX_PCB_KailhSocket_LTST-A683CEGBW:CherryMX_1.00u_PCB_KailhSocket_LTST-A683CEGBW, F.Cu at (231.8, 254.0)
- added MX72: N, CherryMX_PCB_KailhSocket_LTST-A683CEGBW:CherryMX_1.00u_PCB_KailhSocket_LTST-A683CEGBW, F.Cu at (250.8, 254.0)
- added MX73: M, CherryMX_PCB_KailhSocket_LTST-A683CEGBW:CherryMX_1.00u_PCB_KailhSocket_LTST-A683CEGBW, F.Cu at (269.9, 254.0)
- added MX74: ,/<, CherryMX_PCB_KailhSocket_LTST-A683CEGBW:CherryMX_1.00u_PCB_KailhSocket_LTST-A683CEGBW, F.Cu at (288.9, 254.0)
- added MX75: ./>, CherryMX_PCB_KailhSocket_LTST-A683CEGBW:CherryMX_1.00u_PCB_KailhSocket_LTST-A683CEGBW, F.Cu at (308.0, 254.0)
- added MX76: /, CherryMX_PCB_KailhSocket_LTST-A683CEGBW:CherryMX_1.00u_PCB_KailhSocket_LTST-A683CEGBW, F.Cu at (327.0, 254.0)
- added MX77: RSHIFT, CherryMX_PCB_KailhSocket_StabWireBottom_LTST-A683CEGBW:CherryMX_2.75u_PCB_KailhSocket_StabWireBottom_LTST-A683CEGBW, F.Cu at (362.7, 254.0)
- added MX79: M5, CherryMX_PCB_KailhSocket_LTST-A683CEGBW:CherryMX_1.00u_PCB_KailhSocket_LTST-A683CEGBW, F.Cu at (88.9, 273.0)
- added MX80: LCTRL, CherryMX_PCB_KailhSocket_LTST-A683CEGBW:CherryMX_1.25u_PCB_KailhSocket_LTST-A683CEGBW, F.Cu at (115.1, 273.0)
- added MX81: LGUI, CherryMX_PCB_KailhSocket_LTST-A683CEGBW:CherryMX_1.25u_PCB_KailhSocket_LTST-A683CEGBW, F.Cu at (138.9, 273.0)
- added MX82: LALT, CherryMX_PCB_KailhSocket_LTST-A683CEGBW:CherryMX_1.25u_PCB_KailhSocket_LTST-A683CEGBW, F.Cu at (162.7, 273.0)
- added MX85: RGUI, CherryMX_PCB_KailhSocket_LTST-A683CEGBW:CherryMX_1.25u_PCB_KailhSocket_LTST-A683CEGBW, F.Cu at (329.4, 273.0)
- added MX86: MENU, CherryMX_PCB_KailhSocket_LTST-A683CEGBW:CherryMX_1.25u_PCB_KailhSocket_LTST-A683CEGBW, F.Cu at (353.2, 273.0)
- added MX87: RCTRL, CherryMX_PCB_KailhSocket_LTST-A683CEGBW:CherryMX_1.25u_PCB_KailhSocket_LTST-A683CEGBW, F.Cu at (377.0, 273.0)
- added MX88: LEFT, CherryMX_PCB_KailhSocket_LTST-A683CEGBW:CherryMX_1.00u_PCB_KailhSocket_LTST-A683CEGBW, F.Cu at (408.0, 273.0)
- added MX89: DOWN, CherryMX_PCB_KailhSocket_LTST-A683CEGBW:CherryMX_1.00u_PCB_KailhSocket_LTST-A683CEGBW, F.Cu at (427.0, 273.0)
- added MX90: RIGHT, CherryMX_PCB_KailhSocket_LTST-A683CEGBW:CherryMX_1.00u_PCB_KailhSocket_LTST-A683CEGBW, F.Cu at (446.1, 273.0)
- added U3: PRTR5V0U2X, random-keyboard-parts:SOT143B, B.Cu at (131.8, 166.7)
- D+1, D+2, D+3, D+4, D-1, D-2, D-3, D-4: footprint TestPoint:TestPoint_Pad_1.0x1.0mm -> TestPoint:TestPoint_Pad_1.5x1.5mm
- MX53, MX63, MX78: footprint custom-footprints:CherryMX_1.00u_PCB_KailhSocket_LTST-A683CEGBW -> CherryMX_PCB_KailhSocket_LTST-A683CEGBW:CherryMX_1.00u_PCB_KailhSocket_LTST-A683CEGBW
- MX64: footprint custom-footprints:CherryMX_2.25u_PCB_KailhSocket_LTST-A683CEGBW -> CherryMX_PCB_KailhSocket_StabWireBottom_LTST-A683CEGBW:CherryMX_2.25u_PCB_KailhSocket_StabWireBottom_LTST-A683CEGBW
- MX83: footprint custom-footprints:CherryMX_6.25u_PCB_KailhSocket_LTST-A683CEGBW -> CherryMX_PCB_KailhSocket_StabWireTop_LTST-A683CEGBW:CherryMX_6.25u_PCB_KailhSocket_StabWireTop_LTST-A683CEGBW
- MX84: footprint custom-footprints:CherryMX_1.25u_PCB_KailhSocket_LTST-A683CEGBW -> CherryMX_PCB_KailhSocket_LTST-A683CEGBW:CherryMX_1.25u_PCB_KailhSocket_LTST-A683CEGBW
- R28: value 330 -> 100k; footprint Resistor_SMD:R_0805_2012Metric -> Resistor_SMD:R_0603_1608Metric
- U1: value SD00HA -> FE1.1s; footprint Package_TO_SOT_SMD:SOT-23-5 -> Package_SO:SSOP-28_3.9x9.9mm_P0.635mm
- moved R5 262.3 mm to (130.6, 176.2), turned to 90 degrees
- moved R6 261.9 mm to (132.9, 176.2), turned to 90 degrees
- moved FB15 185.9 mm to (388.9, 216.7)
- moved BOOT0 175.0 mm to (436.5, 242.9)
- moved R11 172.3 mm to (222.6, 177.0), turned to 270 degrees
- moved R9 170.9 mm to (225.0, 177.0), turned to 270 degrees
- moved USB2 156.9 mm to (222.2, 148.4), turned to 0 degrees
- moved FB7 152.5 mm to (230.2, 159.5)
- moved R14 143.8 mm to (226.3, 159.5)
- moved D1 140.7 mm to (214.3, 159.5), turned to 0 degrees
- moved F3 139.6 mm to (219.9, 164.3), turned to 90 degrees
- moved FB3 139.3 mm to (219.9, 169.1), turned to 90 degrees
- moved R2 137.9 mm to (210.3, 159.5), turned to 0 degrees
- moved C6 136.1 mm to (223.8, 164.3)
- moved U4 135.7 mm to (223.8, 168.3), turned to 180 degrees
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Connections:
- D2 pad 2: VBUS -> +5V
- FB1 pad 1: PORT1-4_PWR -> +5V
- FB3 pad 1: PORT1-4_PWR -> +5V
- FB6 pad 1: PORT1-4_PWR -> +5V
- R11 pad 1: Net-(D+2-Pad1) -> Net-(D-2-Pad1)
- R11 pad 2: HUB_PORT2_D+ -> HUB_PORT2_D-
- R28 pad 1: GND -> +3V3
- R28 pad 2: Net-(D6-Pad1) -> BUSJ
- R5 pad 1: Net-(D+3-Pad1) -> HUB_PORT3_D-
- R5 pad 2: HUB_PORT3_D+ -> Net-(D-3-Pad1)
- R51 pad 2: Net-(FE2.1-Pad27) -> Net-(R51-Pad2)
- R6 pad 1: Net-(D-3-Pad1) -> HUB_PORT3_D+
- R6 pad 2: HUB_PORT3_D- -> Net-(D+3-Pad1)
- R9 pad 1: Net-(D-2-Pad1) -> Net-(D+2-Pad1)
- R9 pad 2: HUB_PORT2_D- -> HUB_PORT2_D+
- U1 pad 1: Net-(D12-Pad2) -> GND
- U1 pad 2: GND -> HUB_XOUT
- U1 pad 3: Net-(U1-Pad3) -> HUB_XIN
- U1 pad 4: VBUS -> HUB_PORT4_D-
- U1 pad 5: VBUS -> HUB_PORT4_D+
- U2 pad 4: VBUS -> +5V
- UD3 pad 1: Net-(R46-Pad1) -> HUB_DRV
- UD3 pad 2: HUB_DRV -> Net-(R37-Pad1)
- UD4 pad 1: Net-(R47-Pad1) -> HUB_DRV
- UD4 pad 2: HUB_DRV -> Net-(R44-Pad1)
- USB1 pad 11: VBUS -> +5V
- USB1 pad 2: VBUS -> +5V
- USB1 pad 3: Net-(USB1-Pad3) -> (no net)
- USB1 pad 9: Net-(USB1-Pad9) -> (no net)
- USB2 pad 3: Net-(USB2-Pad3) -> (no net)
- USB2 pad 9: Net-(USB2-Pad9) -> (no net)
Routing:
- net GND: track 1973.6 -> 75.2 mm, vias 498 -> 244
- net ENCODER_A: track 676.2 -> 6.20 mm, vias 3 -> 1
- net PORT1-4_PWR: track 640.4 -> 0.00 mm, vias 2 -> 0
- net +5V: track 3215.7 -> 2764.6 mm, vias 21 -> 2
- net DOUT3: track 389.3 -> 0.00 mm, vias 2 -> 0
- net Net-(D+2-Pad1): track 375.0 -> 26.4 mm, vias 2 -> 0
- net Net-(D-2-Pad1): track 374.1 -> 28.8 mm, vias 2 -> 0
- net ENCODER_B1: track 343.8 -> 6.39 mm
- net Net-(D-3-Pad1): track 345.8 -> 16.7 mm, vias 2 -> 0
- net Net-(D+3-Pad1): track 344.6 -> 17.2 mm, vias 2 -> 0
- net BKL_DATA_IN_3V3: track 327.5 -> 8.53 mm, vias 1 -> 0
- net ENCODER_B2: track 301.7 -> 6.60 mm
- net PORT5-7PWR: track 274.5 -> 0.00 mm, vias 3 -> 0
- net ROW2: track 624.2 -> 389.0 mm, vias 4 -> 0
- net Net-(D+1-Pad1): track 242.3 -> 16.9 mm
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Other:
- board size 395.3 x 138.1 mm -> 3.4 x 3 mm
