File: PCB/custom_keyboard (f303).kicad_pcb (KiCad board)
At the start: 2 copper layers, 3.4 x 3 mm, 102 parts, among them U1 FE1.1s, U2 PRTR5V0U2X, U3 PRTR5V0U2X, U4 PRTR5V0U2X, U5 24LC04BT-I/SN, U6 PRTR5V0U2X, Y1 12MHz

Commit message: 2nd prototype
Parts:
- removed C12, C4, C6: 100uF, Capacitor_SMD:C_1206_3216Metric
- removed C14: 100nF, Capacitor_SMD:C_0805_2012Metric
- removed C15: 4.7uF, Capacitor_SMD:C_0805_2012Metric
- removed C2, C5: 22pF, Capacitor_SMD:C_0805_2012Metric
- removed C36, C37: 10uF, Capacitor_SMD:C_0805_2012Metric
- removed D+2, D+3, D+4, D-2, D-3, D-4: TestPoint_Small, TestPoint:TestPoint_Pad_1.5x1.5mm
- removed D1, D10, D5, D7: Red, LED_SMD:LED_0805_2012Metric
- removed F2, F3, F4: 500mA, Fuse:Fuse_1206_3216Metric
- removed FB1, FB3, FB4, FB6, FB7, FB9: 60 @ 100 MHz, Inductor_SMD:L_0805_2012Metric
- removed R10, R2, R30, R37, R44, R63: 330, Resistor_SMD:R_0805_2012Metric
- removed R11, R23, R26, R5, R6, R9: 22, Resistor_SMD:R_0805_2012Metric
- removed R14, R7: 56K, Resistor_SMD:R_0805_2012Metric
- removed R28, R29, R32: 100k, Resistor_SMD:R_0603_1608Metric
- removed R31: 47k, Resistor_SMD:R_0805_2012Metric
- removed R51: 2.7k, Resistor_SMD:R_0805_2012Metric
- removed U1: FE1.1s, Package_SO:SSOP-28_3.9x9.9mm_P0.635mm
- removed U3, U4, U6: PRTR5V0U2X, random-keyboard-parts:SOT143B
- removed U5: 24LC04BT-I/SN, custom-footprints:24LC04
- removed UD1, UD2, UD3, UD4: Green, LED_SMD:LED_0805_2012Metric
- removed USB2: HRO-TYPE-C-31-M-12, Type-C:HRO-TYPE-C-31-M-12-Assembly
- removed USB3, USB4: USB_A, random-keyboard-parts:USB-A-Generic
- removed Y1: 12MHz, Crystal:Crystal_SMD_3225-4Pin_3.2x2.5mm
- added BOOT1: TestPoint_Small, TestPoint:TestPoint_THTPad_D1.0mm_Drill0.5mm, B.Cu at (395.3, 241.3)
- added C1: 100uF, Capacitor_SMD:C_1206_3216Metric, B.Cu at (282.6, 178.6)
- added C13: 100nF, Capacitor_SMD:C_0805_2012Metric, B.Cu at (426.2, 231.0)
- added C18: 100nF, Capacitor_SMD:C_0805_2012Metric, B.Cu at (413.5, 252.4)
- added C19: 100nF, Capacitor_SMD:C_0805_2012Metric, B.Cu at (401.6, 241.3)
- added C20: 100nF, Capacitor_SMD:C_0805_2012Metric, B.Cu at (415.1, 238.9)
- added C21: 10uF, Capacitor_SMD:C_0805_2012Metric, B.Cu at (415.9, 252.4)
- added C22: 100nF, Capacitor_SMD:C_0805_2012Metric, B.Cu at (415.9, 248.4)
- added C23: 10nF, Capacitor_SMD:C_0805_2012Metric, B.Cu at (405.6, 254.0)
- added C24: 1uF, Capacitor_SMD:C_0805_2012Metric, B.Cu at (403.3, 254.0)
- added C3: 20pF, Capacitor_SMD:C_0805_2012Metric, B.Cu at (414.3, 257.2)
- added C43: 1uF, Capacitor_SMD:C_0805_2012Metric, B.Cu at (404.8, 234.9)
- added C44: 1uF, Capacitor_SMD:C_0805_2012Metric, B.Cu at (415.1, 231.0)
- added C7: 20pF, Capacitor_SMD:C_0805_2012Metric, B.Cu at (404.6, 257.2)
- added COL15: TestPoint_Small, TestPoint:TestPoint_THTPad_D1.0mm_Drill0.5mm, B.Cu at (400.8, 191.3)
- added D11: Red, LED_SMD:LED_0805_2012Metric, B.Cu at (417.5, 227.8)
- added ENCA1: TestPoint_Small, TestPoint:TestPoint_THTPad_D1.0mm_Drill0.5mm, B.Cu at (396.1, 250.8)
- added ENCB1: TestPoint_Small, TestPoint:TestPoint_THTPad_D1.0mm_Drill0.5mm, B.Cu at (397.6, 252.4)
- added ENCB2: TestPoint_Small, TestPoint:TestPoint_THTPad_D1.0mm_Drill0.5mm, B.Cu at (394.5, 249.2)
- added F1: 500mA, Fuse:Fuse_1206_3216Metric, B.Cu at (290.5, 178.6)
- added F8: 500mA, Fuse:Fuse_1206_3216Metric, B.Cu at (407.2, 231.8)
- added J1: Conn_01x04, Connector_PinSocket_2.54mm:PinSocket_1x04_P2.54mm_Vertical, B.Cu at (420.7, 233.3)
- added J2: Conn_01x04_Female, random-keyboard-parts:JST-SR-4, B.Cu at (396.9, 227.8)
- added MX27: -/_, CherryMX_PCB_KailhSocket_LTST-A683CEGBW:CherryMX_1.00u_PCB_KailhSocket_LTST-A683CEGBW, F.Cu at (322.2, 196.8)
- added MX28: =/+, CherryMX_PCB_KailhSocket_LTST-A683CEGBW:CherryMX_1.00u_PCB_KailhSocket_LTST-A683CEGBW, F.Cu at (341.3, 196.8)
- added MX29: BACKSPACE, CherryMX_PCB_KailhSocket_StabWireBottom_LTST-A683CEGBW:CherryMX_2.00u_PCB_KailhSocket_StabWireBottom_LTST-A683CEGBW, F.Cu at (369.9, 196.8)
- added R19: 1k, Resistor_SMD:R_0805_2012Metric, B.Cu at (440.5, 238.0)
- added R22: 10k, Resistor_SMD:R_0805_2012Metric, B.Cu at (428.6, 232.6)
- added R24: 330, Resistor_SMD:R_0805_2012Metric, B.Cu at (439.7, 229.4)
- added R25: 10k, Resistor_SMD:R_0805_2012Metric, B.Cu at (428.6, 239.7)
- added R27: 10k, Resistor_SMD:R_0805_2012Metric, B.Cu at (398.4, 241.3)
- added R38: 10k, Resistor_SMD:R_0805_2012Metric, B.Cu at (450.0, 238.9)
- added R58: 1.5k, Resistor_SMD:R_0805_2012Metric, B.Cu at (414.7, 234.1)
- added R64: 330, Resistor_SMD:R_0805_2012Metric, B.Cu at (415.1, 227.8)
- added SW1: SW_Push, random-keyboard-parts:SKQG-1155865, B.Cu at (434.2, 230.2)
- added SW2: SW_Push, random-keyboard-parts:SKQG-1155865, B.Cu at (434.2, 238.9)
- added U12: XC6206P332MR, Package_TO_SOT_SMD:SOT-23, B.Cu at (411.1, 230.2)
- added U13: 74LVC1G34, Package_TO_SOT_SMD:SOT-23-5, B.Cu at (400.0, 234.9)
- added U14: STM32F303CBT6, Package_QFP:LQFP-48_7x7mm_P0.5mm, B.Cu at (408.8, 245.3)
- added X1: TestPoint_Small, TestPoint:TestPoint_THTPad_D1.0mm_Drill0.5mm, B.Cu at (411.1, 256.4)
- added X2: TestPoint_Small, TestPoint:TestPoint_THTPad_D1.0mm_Drill0.5mm, B.Cu at (408.0, 256.4)
- added Y2: 8MHz, Crystal:Crystal_SMD_HC49-SD, B.Cu at (409.5, 261.1)
- moved R3 122.0 mm to (409.9, 234.1)
- moved R4 122.0 mm to (412.3, 234.1)
- moved FB15 21.3 mm to (404.0, 231.8), turned to 180 degrees
- moved R8 9.26 mm to (304.0, 164.3)
- moved D2 4.63 mm to (304.0, 161.9), turned to 180 degrees
- moved BOOT0 3.17 mm to (439.7, 242.9)
- moved D+1 2.38 mm to (309.5, 167.5)
- moved D-1 2.38 mm to (306.4, 167.5)
- moved U2 2.38 mm to (308.0, 162.7)
- moved FB5 0.79 mm to (315.9, 160.3)
- moved R12 0.79 mm to (311.9, 160.3)
Connections:
- net Net-(D+1-Pad1) renamed D+
- net Net-(D-1-Pad1) renamed D-
- R3 pad 2: HUB_D- -> KEYBOARD_D-
- R4 pad 2: HUB_D+ -> KEYBOARD_D+
Routing:
- net ENCODER_A: track 6.20 -> 487.0 mm, vias 1 -> 3
- net ENCODER_B1: track 6.39 -> 412.8 mm, vias 1 -> 2
- net DOUT3: track 0.00 -> 387.2 mm, vias 0 -> 2
- net BKL_DATA_IN: track 5.00 -> 349.1 mm
- net HUB_PORT3_D-: track 194.5 -> 0.00 mm
- net HUB_PORT3_D+: track 193.0 -> 0.00 mm
- net D-: track 19.7 -> 181.2 mm
- net D+: track 16.9 -> 178.3 mm
- net ENCODER_B2: track 6.60 -> 155.2 mm, vias 1 -> 2
- net HUB_PORT4_D+: track 134.0 -> 0.00 mm
- net +5V: track 2764.6 -> 2897.3 mm, vias 2 -> 8
- net HUB_PORT4_D-: track 132.5 -> 0.00 mm
- net COL17: track 104.2 -> 231.6 mm
- net HUB_PORT2_D-: track 95.9 -> 0.00 mm
- net HUB_PORT2_D+: track 94.4 -> 0.00 mm
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Other:
- board text removed: "GND"
- board text removed: "JLCJLCJLCJLC"
- board text removed: "SWCLK"
- board text removed: "SWDIO"
