File: PCB/_autosave-custom_keyboard (f303).sch (KiCad schematic (older format))
At the start: 363 parts, among them J1 Conn_01x04, J2 SM04B-SRSS-TB(LF)(SN), SW1 SW_Push, SW2 SW_Push, U1 SRV05-4, U12 XC6206P332MR, U13 74LVC1G34, U14 STM32F303CBT6, X1 TestPoint_Small, X2 TestPoint_Small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

Commit message: Changed ESD protection IC
Connections:
- net +5V: no longer D2.2 (A), F1.2, FB15.2, J2.1 (Pin_1), U1.5 (VP), USB1.11 (VBUS), USB1.2 (VBUS)
- new net VBUS: D2.2 (A), F1.2, FB15.2, J2.1 (Pin_1), U1.5 (VP), USB1.11 (VBUS), USB1.2 (VBUS)
- no-connect marks 4 -> 6
Other:
- moved on the sheet: C1, F1
Changed lines of the file:
@@
 $EndComp
 Wire Wire Line
-	22250 12750 22250 12400
-Wire Wire Line
 	22550 12750 22250 12750
 Text Notes 22700 12150 0    118  ~ 24
@@
 Wire Wire Line
 	16250 15850 16250 16050
-$Comp
-L power:+5V #PWR0261
-U 1 1 96041F90
-P 22250 12400
-F 0 "#PWR0261" H 22250 12250 50  0001 C CNN
-F 1 "+5V" H 22100 12450 50  0000 C CNN
-F 2 "" H 22250 12400 50  0001 C CNN
-F 3 "" H 22250 12400 50  0001 C CNN
-	1    22250 12400
-	-1   0    0    -1
-$EndComp
 Wire Wire Line
 	22650 13300 22650 13250
@@
 	1    0    0    -1
 $EndComp
-$Comp
-L power:+5V #PWR01
-U 1 1 6409DD35
-P 3900 2250
-F 0 "#PWR01" H 3900 2100 50  0001 C CNN
-F 1 "+5V" H 4000 2350 50  0000 C CNN
-F 2 "" H 3900 2250 50  0001 C CNN
-F 3 "" H 3900 2250 50  0001 C CNN
-	1    3900 2250
-	1    0    0    -1
-$EndComp
 Text Notes 14700 2150 0    276  ~ 55
 Keyboard Matrix\n
@@
 P 4700 2250
 F 0 "#PWR02" H 4700 2100 50  0001 C CNN
-F 1 "+5V" H 4800 2350 50  0000 C CNN
+F 1 "+5V" H 4800 2300 50  0000 C CNN
 F 2 "" H 4700 2250 50  0001 C CNN
 F 3 "" H 4700 2250 50  0001 C CNN
@@
 L Device:Polyfuse_Small F1
 U 1 1 636D2008
-P 4300 2350
-F 0 "F1" V 4095 2350 50  0000 C CNN
-F 1 "500mA" V 4186 2350 50  0000 C CNN
-F 2 "Fuse:Fuse_1206_3216Metric" H 4350 2150 50  0001 L CNN
-F 3 "~" H 4300 2350 50  0001 C CNN
-F 4 "C70069" H 4300 2350 50  0001 C CNN "LCSC Part"
-	1    4300 2350
+P 4200 2350
+F 0 "F1" V 3995 2350 50  0000 C CNN
+F 1 "500mA" V 4086 2350 50  0000 C CNN
+F 2 "Fuse:Fuse_1206_3216Metric" H 4250 2150 50  0001 L CNN
+F 3 "~" H 4200 2350 50  0001 C CNN
+F 4 "C70069" H 4200 2350 50  0001 C CNN "LCSC Part"
+	1    4200 2350
 	0    1    1    0
 $EndComp
 Wire Wire Line
-	4150 2350 3900 2350
-Connection ~ 4150 2350
+	4400 2450 4400 2350
 Wire Wire Line
-	4150 2450 4150 2350
-Wire Wire Line
-	4150 2700 4150 2650
+	4400 2700 4400 2650
 $Comp
 L Device:C_Small C1
 U 1 1 61F55865
-P 4150 2550
-F 0 "C1" H 4000 2600 50  0000 C CNN
-F 1 "100uF" H 3950 2500 50  0000 C CNN
-F 2 "Capacitor_SMD:C_1206_3216Metric" H 4150 2550 50  0001 C CNN
-F 3 "~" H 4150 2550 50  0001 C CNN
-F 4 "C15008" H 4150 2550 50  0001 C CNN "LCSC Part"
-	1    4150 2550
-	-1   0    0    -1
+P 4400 2550
+F 0 "C1" H 4250 2600 50  0000 C CNN
+F 1 "100uF" H 4200 2500 50  0000 C CNN
+F 2 "Capacitor_SMD:C_1206_3216Metric" H 4400 2550 50  0001 C CNN
+F 3 "~" H 4400 2550 50  0001 C CNN
+F 4 "C15008" H 4400 2550 50  0001 C CNN "LCSC Part"
+	1    4400 2550
+	1    0    0    -1
 $EndComp
 $Comp
 L power:GND #PWR03
 U 1 1 61F51D49
-P 4150 2700
-F 0 "#PWR03" H 4150 2450 50  0001 C CNN
-F 1 "GND" H 4000 2650 50  0000 C CNN
-F 2 "" H 4150 2700 50  0001 C CNN
-F 3 "" H 4150 2700 50  0001 C CNN
-	1    4150 2700
+P 4400 2700
+F 0 "#PWR03" H 4400 2450 50  0001 C CNN
+F 1 "GND" H 4250 2650 50  0000 C CNN
+F 2 "" H 4400 2700 50  0001 C CNN
+F 3 "" H 4400 2700 50  0001 C CNN
+	1    4400 2700
 	-1   0    0    -1
 $EndComp
 Wire Wire Line
-	4400 2350 4700 2350
-Wire Wire Line
 	4700 2350 4700 2250
 Wire Wire Line
 	3900 2350 3900 2250
-Wire Wire Line
-	4200 2350 4150 2350
 Text Notes 3850 1950 0    118  ~ 24
 LED Fuse
@@
 	0    1    1    0
 $EndComp
-$Comp
-L power:+5V #PWR0184
-U 1 1 FBAA197C
-P 17050 12450
-F 0 "#PWR0184" H 17050 12300 50  0001 C CNN
-F 1 "+5V" H 16900 12500 50  0000 C CNN
-F 2 "" H 17050 12450 50  0001 C CNN
-F 3 "" H 17050 12450 50  0001 C CNN
-	1    17050 12450
-	-1   0    0    -1
-$EndComp
 Text GLabel 13800 12600 0    50   Input ~ 0
 ROT2_COL
@@
 D+
 $Comp
-L power:+5V #PWR0188
-U 1 1 625E1919
-P 20950 12550
-F 0 "#PWR0188" H 20950 12400 50  0001 C CNN
-F 1 "+5V" H 20800 12600 50  0000 C CNN
-F 2 "" H 20950 12550 50  0001 C CNN
-F 3 "" H 20950 12550 50  0001 C CNN
-	1    20950 12550
-	1    0    0    -1
-$EndComp
-$Comp
 L power:GND #PWR0189
 U 1 1 625E2145
@@
 	17550 13300 17700 13300
 $Comp
-L power:+5V #PWR0185
-U 1 1 66B49E7A
-P 17700 13200
-F 0 "#PWR0185" H 17700 13050 50  0001 C CNN
-F 1 "+5V" H 17550 13250 50  0000 C CNN
-F 2 "" H 17700 13200 50  0001 C CNN
-F 3 "" H 17700 13200 50  0001 C CNN
-	1    17700 13200
-	1    0    0    -1
-$EndComp
-$Comp
 L Device:Ferrite_Bead_Small FB5
 U 1 1 66EC0E90
@@
 $EndComp
 $Comp
-L power:GND #PWR?
+L power:GND #PWR0186
 U 1 1 6A8298AD
 P 18050 13700
-F 0 "#PWR?" H 18050 13450 50  0001 C CNN
+F 0 "#PWR0186" H 18050 13450 50  0001 C CNN
 F 1 "GND" H 18055 13527 50  0000 C CNN
 F 2 "" H 18050 13700 50  0001 C CNN
@@
 Wire Wire Line
 	17550 13500 18100 13500
+Wire Wire Line
+	22250 12500 22250 12750
+$Comp
+L power:VBUS #PWR0184
+U 1 1 6D549303
+P 17050 12450
+F 0 "#PWR0184" H 17050 12300 50  0001 C CNN
+F 1 "VBUS" H 17065 12623 50  0000 C CNN
+F 2 "" H 17050 12450 50  0001 C CNN
+F 3 "" H 17050 12450 50  0001 C CNN
+	1    17050 12450
+	1    0    0    -1
+$EndComp
+$Comp
+L power:VBUS #PWR0185
+U 1 1 6D549A45
+P 17700 13200
+F 0 "#PWR0185" H 17700 13050 50  0001 C CNN
+F 1 "VBUS" H 17550 13250 50  0000 C CNN
+F 2 "" H 17700 13200 50  0001 C CNN
+F 3 "" H 17700 13200 50  0001 C CNN
+	1    17700 13200
+	1    0    0    -1
+$EndComp
+$Comp
+L power:VBUS #PWR0188
+U 1 1 6D54A565
+P 20950 12550
+F 0 "#PWR0188" H 20950 12400 50  0001 C CNN
+F 1 "VBUS" H 20800 12600 50  0000 C CNN
+F 2 "" H 20950 12550 50  0001 C CNN
+F 3 "" H 20950 12550 50  0001 C CNN
+	1    20950 12550
+	1    0    0    -1
+$EndComp
+$Comp
+L power:VBUS #PWR0190
+U 1 1 6D54AB68
+P 22250 12500
+F 0 "#PWR0190" H 22250 12350 50  0001 C CNN
+F 1 "VBUS" H 22400 12550 50  0000 C CNN
+F 2 "" H 22250 12500 50  0001 C CNN
+F 3 "" H 22250 12500 50  0001 C CNN
+	1    22250 12500
+	1    0    0    -1
+$EndComp
+$Comp
+L power:VBUS #PWR0191
+U 1 1 6D54B729
+P 3900 2250
+F 0 "#PWR0191" H 3900 2100 50  0001 C CNN
+F 1 "VBUS" H 3750 2300 50  0000 C CNN
+F 2 "" H 3900 2250 50  0001 C CNN
+F 3 "" H 3900 2250 50  0001 C CNN
+	1    3900 2250
+	1    0    0    -1
+$EndComp
+NoConn ~ 20450 13150
+NoConn ~ 21450 12950
+$Comp
+L power:PWR_FLAG #FLG0102
+U 1 1 6DF1D92B
+P 4700 2350
+F 0 "#FLG0102" H 4700 2425 50  0001 C CNN
+F 1 "PWR_FLAG" H 4700 2523 50  0000 C CNN
+F 2 "" H 4700 2350 50  0001 C CNN
+F 3 "~" H 4700 2350 50  0001 C CNN
+	1    4700 2350
+	-1   0    0    1
+$EndComp
+Wire Wire Line
+	4100 2350 3900 2350
+Connection ~ 4700 2350
+Connection ~ 4400 2350
+Wire Wire Line
+	4400 2350 4700 2350
+Wire Wire Line
+	4300 2350 4400 2350
 $EndSCHEMATC
