File: PCB/custom_keyboard (f303).sch (KiCad schematic (older format))
At the start: 361 parts, among them J1 Conn_01x04, J2 SM04B-SRSS-TB(LF)(SN), SW1 SW_Push, SW2 SW_Push, U1 SRV05-4, U12 XC6206P332MR, U13 74LVC1G34, U14 STM32F303CBT6, X1 TestPoint_Small, X2 TestPoint_Small, Y2 8MHz

Commit message: Adding IS31FL3731 RGB matrix
Parts:
- removed R22, R25: 10k, Resistor_SMD:R_0805_2012Metric, symbol Device:R_Small
- removed R24: 510, Resistor_SMD:R_0805_2012Metric, symbol Device:R_Small
- removed SW2: SW_Push, random-keyboard-parts:SKQG-1155865, symbol Switch:SW_Push
- added C10, C12, C4, C5: 1uF, Capacitor_SMD:C_0805_2012Metric, symbol Device:C_Small
- added C11, C6: 100nF, Capacitor_SMD:C_0805_2012Metric, symbol Device:C_Small
- added C2: 4.7uF, Capacitor_SMD:C_0805_2012Metric, symbol Device:C_Small
- added I1, I2, I3: IS31FL3731-QFLS2, Package_DFN_QFN:QFN-28-1EP_4x4mm_P0.4mm_EP2.3x2.3mm, symbol random-keyboard-parts:IS31FL3731-QFLS2
- added LED1, LED10, LED11, LED12, LED13, LED14, LED15, LED16, LED17, LED18, LED19, LED2, LED20, LED21, LED22, LED23, LED24, LED25, LED26, LED27, LED28, LED29, LED3, LED30, LED31, LED32, LED4, LED5, LED6, LED7, LED8, LED9: RGB-6028, random-keyboard-parts:RGB-6028, symbol random-keyboard-parts:RGB-6028
- added Q1: 2N7002, Package_TO_SOT_SMD:SOT-23, symbol Transistor_FET:2N7002
- added R10, R16, R17, R7: 100k, Resistor_SMD:R_0805_2012Metric, symbol Device:R_Small
- added R11, R18: 20k, Resistor_SMD:R_0805_2012Metric, symbol Device:R_Small
- added R14, R15, R9: 4.7k, Resistor_SMD:R_0805_2012Metric, symbol Device:R_Small
- added R5, R6: 10k, Resistor_SMD:R_0805_2012Metric, symbol Device:R_Small
- R19: value 1k -> 20k; LCSC Part C17513 -> C17798
- R38, R39: value 10k -> 4.7k; LCSC Part C17414 -> C17673
- SW1: LCSC Part C318884 -> (none)
Connections:
- net +3V3: now also SW1.2, R14.1, R15.1, R5.1, R9.1; no longer R19.1
- net BOOT0: now also SW1.1, C2.2, R6.1
- net GND: now also R19.1, C10.2, C11.2, C12.2, C4.2, C5.2, C6.2, I1.29 (Thermal), I1.5 (GND), I2.29 (Thermal), I2.5 (GND), I3.29 (Thermal), I3.5 (GND), Q1.2 (S), R10.2, R11.1, R16.2, R17.2, R18.1, R6.2, R7.2
- net KEYBOARD_RESET: now also C4.1, Q1.3 (D), R5.2; no longer C13.1, SW1.2
- net VCC: no longer C43.1, F8.1, OL1.3 (VCC), U12.3 (VI)
- net at R19.2: now also I3.6 (R_EXT)
- net KEYBOARD_SCL renamed SCL
- net SCL: now also I1.18 (AD), I1.20 (SCL), I2.20 (SCL), I3.20 (SCL)
- net KEYBOARD_SDA renamed SDA
- net SDA: now also I1.19 (SDA), I2.18 (AD), I2.19 (SDA), I3.19 (SDA)
- new net: C2.1, Q1.1 (G), R7.1
- new net: I1.6 (R_EXT), R11.2
- new net: I2.6 (R_EXT), R18.2
- new net 1CA1: I1.21 (CA1), LED1.2 (C), LED2.2 (C), LED3.2 (C), LED4.2 (C), LED5.2 (C), LED6.2 (C), LED7.2 (C), LED8.2 (C), LED9.1 (A), LED9.1 (A), LED9.1 (A)
- new net 1CA2: I1.22 (CA2), LED1.1 (A), LED1.1 (A), LED1.1 (A), LED10.1 (A), LED10.1 (A), LED10.1 (A), LED2.3 (C), LED3.3 (C), LED4.3 (C), LED5.3 (C), LED6.3 (C), LED7.3 (C), LED8.3 (C)
- new net 1CA3: I1.23 (CA3), LED1.3 (C), LED11.1 (A), LED11.1 (A), LED11.1 (A), LED2.1 (A), LED2.1 (A), LED2.1 (A), LED3.4 (C), LED4.4 (C), LED5.4 (C), LED6.4 (C), LED7.4 (C), LED8.4 (C)
- new net 1CA4: I1.24 (CA4), LED1.4 (C), LED12.1 (A), LED12.1 (A), LED12.1 (A), LED2.4 (C), LED3.1 (A), LED3.1 (A), LED3.1 (A)
- new net 1CA5: I1.25 (CA5), LED13.1 (A), LED13.1 (A), LED13.1 (A), LED4.1 (A), LED4.1 (A), LED4.1 (A)
- new net 1CA6: I1.26 (CA6), LED14.1 (A), LED14.1 (A), LED14.1 (A), LED15.4 (C), LED16.4 (C), LED5.1 (A), LED5.1 (A), LED5.1 (A)
- new net 1CA7: I1.27 (CA7), LED10.4 (C), LED11.4 (C), LED12.4 (C), LED13.4 (C), LED14.4 (C), LED15.1 (A), LED15.1 (A), LED15.1 (A), LED16.3 (C), LED6.1 (A), LED6.1 (A), LED6.1 (A), LED9.4 (C)
- new net 1CA8: I1.28 (CA8), LED10.3 (C), LED11.3 (C), LED12.3 (C), LED13.3 (C), LED14.3 (C), LED15.3 (C), LED16.1 (A), LED16.1 (A), LED16.1 (A), LED7.1 (A), LED7.1 (A), LED7.1 (A), LED9.3 (C)
- new net 1CA9: I1.1 (CA9), LED10.2 (C), LED11.2 (C), LED12.2 (C), LED13.2 (C), LED14.2 (C), LED15.2 (C), LED16.2 (C), LED8.1 (A), LED8.1 (A), LED8.1 (A), LED9.2 (C)
- new net 1CB1: I1.7 (CB1), LED17.2 (C), LED18.2 (C), LED19.2 (C), LED20.2 (C), LED21.2 (C), LED22.2 (C), LED23.2 (C), LED24.2 (C), LED25.1 (A), LED25.1 (A), LED25.1 (A)
- new net 1CB2: I1.8 (CB2), LED17.1 (A), LED17.1 (A), LED17.1 (A), LED18.3 (C), LED19.3 (C), LED20.3 (C), LED21.3 (C), LED22.3 (C), LED23.3 (C), LED24.3 (C), LED26.1 (A), LED26.1 (A), LED26.1 (A)
- new net 1CB3: I1.9 (CB3), LED17.3 (C), LED18.1 (A), LED18.1 (A), LED18.1 (A), LED19.4 (C), LED20.4 (C), LED21.4 (C), LED22.4 (C), LED23.4 (C), LED24.4 (C), LED27.1 (A), LED27.1 (A), LED27.1 (A)
- new net 1CB4: I1.10 (CB4), LED17.4 (C), LED18.4 (C), LED19.1 (A), LED19.1 (A), LED19.1 (A), LED28.1 (A), LED28.1 (A), LED28.1 (A)
- new net 1CB5: I1.11 (CB5), LED20.1 (A), LED20.1 (A), LED20.1 (A), LED29.1 (A), LED29.1 (A), LED29.1 (A)
- new net 1CB6: I1.12 (CB6), LED21.1 (A), LED21.1 (A), LED21.1 (A), LED30.1 (A), LED30.1 (A), LED30.1 (A), LED31.4 (C), LED32.4 (C)
- new net 1CB7: I1.13 (CB7), LED22.1 (A), LED22.1 (A), LED22.1 (A), LED25.4 (C), LED26.4 (C), LED27.4 (C), LED28.4 (C), LED29.4 (C), LED30.4 (C), LED31.1 (A), LED31.1 (A), LED31.1 (A), LED32.3 (C)
- new net 1CB8: I1.14 (CB8), LED23.1 (A), LED23.1 (A), LED23.1 (A), LED25.3 (C), LED26.3 (C), LED27.3 (C), LED28.3 (C), LED29.3 (C), LED30.3 (C), LED31.3 (C), LED32.1 (A), LED32.1 (A), LED32.1 (A)
- new net 1CB9: I1.15 (CB9), LED24.1 (A), LED24.1 (A), LED24.1 (A), LED25.2 (C), LED26.2 (C), LED27.2 (C), LED28.2 (C), LED29.2 (C), LED30.2 (C), LED31.2 (C), LED32.2 (C)
- new net 2CA1: I2.21 (CA1)
- new net 2CA2: I2.22 (CA2)
- new net 2CA3: I2.23 (CA3)
- new net 2CA4: I2.24 (CA4)
- new net 2CA5: I2.25 (CA5)
- new net 2CA6: I2.26 (CA6)
- new net 2CA7: I2.27 (CA7)
- new net 2CA8: I2.28 (CA8)
- new net 2CA9: I2.1 (CA9)
- new net 2CB1: I2.7 (CB1)
- new net 2CB2: I2.8 (CB2)
- new net 2CB3: I2.9 (CB3)
- new net 2CB4: I2.10 (CB4)
- new net 2CB5: I2.11 (CB5)
- new net 2CB6: I2.12 (CB6)
- new net 2CB7: I2.13 (CB7)
- new net 2CB8: I2.14 (CB8)
- new net 2CB9: I2.15 (CB9)
- new net 3CA1: I3.21 (CA1)
- new net 3CA2: I3.22 (CA2)
- new net 3CA3: I3.23 (CA3)
- new net 3CA4: I3.24 (CA4)
- new net 3CA5: I3.25 (CA5)
- new net 3CA6: I3.26 (CA6)
- new net 3CA7: I3.27 (CA7)
- new net 3CA8: I3.28 (CA8)
- new net 3CA9: I3.1 (CA9)
- new net 3CB1: I3.7 (CB1)
- new net 3CB2: I3.8 (CB2)
- new net 3CB3: I3.9 (CB3)
- new net 3CB4: I3.10 (CB4)
- new net 3CB5: I3.11 (CB5)
- new net 3CB6: I3.12 (CB6)
- new net 3CB7: I3.13 (CB7)
- new net 3CB8: I3.14 (CB8)
- new net 3CB9: I3.15 (CB9)
- new net INTB: I1.4 (INTB), I2.4 (INTB), I3.4 (INTB), R14.2, R15.2, R9.2
- new net KEYBOARD_5V: C10.1, C11.1, C12.1, C13.1, C43.1, C5.1, C6.1, F8.1, I1.2 (VCC), I2.2 (VCC), I3.18 (AD), I3.2 (VCC), OL1.3 (VCC), U12.3 (VI)
- new net SDB: I1.3 (SDB), I2.3 (SDB), I3.3 (SDB), R10.1, R16.1, R17.1
- no-connect marks 6 -> 12
Other:
- moved on the sheet: BKL3, BKL5, BOOT0, BOOT1, C1, C18, C19, C20, C21, C22, C23, C24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

Commit message: Replaced keyboard matrix schematic
Parts:
- removed LC1, LC10, LC11, LC12, LC13, LC14, LC15, LC16, LC17, LC18, LC19, LC2, LC20, LC21, LC22, LC23, LC24, LC25, LC26, LC27, LC28, LC29, LC3, LC30, LC31, LC32, LC33, LC34, LC35, LC36, LC37, LC38, LC39, LC4, LC40, LC41, LC42, LC43, LC44, LC45, LC46, LC47, LC48, LC49, LC5, LC50, LC51, LC52, LC53, LC54, LC55, LC56, LC57, LC58, LC59, LC6, LC60, LC61, LC62, LC63, LC64, LC65, LC66, LC67, LC68, LC69, LC7, LC70, LC71, LC72, LC73, LC74, LC75, LC76, LC77, LC78, LC79, LC8, LC80, LC81, LC82, LC83, LC84, LC85, LC86, LC87, LC88, LC89, LC9, LC90: 10uF, Capacitor_SMD:C_0805_2012Metric, symbol Device:C_Small
- removed R1: 470, Resistor_SMD:R_0805_2012Metric, symbol Device:R_Small
- MX1, MX10, MX11, MX12, MX13, MX14, MX15, MX16, MX17, MX18, MX19, MX2, MX20, MX21, MX22, MX23, MX24, MX25, MX26, MX27, MX28, MX3, MX30, MX31, MX32, MX33, MX35, MX36, MX37, MX38, MX39, MX4, MX40, MX41, MX42, MX43, MX44, MX45, MX46, MX48, MX49, MX5, MX50, MX51, MX53, MX54, MX55, MX56, MX57, MX58, MX59, MX6, MX60, MX61, MX62, MX63, MX65, MX67, MX68, MX69, MX7, MX70, MX71, MX72, MX73, MX74, MX75, MX76, MX78, MX79, MX8, MX88, MX89, MX9, MX90: footprint CherryMX_PCB_KailhSocket_LTST-A683CEGBW:CherryMX_1.00u_PCB_KailhSocket_LTST-A683CEGBW -> MX_Only:MXOnly-1U-Hotswap; symbol CherryMX:CherryMX_LTST-A683CEGBW -> CherryMX:CherryMX
- MX29: footprint CherryMX_PCB_KailhSocket_StabWireBottom_LTST-A683CEGBW:CherryMX_2.00u_PCB_KailhSocket_StabWireBottom_LTST-A683CEGBW -> MX_Only:MXOnly-2U-Hotswap; symbol CherryMX:CherryMX_LTST-A683CEGBW -> CherryMX:CherryMX
- MX34, MX47: footprint CherryMX_PCB_KailhSocket_LTST-A683CEGBW:CherryMX_1.50u_PCB_KailhSocket_LTST-A683CEGBW -> MX_Only:MXOnly-1.5U-Hotswap; symbol CherryMX:CherryMX_LTST-A683CEGBW -> CherryMX:CherryMX
- MX52: footprint CherryMX_PCB_KailhSocket_LTST-A683CEGBW:CherryMX_1.75u_PCB_KailhSocket_LTST-A683CEGBW -> MX_Only:MXOnly-1.75U-Hotswap; symbol CherryMX:CherryMX_LTST-A683CEGBW -> CherryMX:CherryMX
- MX64, MX66: footprint CherryMX_PCB_KailhSocket_StabWireBottom_LTST-A683CEGBW:CherryMX_2.25u_PCB_KailhSocket_StabWireBottom_LTST-A683CEGBW -> MX_Only:MXOnly-2.25U-Hotswap; symbol CherryMX:CherryMX_LTST-A683CEGBW -> CherryMX:CherryMX
- MX77: footprint CherryMX_PCB_KailhSocket_StabWireBottom_LTST-A683CEGBW:CherryMX_2.75u_PCB_KailhSocket_StabWireBottom_LTST-A683CEGBW -> MX_Only:MXOnly-2.75U-Hotswap; symbol CherryMX:CherryMX_LTST-A683CEGBW -> CherryMX:CherryMX
- MX80, MX81, MX82, MX84, MX85, MX86, MX87: footprint CherryMX_PCB_KailhSocket_LTST-A683CEGBW:CherryMX_1.25u_PCB_KailhSocket_LTST-A683CEGBW -> MX_Only:MXOnly-1.25U-Hotswap; symbol CherryMX:CherryMX_LTST-A683CEGBW -> CherryMX:CherryMX
- MX83: footprint CherryMX_PCB_KailhSocket_StabWireBottom_LTST-A683CEGBW:CherryMX_6.25u_PCB_KailhSocket_StabWireBottom_LTST-A683CEGBW -> MX_Only:MXOnly-6.25U-Hotswap; symbol CherryMX:CherryMX_LTST-A683CEGBW -> CherryMX:CherryMX
Connections:
- net +5V: no longer MX1.6 (VDD), MX10.6 (VDD), MX11.6 (VDD), MX12.6 (VDD), MX13.6 (VDD), MX14.6 (VDD), MX15.6 (VDD), MX16.6 (VDD), MX17.6 (VDD), MX18.6 (VDD), MX19.6 (VDD), MX2.6 (VDD), MX20.6 (VDD), MX21.6 (VDD), MX22.6 (VDD), MX23.6 (VDD), MX24.6 (VDD), MX25.6 (VDD), MX26.6 (VDD), MX27.6 (VDD), MX28.6 (VDD), MX29.6 (VDD), MX3.6 (VDD), MX30.6 (VDD), MX31.6 (VDD), MX32.6 (VDD), MX33.6 (VDD), MX34.6 (VDD), MX35.6 (VDD), MX36.6 (VDD), MX37.6 (VDD), MX38.6 (VDD), MX39.6 (VDD), MX4.6 (VDD), MX40.6 (VDD), MX41.6 (VDD), MX42.6 (VDD), MX43.6 (VDD), MX44.6 (VDD), MX45.6 (VDD), MX46.6 (VDD), MX47.6 (VDD), MX48.6 (VDD), MX49.6 (VDD), MX5.6 (VDD), MX50.6 (VDD), MX51.6 (VDD), MX52.6 (VDD), MX53.6 (VDD), MX54.6 (VDD), MX55.6 (VDD), MX56.6 (VDD), MX57.6 (VDD), MX58.6 (VDD), MX59.6 (VDD), MX6.6 (VDD), MX60.6 (VDD), MX61.6 (VDD), MX62.6 (VDD), MX63.6 (VDD), MX64.6 (VDD), MX65.6 (VDD), MX66.6 (VDD), MX67.6 (VDD), MX68.6 (VDD), MX69.6 (VDD), MX7.6 (VDD), MX70.6 (VDD), MX71.6 (VDD), MX72.6 (VDD), MX73.6 (VDD), MX74.6 (VDD), MX75.6 (VDD), MX76.6 (VDD), MX77.6 (VDD), MX78.6 (VDD), MX79.6 (VDD), MX8.6 (VDD), MX80.6 (VDD), MX81.6 (VDD), MX82.6 (VDD), MX83.6 (VDD), MX84.6 (VDD), MX85.6 (VDD), MX86.6 (VDD), MX87.6 (VDD), MX88.6 (VDD), MX89.6 (VDD), MX9.6 (VDD), MX90.6 (VDD)
- net COL11: no longer MX44.1
- net COL17: no longer MX32.1, MX50.1
- net GND: no longer MX1.3 (VSS), MX10.3 (VSS), MX11.3 (VSS), MX12.3 (VSS), MX13.3 (VSS), MX14.3 (VSS), MX15.3 (VSS), MX16.3 (VSS), MX17.3 (VSS), MX18.3 (VSS), MX19.3 (VSS), MX2.3 (VSS), MX20.3 (VSS), MX21.3 (VSS), MX22.3 (VSS), MX23.3 (VSS), MX24.3 (VSS), MX25.3 (VSS), MX26.3 (VSS), MX27.3 (VSS), MX28.3 (VSS), MX29.3 (VSS), MX3.3 (VSS), MX30.3 (VSS), MX31.3 (VSS), MX32.3 (VSS), MX33.3 (VSS), MX34.3 (VSS), MX35.3 (VSS), MX36.3 (VSS), MX37.3 (VSS), MX38.3 (VSS), MX39.3 (VSS), MX4.3 (VSS), MX40.3 (VSS), MX41.3 (VSS), MX42.3 (VSS), MX43.3 (VSS), MX44.3 (VSS), MX45.3 (VSS), MX46.3 (VSS), MX47.3 (VSS), MX48.3 (VSS), MX49.3 (VSS), MX5.3 (VSS), MX50.3 (VSS), MX51.3 (VSS), MX52.3 (VSS), MX53.3 (VSS), MX54.3 (VSS), MX55.3 (VSS), MX56.3 (VSS), MX57.3 (VSS), MX58.3 (VSS), MX59.3 (VSS), MX6.3 (VSS), MX60.3 (VSS), MX61.3 (VSS), MX62.3 (VSS), MX63.3 (VSS), MX64.3 (VSS), MX65.3 (VSS), MX66.3 (VSS), MX67.3 (VSS), MX68.3 (VSS), MX69.3 (VSS), MX7.3 (VSS), MX70.3 (VSS), MX71.3 (VSS), MX72.3 (VSS), MX73.3 (VSS), MX74.3 (VSS), MX75.3 (VSS), MX76.3 (VSS), MX77.3 (VSS), MX78.3 (VSS), MX79.3 (VSS), MX8.3 (VSS), MX80.3 (VSS), MX81.3 (VSS), MX82.3 (VSS), MX83.3 (VSS), MX84.3 (VSS), MX85.3 (VSS), MX86.3 (VSS), MX87.3 (VSS), MX88.3 (VSS), MX89.3 (VSS), MX9.3 (VSS), MX90.3 (VSS)
- net ROW2: no longer KD44.1 (K)
- net at MX44.2: no longer KD44.2 (A)
- removed net DOUT1: MX14.5 (DOUT), MX15.4 (DIN)
- removed net DOUT2: MX32.5 (DOUT), MX33.4 (DIN)
- removed net DOUT3: MX50.5 (DOUT), MX51.4 (DIN)
- removed net DOUT4: MX64.5 (DOUT), MX65.4 (DIN)
- removed net DOUT5: MX78.5 (DOUT), MX79.4 (DIN)
- no-connect marks 12 -> 11
Other:
- moved on the sheet: C5, C6, I1, KD1, KD10, KD11, KD12, KD13, KD14, KD15, KD16, KD17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

Commit message: Fixed issues with matrix
Connections:
- net COL11: now also MX44.1
- net ROW2: now also KD44.1 (K)
- net at MX44.2: now also KD44.2 (A)
Other:
- moved on the sheet: C10, C11, C12, C13, I2, I3, LED10A, LED10B, LED10C, LED11A, LED11B, LED11C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
