File: PCB/keyboard0.kicad_sch (KiCad schematic)
At the start: 371 parts, among them J1 Conn_01x04, J2 SM04B-SRSS-TB(LF)(SN), J3 Conn_01x03, Q1 2N7002, SW1 SW_Push, U1 SRV05-4, U12 XC6206P332MR, U14 STM32F303CBT6, X1 TestPoint_Small, X2 TestPoint_Small, Y2 8MHz

Commit message: Switched RGB lighting to SK6812s
Parts:
- removed C1, C11, C13, C6, C8, C9: 100nF, Capacitor_SMD:C_0805_2012Metric, symbol Device:C_Small
- removed C10, C12, C5: 1uF, Capacitor_SMD:C_0805_2012Metric, symbol Device:C_Small
- removed D+1, D-1: TestPoint_Small, TestPoint:TestPoint_Pad_1.5x1.5mm, symbol Connector:TestPoint_Small
- removed I1, I2, I3: IS31FL3731-QFLS2, Package_DFN_QFN:QFN-28-1EP_4x4mm_P0.4mm_EP2.3x2.3mm, symbol random-keyboard-parts:IS31FL3731-QFLS2
- removed LED1, LED10, LED11, LED12, LED13, LED14, LED15, LED16, LED17, LED18, LED19, LED2, LED20, LED21, LED22, LED23, LED24, LED25, LED26, LED27, LED28, LED29, LED3, LED30, LED31, LED32, LED33, LED34, LED35, LED36, LED37, LED38, LED39, LED4, LED40, LED41, LED42, LED43, LED44, LED45, LED46, LED47, LED48, LED49, LED5, LED50, LED51, LED52, LED53, LED54, LED55, LED56, LED57, LED58, LED59, LED6, LED60, LED61, LED62, LED63, LED64, LED65, LED66, LED67, LED68, LED69, LED7, LED70, LED71, LED72, LED73, LED74, LED75, LED76, LED77, LED78, LED79, LED8, LED80, LED81, LED82, LED83, LED84, LED85, LED86, LED87, LED88, LED89, LED9, LED90: LED_ABGR, custom-footprints:MHT151RGBCT_with_outline, symbol Device:LED_ABGR
- removed R11, R15, R16: 20k, Resistor_SMD:R_0805_2012Metric, symbol Device:R_Small
- added LC1, LC10, LC11, LC12, LC13, LC14, LC15, LC16, LC17, LC18, LC19, LC2, LC20, LC21, LC22, LC23, LC24, LC25, LC26, LC27, LC28, LC29, LC3, LC30, LC31, LC32, LC33, LC34, LC35, LC36, LC37, LC38, LC39, LC4, LC40, LC41, LC42, LC43, LC44, LC45, LC46, LC47, LC48, LC49, LC5, LC50, LC51, LC52, LC53, LC54, LC55, LC56, LC57, LC58, LC59, LC6, LC60, LC61, LC62, LC63, LC64, LC65, LC66, LC67, LC68, LC69, LC7, LC70, LC71, LC72, LC73, LC74, LC75, LC76, LC77, LC78, LC79, LC8, LC80, LC81, LC82, LC83, LC84, LC85, LC86, LC87, LC88, LC89, LC9, LC90: 100nF, Capacitor_SMD:C_0805_2012Metric, symbol Device:C_Small
- added LED1, LED10, LED11, LED12, LED13, LED14, LED15, LED16, LED17, LED18, LED19, LED2, LED20, LED21, LED22, LED23, LED24, LED25, LED26, LED27, LED28, LED29, LED3, LED30, LED31, LED32, LED33, LED34, LED35, LED36, LED37, LED38, LED39, LED4, LED40, LED41, LED42, LED43, LED44, LED45, LED46, LED47, LED48, LED49, LED5, LED50, LED51, LED52, LED53, LED54, LED55, LED56, LED57, LED58, LED59, LED6, LED60, LED61, LED62, LED63, LED64, LED65, LED66, LED67, LED68, LED69, LED7, LED70, LED71, LED72, LED73, LED74, LED75, LED76, LED77, LED78, LED79, LED8, LED80, LED81, LED82, LED83, LED84, LED85, LED86, LED87, LED88, LED89, LED9, LED90: SK6812MINI, custom-footprints:YS-SK6812MINI-E, symbol LED:SK6812MINI
- added U2: 74LVC1G34, Package_TO_SOT_SMD:SOT-23-5_HandSoldering, symbol 74xGxx:74LVC1G34
- added U3: SRV05-4, Package_TO_SOT_SMD:SOT-23-6_Handsoldering, symbol Power_Protection:SRV05-4
- FB1, FB15, FB5: symbol Device:Ferrite_Bead_Small -> Device:FerriteBead_Small
- ROT1, ROT2: symbol Device:Rotary_Encoder_Switch -> Device:RotaryEncoder_Switch
- U1: footprint Package_TO_SOT_SMD:SOT-23-6 -> Package_TO_SOT_SMD:SOT-23-6_Handsoldering
- renumbered BOOT1 to BKL1
Connections:
- net VCC is gone; now on net VBUS: D5.2 (A), F8.1, J2.1 (Pin_1)
- net +5V: now also FB1.2, FB15.2, LC1.2, LC10.2, LC11.2, LC12.2, LC13.2, LC14.2, LC15.2, LC16.2, LC17.2, LC18.2, LC19.2, LC2.2, LC20.2, LC21.2, LC22.2, LC23.2, LC24.2, LC25.2, LC26.2, LC27.2, LC28.2, LC29.2, LC3.2, LC30.2, LC31.2, LC32.2, LC33.2, LC34.2, LC35.2, LC36.2, LC37.2, LC38.2, LC39.2, LC4.2, LC40.2, LC41.2, LC42.2, LC43.2, LC44.2, LC45.2, LC46.2, LC47.2, LC48.2, LC49.2, LC5.2, LC50.2, LC51.2, LC52.2, LC53.2, LC54.2, LC55.2, LC56.2, LC57.2, LC58.2, LC59.2, LC6.2, LC60.2, LC61.2, LC62.2, LC63.2, LC64.2, LC65.2, LC66.2, LC67.2, LC68.2, LC69.2, LC7.2, LC70.2, LC71.2, LC72.2, LC73.2, LC74.2, LC75.2, LC76.2, LC77.2, LC78.2, LC79.2, LC8.2, LC80.2, LC81.2, LC82.2, LC83.2, LC84.2, LC85.2, LC86.2, LC87.2, LC88.2, LC89.2, LC9.2, LC90.2, LED1.4 (VDD), LED10.4 (VDD), LED11.4 (VDD), LED12.4 (VDD), LED13.4 (VDD), LED14.4 (VDD), LED15.4 (VDD), LED16.4 (VDD), LED17.4 (VDD), LED18.4 (VDD), LED19.4 (VDD), LED2.4 (VDD), LED20.4 (VDD), LED21.4 (VDD), LED22.4 (VDD), LED23.4 (VDD), LED24.4 (VDD), LED25.4 (VDD), LED26.4 (VDD), LED27.4 (VDD), LED28.4 (VDD), LED29.4 (VDD), LED3.4 (VDD), LED30.4 (VDD), LED31.4 (VDD), LED32.4 (VDD), LED33.4 (VDD), LED34.4 (VDD), LED35.4 (VDD), LED36.4 (VDD), LED37.4 (VDD), LED38.4 (VDD), LED39.4 (VDD), LED4.4 (VDD), LED40.4 (VDD), LED41.4 (VDD), LED42.4 (VDD), LED43.4 (VDD), LED44.4 (VDD), LED45.4 (VDD), LED46.4 (VDD), LED47.4 (VDD), LED48.4 (VDD), LED49.4 (VDD), LED5.4 (VDD), LED50.4 (VDD), LED51.4 (VDD), LED52.4 (VDD), LED53.4 (VDD), LED54.4 (VDD), LED55.4 (VDD), LED56.4 (VDD), LED57.4 (VDD), LED58.4 (VDD), LED59.4 (VDD), LED6.4 (VDD), LED60.4 (VDD), LED61.4 (VDD), LED62.4 (VDD), LED63.4 (VDD), LED64.4 (VDD), LED65.4 (VDD), LED66.4 (VDD), LED67.4 (VDD), LED68.4 (VDD), LED69.4 (VDD), LED7.4 (VDD), LED70.4 (VDD), LED71.4 (VDD), LED72.4 (VDD), LED73.4 (VDD), LED74.4 (VDD), LED75.4 (VDD), LED76.4 (VDD), LED77.4 (VDD), LED78.4 (VDD), LED79.4 (VDD), LED8.4 (VDD), LED80.4 (VDD), LED81.4 (VDD), LED82.4 (VDD), LED83.4 (VDD), LED84.4 (VDD), LED85.4 (VDD), LED86.4 (VDD), LED87.4 (VDD), LED88.4 (VDD), LED89.4 (VDD), LED9.4 (VDD), LED90.4 (VDD), U2.5 (VCC), U3.5 (VP)
- net BOOT1: no longer BKL1.1, U14.20 (PB2)
- net COL0: now also ROT1.S1
- net COL17: now also ROT2.S1
- net D+: now also U3.1 (IO1)
- net D-: now also U3.6 (IO4)
- net ENCODER_A: now also ROT1.A, ROT2.A
- net ENCODER_B1: now also ROT1.B
- net ENCODER_B2: now also ROT2.B
- net Earth: now also FB5.2
- net GND: now also FB5.1, ROT1.C, ROT2.C, LC1.1, LC10.1, LC11.1, LC12.1, LC13.1, LC14.1, LC15.1, LC16.1, LC17.1, LC18.1, LC19.1, LC2.1, LC20.1, LC21.1, LC22.1, LC23.1, LC24.1, LC25.1, LC26.1, LC27.1, LC28.1, LC29.1, LC3.1, LC30.1, LC31.1, LC32.1, LC33.1, LC34.1, LC35.1, LC36.1, LC37.1, LC38.1, LC39.1, LC4.1, LC40.1, LC41.1, LC42.1, LC43.1, LC44.1, LC45.1, LC46.1, LC47.1, LC48.1, LC49.1, LC5.1, LC50.1, LC51.1, LC52.1, LC53.1, LC54.1, LC55.1, LC56.1, LC57.1, LC58.1, LC59.1, LC6.1, LC60.1, LC61.1, LC62.1, LC63.1, LC64.1, LC65.1, LC66.1, LC67.1, LC68.1, LC69.1, LC7.1, LC70.1, LC71.1, LC72.1, LC73.1, LC74.1, LC75.1, LC76.1, LC77.1, LC78.1, LC79.1, LC8.1, LC80.1, LC81.1, LC82.1, LC83.1, LC84.1, LC85.1, LC86.1, LC87.1, LC88.1, LC89.1, LC9.1, LC90.1, LED1.2 (VSS), LED10.2 (VSS), LED11.2 (VSS), LED12.2 (VSS), LED13.2 (VSS), LED14.2 (VSS), LED15.2 (VSS), LED16.2 (VSS), LED17.2 (VSS), LED18.2 (VSS), LED19.2 (VSS), LED2.2 (VSS), LED20.2 (VSS), LED21.2 (VSS), LED22.2 (VSS), LED23.2 (VSS), LED24.2 (VSS), LED25.2 (VSS), LED26.2 (VSS), LED27.2 (VSS), LED28.2 (VSS), LED29.2 (VSS), LED3.2 (VSS), LED30.2 (VSS), LED31.2 (VSS), LED32.2 (VSS), LED33.2 (VSS), LED34.2 (VSS), LED35.2 (VSS), LED36.2 (VSS), LED37.2 (VSS), LED38.2 (VSS), LED39.2 (VSS), LED4.2 (VSS), LED40.2 (VSS), LED41.2 (VSS), LED42.2 (VSS), LED43.2 (VSS), LED44.2 (VSS), LED45.2 (VSS), LED46.2 (VSS), LED47.2 (VSS), LED48.2 (VSS), LED49.2 (VSS), LED5.2 (VSS), LED50.2 (VSS), LED51.2 (VSS), LED52.2 (VSS), LED53.2 (VSS), LED54.2 (VSS), LED55.2 (VSS), LED56.2 (VSS), LED57.2 (VSS), LED58.2 (VSS), LED59.2 (VSS), LED6.2 (VSS), LED60.2 (VSS), LED61.2 (VSS), LED62.2 (VSS), LED63.2 (VSS), LED64.2 (VSS), LED65.2 (VSS), LED66.2 (VSS), LED67.2 (VSS), LED68.2 (VSS), LED69.2 (VSS), LED7.2 (VSS), LED70.2 (VSS), LED71.2 (VSS), LED72.2 (VSS), LED73.2 (VSS), LED74.2 (VSS), LED75.2 (VSS), LED76.2 (VSS), LED77.2 (VSS), LED78.2 (VSS), LED79.2 (VSS), LED8.2 (VSS), LED80.2 (VSS), LED81.2 (VSS), LED82.2 (VSS), LED83.2 (VSS), LED84.2 (VSS), LED85.2 (VSS), LED86.2 (VSS), LED87.2 (VSS), LED88.2 (VSS), LED89.2 (VSS), LED9.2 (VSS), LED90.2 (VSS), U2.3 (GND), U3.2 (VN)
- net at D4.2 (A): now also ROT2.S2
- net at D3.2 (A): now also ROT1.S2
- net at F8.2: now also FB15.1
- net at F1.2: now also FB1.1
- new net: LED76.1 (DOUT), LED77.3 (DIN)
- new net: LED75.1 (DOUT), LED76.3 (DIN)
- new net: LED39.1 (DOUT), LED40.3 (DIN)
- new net: LED72.1 (DOUT), LED73.3 (DIN)
- new net: LED71.1 (DOUT), LED72.3 (DIN)
- new net: LED32.1 (DOUT), LED33.3 (DIN)
- new net: LED31.1 (DOUT), LED32.3 (DIN)
- new net: LED43.1 (DOUT), LED44.3 (DIN)
- new net: LED42.1 (DOUT), LED43.3 (DIN)
- new net: LED59.1 (DOUT), LED60.3 (DIN)
- new net: LED58.1 (DOUT), LED59.3 (DIN)
- new net: LED82.1 (DOUT), LED83.3 (DIN)
- new net: LED81.1 (DOUT), LED82.3 (DIN)
- new net: LED83.1 (DOUT), LED84.3 (DIN)
- new net: LED14.1 (DOUT), LED15.3 (DIN)
- new net: LED13.1 (DOUT), LED14.3 (DIN)
- new net: LED68.1 (DOUT), LED69.3 (DIN)
- new net: LED67.1 (DOUT), LED68.3 (DIN)
- new net: LED35.1 (DOUT), LED36.3 (DIN)
- new net: LED34.1 (DOUT), LED35.3 (DIN)
- new net: LED18.1 (DOUT), LED19.3 (DIN)
- new net: LED17.1 (DOUT), LED18.3 (DIN)
- new net: LED74.1 (DOUT), LED75.3 (DIN)
- new net: LED88.1 (DOUT), LED89.3 (DIN)
- new net: LED87.1 (DOUT), LED88.3 (DIN)
- new net: LED54.1 (DOUT), LED55.3 (DIN)
- new net: LED53.1 (DOUT), LED54.3 (DIN)
- new net: LED57.1 (DOUT), LED58.3 (DIN)
- new net: LED15.1 (DOUT), LED16.3 (DIN)
- new net: LED52.1 (DOUT), LED53.3 (DIN)
- new net: LED51.1 (DOUT), LED52.3 (DIN)
- new net: LED79.1 (DOUT), LED80.3 (DIN)
- new net: LED78.1 (DOUT), LED79.3 (DIN)
- new net: LED49.1 (DOUT), LED50.3 (DIN)
- new net: LED48.1 (DOUT), LED49.3 (DIN)
- new net: LED22.1 (DOUT), LED23.3 (DIN)
- new net: LED21.1 (DOUT), LED22.3 (DIN)
- new net: LED77.1 (DOUT), LED78.3 (DIN)
- new net: LED27.1 (DOUT), LED28.3 (DIN)
- new net: LED26.1 (DOUT), LED27.3 (DIN)
- new net: LED69.1 (DOUT), LED70.3 (DIN)
- new net: LED10.3 (DIN), LED9.1 (DOUT)
- new net: LED45.1 (DOUT), LED46.3 (DIN)
- new net: LED44.1 (DOUT), LED45.3 (DIN)
- new net: LED1.1 (DOUT), LED2.3 (DIN)
- new net: LED89.1 (DOUT), LED90.3 (DIN)
- new net: LED33.1 (DOUT), LED34.3 (DIN)
- new net: LED38.1 (DOUT), LED39.3 (DIN)
- new net: LED37.1 (DOUT), LED38.3 (DIN)
- new net: LED11.1 (DOUT), LED12.3 (DIN)
- new net: LED86.1 (DOUT), LED87.3 (DIN)
- new net: LED85.1 (DOUT), LED86.3 (DIN)
- new net: LED8.1 (DOUT), LED9.3 (DIN)
- new net: LED7.1 (DOUT), LED8.3 (DIN)
- new net: LED41.1 (DOUT), LED42.3 (DIN)
- new net: LED56.1 (DOUT), LED57.3 (DIN)
- new net: LED12.1 (DOUT), LED13.3 (DIN)
- new net: LED66.1 (DOUT), LED67.3 (DIN)
- new net: LED36.1 (DOUT), LED37.3 (DIN)
- new net: LED65.1 (DOUT), LED66.3 (DIN)
- new net: LED2.1 (DOUT), LED3.3 (DIN)
- new net: LED25.1 (DOUT), LED26.3 (DIN)
- new net: LED24.1 (DOUT), LED25.3 (DIN)
- new net: LED6.1 (DOUT), LED7.3 (DIN)
- new net: LED5.1 (DOUT), LED6.3 (DIN)
- new net: LED63.1 (DOUT), LED64.3 (DIN)
- new net: LED62.1 (DOUT), LED63.3 (DIN)
- new net: LED55.1 (DOUT), LED56.3 (DIN)
- new net: LED46.1 (DOUT), LED47.3 (DIN)
- new net: LED47.1 (DOUT), LED48.3 (DIN)
- new net: LED19.1 (DOUT), LED20.3 (DIN)
- new net: LED4.1 (DOUT), LED5.3 (DIN)
- new net: LED3.1 (DOUT), LED4.3 (DIN)
- new net: LED61.1 (DOUT), LED62.3 (DIN)
- new net: LED29.1 (DOUT), LED30.3 (DIN)
- new net: LED16.1 (DOUT), LED17.3 (DIN)
- new net: LED73.1 (DOUT), LED74.3 (DIN)
- new net: LED23.1 (DOUT), LED24.3 (DIN)
- new net: LED28.1 (DOUT), LED29.3 (DIN)
- new net: LED64.1 (DOUT), LED65.3 (DIN)
- new net: LED84.1 (DOUT), LED85.3 (DIN)
- new net BKL_5V: LED1.3 (DIN), U2.4
- new net BLK_3V3: BKL1.1, U14.20 (PB2), U2.2
- new net DOUT_1: LED10.1 (DOUT), LED11.3 (DIN)
- new net DOUT_2: LED20.1 (DOUT), LED21.3 (DIN)
- new net DOUT_3: LED30.1 (DOUT), LED31.3 (DIN)
- new net DOUT_4: LED40.1 (DOUT), LED41.3 (DIN)
- new net DOUT_5: LED50.1 (DOUT), LED51.3 (DIN)
- new net DOUT_6: LED60.1 (DOUT), LED61.3 (DIN)
- new net DOUT_7: LED70.1 (DOUT), LED71.3 (DIN)
- new net DOUT_8: LED80.1 (DOUT), LED81.3 (DIN)
- no-connect marks 12 -> 9
Other:
- note added: "JST ESD"
- note removed: "I1"
- note removed: "I2"
- note removed: "I3"

Commit message: backlight assigned to A9
Parts:
- removed R27: 10k, Resistor_SMD:R_0805_2012Metric, symbol Device:R_Small
Connections:
- net COL0: now also U14.30 (PA9); no longer U14.31 (PA10)
- net A9 renamed B2
- net B2: now also U14.20 (PB2); no longer U14.30 (PA9)
- net BLK_3V3 renamed BKL_3V3
- net BKL_3V3: now also U14.31 (PA10); no longer U14.20 (PB2)
Other:
- moved on the sheet: BKL1, COL0

Commit message: Reassigned bottom rows (no longer compatible with p2)
Parts:
- removed ENCA1, ENCB1, ENCB2: TestPoint_Small, TestPoint:TestPoint_THTPad_D1.0mm_Drill0.5mm, symbol Connector:TestPoint_Small
- added KD1-1, KD14-1: SOD-123, Diode_SMD:D_SOD-123, symbol Device:D_Small
- added MX1-1: Optional, custom-footprints:CherryMX_1.00u_PCB_KailhSocket, symbol CherryMX:CherryMX
- added MX14-1: SCKL, custom-footprints:CherryMX_1.00u_PCB_KailhSocket, symbol CherryMX:CherryMX
- MX83: footprint custom-footprints:CherryMX_6.25u_PCB_KailhSocket_StabWireBottom -> custom-footprints:CherryMX_6.25u_PCB_KailhSocket_StabWireTop
Connections:
- net COL10: now also MX74.1; no longer MX75.1, MX84.1
- net COL11: now also MX75.1, MX84.1; no longer MX76.1, MX85.1
- net COL12: now also MX76.1, MX85.1
- net COL2: now also MX1-1.1; no longer MX67.1
- net COL3: now also MX67.1; no longer MX68.1
- net COL4: now also MX68.1; no longer MX69.1
- net COL5: now also MX69.1; no longer MX70.1
- net COL6: now also MX70.1; no longer MX71.1, MX83.1
- net COL7: now also MX71.1, MX83.1; no longer MX72.1
- net COL8: now also MX72.1; no longer MX73.1
- net COL9: now also MX73.1; no longer MX74.1
- net ROT1_ROW: now also KD1-1.1 (K), KD14-1.1 (K)
- new net: KD14-1.2 (A), MX14-1.2
- new net: KD1-1.2 (A), MX1-1.2
Other:
- moved on the sheet: KD67, KD68, KD69, KD70, KD71, KD72, KD73, KD74, KD75, KD76, KD83, KD84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

Commit message: Flipped enter stabilizer
Parts:
- MX64: footprint custom-footprints:CherryMX_2.25u_PCB_KailhSocket_StabWireBottom -> custom-footprints:CherryMX_2.25u_PCB_KailhSocket_StabWireTop
Changed lines of the file:
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@@
     (property "Reference" "MX64" (id 0) (at 392.43 146.431 0))
     (property "Value" "ENTER" (id 1) (at 392.43 148.7424 0))
-    (property "Footprint" "custom-footprints:CherryMX_2.25u_PCB_KailhSocket_StabWireBottom" (id 2) (at 392.43 158.75 0)
+    (property "Footprint" "custom-footprints:CherryMX_2.25u_PCB_KailhSocket_StabWireTop" (id 2) (at 392.43 158.75 0)
       (effects (font (size 1.27 1.27)) hide)
     )
@@
     )
     (path "/00000000-0000-0000-0000-000091a30e9e"
-      (reference "MX64") (unit 1) (value "ENTER") (footprint "custom-footprints:CherryMX_2.25u_PCB_KailhSocket_StabWireBottom")
+      (reference "MX64") (unit 1) (value "ENTER") (footprint "custom-footprints:CherryMX_2.25u_PCB_KailhSocket_StabWireTop")
     )
     (path "/00000000-0000-0000-0000-00006f6c5462"

Commit message: Added EVQWD001, exported for production
Parts:
- added D6: SOD-123, Diode_SMD:D_SOD-123, symbol Device:D_Small
- added LOGO2: Vial, custom-footprints:vial_logo, symbol Connector:TestPoint_Small
- added ROT2-1: EVQWGD001, custom-footprints:EVQWGD001, symbol Device:RotaryEncoder_Switch
- MX1.5: renamed from MX1-1; value Optional -> OPT-F0
- MX14.5: renamed from MX14-1; value SCKL -> OPT-SCKL
- ROT1, ROT2: value Rotary_Encoder_Switch -> EC11
Connections:
- net COL17: now also ROT2-1.S1
- net ENCODER_A: now also ROT2-1.A
- net ENCODER_B2: now also ROT2-1.B
- net GND: now also ROT2-1.C
- net ROW4 renamed ROT2-1_ROW
- net ROT2-1_ROW: now also D6.1 (K)
- new net: D6.2 (A), ROT2-1.S2
- no-connect marks 9 -> 10
Other:
- moved on the sheet: D3, D4, ROT1, ROT2
