File: PCB/Plate/custom_keyboard plate v2.kicad_pcb (KiCad board)
At the start: 2 copper layers, 385.7 x 133.3 mm, 1 part

Commit message: Added a lot of flex cuts
Parts:
- moved logo 3.27 mm to (415.9, 252.4)
Other:
- board size 385.7 x 133.3 mm -> 377.8 x 133.3 mm
- board text added: "© 2022 Howard Tseng"
- board text removed: "© 2021 Howard Tseng"

Commit message: Exported plate v2 for production
Parts:
- moved logo 3.17 mm to (412.7, 252.4)
Routing:
- removed copper zone on B.Cu, net (none)
- removed copper zone on F.Cu, net (none)
Other:
- board size 377.8 x 133.3 mm -> 377.8 x 134.9 mm
