File: PCB/Plate/custom_keyboard plate v2.kicad_pcb (KiCad board)
At the start: 2 copper layers, 377.8 x 134.9 mm, 1 part

Commit message: Added screw holes to plate v2
Parts:
- added logo: G***, custom-footprints:logo, B.Cu at (412.7, 255.7)
Other:
- board size 377.8 x 134.9 mm -> 377.8 x 138.1 mm
- net class Default removed
