File: PCB/Plate/custom_keyboard plate v3 bottom.kicad_pcb (KiCad board)
At the start: 2 copper layers, 395.3 x 142.9 mm, 58 parts, among them M2 MountingHole_2.2mm_M2_ISO7380, M2.5 MountingHole_2.5mm, M3 MountingHole_3.2mm_M3

Commit message: Adjusted text and graphics widths
Other:
- board text added: "JLCJLCJLCJLC"
